File: faclon-main/FalconMain/FalconMain.kicad_sch (KiCad schematic)
At the start: 78 parts

Commit message: Add more main board core components
Charger, LP buck, LiPo conns, piezo drivers, lighting driver and conns
Parts:
- removed F? (x3): Fuse_Small, symbol Device:Fuse_Small
- removed J? (x2): Conn_01x02, symbol Connector_Generic:Conn_01x02
- removed R?: ????, symbol Device:R_Small
- removed R?: ?????, symbol Device:R_Small
- added C? (x5): ?????, symbol Device:C_Small
- added D? (x3): D_Schottky_Small, symbol Device:D_Schottky_Small
- added F? (x4): Fuse_Small, symbol Device:Fuse_Small
- added J?: Conn_01x03, symbol Connector_Generic:Conn_01x03
- added J? (x4): Conn_01x02, symbol Connector_Generic:Conn_01x02
- added J?: Conn_01x04, symbol Connector_Generic:Conn_01x04
- added L? (x2): ?????, symbol Device:L_Small
- added Q? (x2): Q_NMOS_GDS, symbol Device:Q_NMOS_GDS
- added R? (x11): ????, symbol Device:R_Small
- added U?: AL8843QSP-13, JetkovKiCADLib:8-SOIC_SO-8EP_DIO, symbol JetkovKiCADLib:AL8843QSP-13
- added U?: BD9E104FJ-E2, JetkovKiCADLib:8-SOIC_8-SOP-J_ROHM, symbol JetkovKiCADLib:BD9E104FJ-E2
Connections:
- net CELL_1S: now also F?.1
- net CELL_2S: now also F?.1
- net CELL_3S: now also F?.1
- net CELL_4S: now also F?.1
- net GND: now also J?.3 (Pin_3), C?.1, C?.1, C?.2, J?.2 (Pin_2), J?.3 (Pin_3), J?.4 (Pin_4), Q?.3 (S), Q?.3 (S), R?.1, R?.1, R?.2, R?.2, U?.1 (GND), U?.2 (GND), U?.4 (GND), U?.7 (PGND), U?.EPAD
- net VBAT: now also D?.2 (A)
- net VDC: now also C?.1, J?.1 (Pin_1), C?.2, C?.2, D?.1 (K), D?.1 (K), D?.1 (K), J?.1 (Pin_1), J?.1 (Pin_1), R?.2, R?.2, U?.2 (VIN), U?.6 (VIN)
- net PWM_LED_LHS: now reaches J?.2 (Pin_2)
- net at R?.1, R?.2: now also Q?.3 (S), D?.2 (A); no longer C?.1
- net ~{CHG_EN}: now reaches R?.1
- net ~{CHG_EN}: now also R?.1, U?.6 (ICHG/EN)
- net at R?.2: now also C?.2, R?.1, U?.9 (REF)
- net at D?.2 (A): now also F?.2; no longer J?.1 (In)
- net at J?.2 (Pin_2): now also F?.2
- net at J?.3 (Pin_3): now also F?.2
- net at J?.4 (Pin_4): now also F?.2
- net at F?.2: now also J?.1 (Pin_1)
- new net: D?.2 (A), L?.1, U?.7 (SW), U?.8 (SW)
- new net: R?.1, R?.2, U?.5 (FB)
- new net: C?.2, L?.1, U?.8 (SW)
- new net: C?.1, U?.1 (BOOT)
- new net: C?.2, U?.6 (COMP)
- new net: J?.2 (Pin_2), Q?.2 (D), R?.1 (x2)
- new net: C?.1, R?.1
- new net: F?.1, J?.1 (In)
- new net +3V5: C?.1, L?.2, R?.1
- new net +5V1: R?.2
- new net 3V5_EN: U?.3 (EN)
- new net FRONT_LED+: J?.1 (Pin_1), R?.1, U?.3 (SET)
- new net FRONT_LED-: J?.2 (Pin_2), L?.2
- new net PWM_LED_FRONT: U?.5 (CTRL)
- new net PWM_LED_REAR1: J?.2 (Pin_2)
- new net PWM_LED_REAR2: J?.3 (Pin_3)
- new net PWM_LED_RHS: J?.2 (Pin_2)
- new net PWM_PIEZO_LHS: Q?.1 (G), R?.2
- new net PWM_PIEZO_RHS: Q?.1 (G), R?.2
- new net VPIEZO: J?.1 (Pin_1), J?.1 (Pin_1), R?.1, R?.1, R?.2, R?.2
Other:
- note added: "---> LDO --->"
- note added: "AC/DC Adapter"
- note added: "Batt "diode" Vf should be < 0.1V @ 5A (0.5W)"
- note added: "Can use "ideal diode" or "power oring" IC to replace VBAT diode with MOSFET"
- note added: "Front"
- note added: "LHS"
- note added: "LiPo Balance"
- note added: "LiPo Main"
- note added: "Lighting"
- note added: "Piezo Drivers"
- note added: "RHS"
- note added: "Rear"
- moved on the sheet: C?, D?, F?, J?, L?, Q?, R?, U?

Commit message: More component selection
Parts:
- removed C? (x4): ?????, symbol Device:C_Small
- removed R? (x8): 10k, symbol Device:R_Small
- added C?: 12pF, symbol Device:C_Small
- added C? (x5): ?????, symbol Device:C_Small
- added C? (x3): 10uF, symbol Device:C_Small
- added C?: 220nF, symbol Device:C_Small
- added C?: 1uF, symbol Device:C_Small
- added C?: 100nF, symbol Device:C_Small
- added D?: D_Schottky_Small, symbol Device:D_Schottky_Small
- added Q? (x2): Q_NMOS_GDS, symbol Device:Q_NMOS_GDS
- added Q?: Q_PMOS_GDS, symbol Device:Q_PMOS_GDS
- added R?: 0R, symbol Device:R_Small
- added R? (x12): 100k, symbol Device:R_Small
- added R? (x10): ????, symbol Device:R_Small
- added R?: 137k, symbol Device:R_Small
- added R?: 28k, symbol Device:R_Small
- C?: value ????? -> 47uF
- C? (x2): value ????? -> 47nF
- C? (x2): value ????? -> 100nF
- C?: value ????? -> 620pF
- C?: value ????? -> 220nF
- C? (x2): value ????? -> 10nF
- C?: value ????? -> 33uF
- C?: value ????? -> 1nF
- C?: value ????? -> 10uF
- C?: value ????? -> 2.2uF
- L?: value ????? -> 10uH
- L?: value ????? -> 47uH
- R?: value ???? -> 113k
- R?: value ???? -> DNP
- R?: value ???? -> 383k
- R?: value ???? -> 22.6m
- R?: value ???? -> 39m
- R? (x2): value ???? -> 4.7R
- R?: value ???? -> 62.6m
- R?: value ???? -> 10k
- R? (x2): value ???? -> 2k
- R? (x3): value ???? -> 100k
- R?: value ???? -> 38.3k
- R?: value ???? -> 133k
- R?: value ???? -> 49.9k
Connections:
- net +19V5: now also C?.2, R?.2
- net +3V5: now also C?.1, C?.1
- net 3V5_EN: now also D?.2 (A); no longer U?.3 (EN)
- net CELL_1S: now also R?.2, R?.2
- net CELL_1S_DIS_EN: now also R?.2
- net CELL_2S: now also R?.2, R?.2
- net CELL_2S_DIS_EN: now also R?.2
- net CELL_3S: now also R?.2, R?.2
- net CELL_3S_DIS_EN: now also R?.2
- net CELL_4S: now also R?.2, R?.2, R?.2
- net CELL_4S_DIS_EN: now also R?.2
- net GND: now also C?.1, C?.1, C?.1, C?.2, C?.2, C?.2, C?.2, C?.2, C?.2, C?.2, Q?.3 (S), Q?.3 (S), R?.1, R?.1, R?.1, R?.1, R?.1, R?.1, R?.1, R?.1, R?.1, R?.1, R?.1
- net PWM_LED_FRONT: now also U?.39 (PB3)
- net PWM_LED_LHS: now also U?.12 (PA2)
- net PWM_LED_REAR1: now also U?.16 (PA6)
- net PWM_LED_REAR2: now also U?.17 (PA7)
- net PWM_LED_RHS: now also U?.13 (PA3)
- net PWM_PIEZO_LHS: now also U?.45 (PB8)
- net PWM_PIEZO_RHS: now also U?.28 (PB15)
- net VDC: now also C?.2, C?.2, C?.2, Q?.3 (S), R?.2
- net ~{CELL_1S_DIS_EN}: now also R?.1
- net ~{CELL_2S_DIS_EN}: now also R?.1
- net ~{CELL_3S_DIS_EN}: now also R?.1
- net ~{CELL_4S_DIS_EN}: now also R?.1
- net ~{CHG_EN}: now also R?.2; no longer R?.1, R?.1, U?.6 (ICHG/EN)
- net SPR_ADC_IN0: now reaches U?.10 (PA0-WKUP1)
- net VSENSE_5V1: now reaches U?.11 (PA1)
- net VSET_ICHG: now reaches U?.14 (PA4)
- net SPI1_SCK: now reaches U?.15 (PA5)
- net VSENSE_CELL_1S: now reaches U?.18 (PB0)
- net VSENSE_CELL_2S: now reaches U?.19 (PB1)
- net EN_CELL_1S_DIS: now reaches U?.20 (PB2)
- net EN_CELL_2S_DIS: now reaches U?.21 (PB10)
- net EN_CELL_3S_DIS: now reaches U?.22 (PB11)
- net VSENSE_CELL_3S: now reaches U?.25 (PB12)
- net VSENSE_CELL_4S: now reaches U?.26 (PB13)
- net EN_CELL_4S_DIS: now reaches U?.27 (PB14)
- net GPIO_SPR: now reaches U?.29 (PA8)
- net USART1_TX: now reaches U?.30 (PA9)
- net USART1_RX: now reaches U?.31 (PA10)
- net USART1_CTS: now reaches U?.32 (PA11)
- net USART1_RTS: now reaches U?.33 (PA12)
- net SWDIO: now reaches U?.34 (PA13)
- net SWCLK: now reaches U?.37 (PA14)
- net SPI1_NSS: now reaches U?.38 (PA15)
- net SPI1_MISO: now reaches U?.40 (PB4)
- net SPI1_MOSI: now reaches U?.41 (PB5)
- net EN_3V5: now reaches U?.42 (PB6)
- net EN_5V1: now reaches U?.43 (PB7)
- net PWM_SPR: now reaches U?.46 (PB9)
- net at R?.1, R?.2, U?.5 (FB): now also C?.2
- net at R?.1, R?.2, U?.9 (REF): now also C?.1
- net at U?.13 (VH): now also C?.1
- new net: Q?.1 (G), R?.2
- new net: Q?.2 (D), R?.1
- new net: Q?.1 (G), Q?.2 (D), R?.1
- new net: R?.1, R?.1, R?.1, U?.6 (ICHG/EN)
- new net: D?.1 (K), R?.1, R?.2, U?.3 (EN)
- new net CELL_1S_ADC: C?.1, R?.1, R?.2
- new net CELL_2S_ADC: C?.1, R?.1, R?.2
- new net CELL_3S_ADC: C?.1, R?.1, R?.2
- new net CELL_4S_ADC: C?.1, C?.1, R?.1, R?.1, R?.2, R?.2
- new net VBAT_EN: Q?.1 (G), R?.2
Other:
- note added: "--> BUCK -->"
- note added: "-> C_{OUT}=20uF, R_{4}=38.3kOhms, C_{4}=620pF Alt: C_{OUT}=30uF, R_{4}=57.6kOhms, C_{4}=430pF Alt: L=22uH"
- note added: "12-14pF"
- note added: "19.5V supply enables power to the MCU MCU should maintain 3V5_EN high"
- note added: "C_{4}=1/[(2pi)(R_{4})(f_{CRS}/6)] =1/[(2pi)(3.83k)(40k/6) =623.32pF~=620pF"
- note added: "ESR < 1R"
- note added: "I_{IN(MAX)}=0.1V/R_{CSS} =0.1V/22.6mOhms =4.43A"
- note added: "I_{RPL}=(V_{OUT})(V_{IN}-V_{OUT})/[(V_{IN})(f_{OSC})(L)] =(3.5V)(15V-3.5V)/[(15V)(570kHz)(10uH)] =0.471A"
- note added: "I_{off}=10uA"
- note added: "I_{off}=?"
- note added: "I_{out}=0.1V/R_{set} R_{set}=0.1V/2.5A ~=0.039R"
- note added: "I_{q}=350uA CTRL floating"
- note added: "L>{V_{BATT}[V_{DCIN(MAX)}-V_{BATT}]}/{[V_{DCIN(MAX)}][f_{SW}][I_{CHG}][LIR]} >((14.8V)(19.5V-14.8V))/((19.5V)(300kHz)(2.5A)(0.3)) >15.85uH"
- note added: "R_{4}=[(2pi)(V_{OUT})(f_{CRS})(C_{OUT})]/[(V_{FB})(G_{MP})(G_{MA})] =[(2pi)(V_{OUT})(f_{CRS})(C_{OUT})]/[(0.8V)(7A/V)(82uA/V)] =13682.8948(V_{OUT})(f_{CRS})(C_{OUT}) =13682.8948(3.5)(40k)(20u) =38.312kOhms~=38.3kOhms"
- note added: "R_{CSB}=0.2V(V_{ICH-EN}/V_{REF})/I_{CHG} =0.2V(3.3V/4.2V)/2.5A ~=62.6mOhms I_{CHG}=0.2V(3.3V/4.2V)/0.0626R=2.5103A"
- note added: "TO DO ------------------------------------ - Decide if/how to do low-batt shutdown/ship-mode - Decide how to handle power ORing - JTAG conn - Select passive component values - Select passive component values for LP LED bucks - Map MCU inputs (need dividers for ADC) - Select LP LDO - Select HP buck regulator - Select remaining passive component values - Select passive components and MOSFETS (shoul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"
- note added: "V_{ICH-EN}=I_{CHG} * 1.3146"
- note added: "V_{Iout}=20(R_{CSB} * I_{chg}) C_{load} < 5nF"
- note added: "V_{OUT}=0.8[(R_{1}+R_{2})/R_{2}] =0.8[(383k+113k)/113k]=3.512V"
- note added: "V_{RPL}=I_{RPL}[R_{ESR}+1/(8(C_{OUT})(f_{OSC}))] =(0.471A)[10mOhm+1/(8(20uF)(570kHz))] =9.87mV"
- note added: "V_{TL}=0.8V V_{TH}=2.5V"
- note added: "V_{VADJ}=9.5(V_{CELL})-9(V_{REF}) =9.5(4.1V)-9(4.2V)=1.15V R_{2}=R_{1}[V_{VADJ}/(V_{REF}-V_{VADJ})] =133k*(1.15/(4.2-1.15)~=49.9k V_{VADJ}=1.14587V V_{CELL}=(1.14587V+9(4.2V))/9.5=4.0996V"
- note added: "f_{CRS}=40kHz"
- note added: "f_{OSC}=570kHz"
- moved on the sheet: C?, D?, F?, J?, L?, R?, U?

Commit message: Cell vsense WIP
Parts:
- removed C? (x4): ?????, symbol Device:C_Small
- removed Q?: Q_NMOS_GDS, symbol Device:Q_NMOS_GDS
- removed R? (x2): ????, symbol Device:R_Small
- removed R?: 100k, symbol Device:R_Small
- added C? (x7): 330nF, symbol Device:C_Small
- added C?: 100nF, symbol Device:C_Small
- added Q? (x4): Q_PMOS_GDS, symbol Device:Q_PMOS_GDS
- added Q?: Q_NMOS_GDS, symbol Device:Q_NMOS_GDS
- added R? (x2): 226k, symbol Device:R_Small
- added R?: 619k, symbol Device:R_Small
- added R?: 576k, symbol Device:R_Small
- added R?: 100k, symbol Device:R_Small
- added R?: 100K, symbol Device:R_Small
- added R?: 750k, symbol Device:R_Small
- added R?: 332k, symbol Device:R_Small
- added R?: 169k, symbol Device:R_Small
- added R?: 698k, symbol Device:R_Small
- C?: value 100nF -> 1uF
- C?: value ????? -> 330nF
- R? (x2): value ???? -> 226k
- R?: value ???? -> 750k
- R?: value ???? -> 332k
- R?: value ???? -> 576k
- R?: value ???? -> 619k
- R?: value ???? -> 698k
- R?: value ???? -> 169k
Connections:
- net +3V3: now also Q?.1 (G), R?.2
- net CELL_1S: now also Q?.3 (S)
- net CELL_1S_ADC: now also C?.1, C?.1, R?.1, R?.2
- net CELL_2S: now also Q?.3 (S)
- net CELL_2S_ADC: now also C?.1, C?.1, R?.1, R?.2
- net CELL_3S: now also Q?.3 (S)
- net CELL_3S_ADC: now also C?.1, C?.1, R?.1, R?.2
- net CELL_4S: now also Q?.3 (S), R?.2
- net CELL_4S_ADC: now also C?.1, R?.1, R?.2
- net GND: now also C?.2, C?.2, C?.2, C?.2, C?.2, C?.2, C?.2, C?.2, Q?.3 (S), R?.1, R?.1, R?.1, R?.1, R?.1
- net VDDA: now also C?.1
- new net: Q?.2 (D), R?.2 (x4)
- new net: Q?.1 (G), Q?.1 (G), Q?.1 (G), Q?.1 (G), Q?.2 (D), R?.1
Other:
- note added: "FETs prevent current injection into MCU IO pins when MCU is unpowered"
- note added: "I_{Q}=250uA I_{off}=10uA P_{off}=148uW"
- note added: "I_{off}=10uA P_{off}=148uW"
- note added: "P=353uW"
- note added: "Place dividers and caps close to MCU pins"
- note added: "R_{TH}=(R_{1}//R_{2}) R_{TH(MAX)}=211k"
- note added: "Set total resistance between 0.8-1MOhm to reduce discharge"
- note added: "T_{RC}=(R1//R2)*C C<(0.1/211k)=474nF"
- note added: "[ST: AN2834] C>131nF"
- note removed: "I_{off}=10uA"
- moved on the sheet: C?, L?

Commit message: Define connectors
Parts:
- removed C? (x4): 330nF, symbol Device:C_Small
- removed J? (x3): Conn_01x02, symbol Connector_Generic:Conn_01x02
- removed J?: Conn_01x04, symbol Connector_Generic:Conn_01x04
- removed J?: Conn_Coaxial_Power, symbol Connector:Conn_Coaxial_Power
- removed R? (x2): 226k, symbol Device:R_Small
- removed R?: 750k, symbol Device:R_Small
- removed R?: 332k, symbol Device:R_Small
- removed R?: 576k, symbol Device:R_Small
- removed R?: 619k, symbol Device:R_Small
- removed R?: 698k, symbol Device:R_Small
- removed R? (x2): ????, symbol Device:R_Small
- removed R?: 169k, symbol Device:R_Small
- removed R?: 100k, symbol Device:R_Small
- added C?: 10uF, symbol Device:C_Small
- added C?: DNP, symbol Device:C_Small
- added C? (x4): ?????, symbol Device:C_Small
- added D? (x2): D_Schottky_Small, symbol Device:D_Schottky_Small
- added J?: Conn_02x03_Odd_Even, symbol Connector_Generic:Conn_02x03_Odd_Even
- added J?: Conn_01x02, symbol Connector_Generic:Conn_01x02
- added J?: Conn_02x05_Odd_Even, symbol Connector_Generic:Conn_02x05_Odd_Even
- added J? (x2): Conn_01x05, symbol Connector_Generic:Conn_01x05
- added J?: Conn_02x15_Odd_Even, symbol Connector_Generic:Conn_02x15_Odd_Even
- added J?: Conn_01x03, symbol Connector_Generic:Conn_01x03
- added L?: 100uH, symbol Device:L_Small
- added R? (x2): 1M, symbol Device:R_Small
- added R? (x2): ????, symbol Device:R_Small
- added R?: 499m, symbol Device:R_Small
- added R?: DNP, symbol Device:R_Small
- added R?: 100k, symbol Device:R_Small
- added U?: AL8843QSP-13, JetkovKiCADLib:8-SOIC_SO-8EP_DIO, symbol JetkovKiCADLib:AL8843QSP-13
- added Y?: 8MHz, symbol Device:Crystal_Small
- added Y?: 32.768kHz, symbol Device:Crystal_Small
Connections:
- net GND is gone; now on net +19V5: C?.1, C?.1, C?.1, C?.1, C?.1, C?.1, C?.1, C?.1, C?.2, C?.2, C?.2, C?.2, C?.2, C?.2, C?.2, C?.2, C?.2, C?.2, C?.2, C?.2, C?.2, C?.2, C?.2, C?.2, C?.2, C?.2, D?.2 (A), J?.1 (Pin_1), J?.2 (Pin_2), J?.3 (Pin_3), J?.3 (Pin_3), Q?.3 (S), Q?.3 (S), Q?.3 (S), Q?.3 (S), Q?.3 (S), Q?.3 (S), Q?.3 (S), Q?.3 (S), R?.1, R?.1, R?.1, R?.1, R?.1, R?.1, R?.1, R?.1, R?.1, R?.1, R?.1, R?.1, R?.1, R?.2, R?.2, R?.2, R?.2, R?.2, U?.1 (GND), U?.12 (GND), U?.2 (GND), U?.23 (VSS_1), U?.35 (VSS_2), U?.4 (GND), U?.47 (VSS_3), U?.7 (PGND), U?.8 (VSSA), U?.EPAD
- net +19V5: now also F?.1, C?.1, C?.1, C?.1, C?.2, C?.2, C?.2, D?.2 (A), J?.1 (Pin_1), J?.11 (Pin_11), J?.12 (Pin_12), J?.21 (Pin_21), J?.29 (Pin_29), J?.3 (Pin_3), J?.3 (Pin_3), J?.3 (Pin_3), J?.30 (Pin_30), J?.4 (Pin_4), J?.4 (Pin_4), J?.4 (Pin_4), J?.5 (Pin_5), J?.5 (Pin_5), J?.6 (Pin_6), J?.7 (Pin_7), J?.7 (Pin_7), J?.8 (Pin_8), J?.9 (Pin_9), R?.1, R?.1, R?.1, U?.1 (GND), U?.2 (GND), U?.EPAD; no longer C?.1, C?.2, D?.1 (K), R?.1, R?.1, R?.2, U?.15 (DCIN)
- net +3V3: now also J?.1 (Pin_1), R?.2
- net +5V1: now also J?.1 (Pin_1), J?.10 (Pin_10), J?.2 (Pin_2), J?.2 (Pin_2), J?.4 (Pin_4), J?.6 (Pin_6), J?.8 (Pin_8), R?.2
- net EN_3V5: now also J?.1 (Pin_1)
- net EN_5V1: now also J?.2 (Pin_2)
- net PWM_LED_FRONT: now also R?.2
- net PWM_LED_LHS: now also J?.5 (Pin_5), R?.2, U?.5 (CTRL)
- net PWM_LED_REAR1: now also J?.9 (Pin_9)
- net PWM_LED_REAR2: now also J?.10 (Pin_10)
- net PWM_LED_RHS: now also J?.5 (Pin_5)
- net SPI1_MISO: now also J?.25 (Pin_25)
- net SPI1_MOSI: now also J?.23 (Pin_23)
- net SPI1_NSS: now also J?.28 (Pin_28)
- net SPI1_SCK: now also J?.27 (Pin_27)
- net SWCLK: now also J?.4 (Pin_4)
- net SWDIO: now also J?.2 (Pin_2)
- net USART1_CTS: now also J?.24 (Pin_24)
- net USART1_RTS: now also J?.20 (Pin_20)
- net USART1_RX: now also J?.26 (Pin_26)
- net USART1_TX: now also J?.22 (Pin_22)
- net VBAT: now also R?.2
- net VDC: now also C?.1, C?.2, D?.1 (K), R?.1, R?.1, U?.15 (DCIN); no longer C?.1, C?.2, C?.2, C?.2, D?.1 (K), D?.1 (K), D?.1 (K), J?.1 (Pin_1), J?.1 (Pin_1), Q?.3 (S), R?.2, R?.2, U?.2 (VIN), U?.6 (VIN)
- net VPIEZO: now also J?.1 (Pin_1), J?.1 (Pin_1), R?.1, R?.1
- net VSET_ICHG: now also J?.3 (Pin_3)
- net SPR_PC13: now reaches U?.2 (PC13_WKUP2)
- net SPR_PC13: now also J?.16 (Pin_16)
- net at U?.3 (PC14-OSC32_IN): now also C?.2, Y?.1
- net at U?.4 (PC15-OSC32_OUT): now also C?.1, Y?.2
- net BOOT0: now reaches U?.44 (BOOT0)
- net BOOT0: now also J?.19 (Pin_19), R?.1, R?.2
- net at U?.5 (PH0-OSC_IN): now also C?.1, Y?.2
- net at U?.6 (PH1-OSC_OUT): now also C?.2, Y?.1
- net NRST: now reaches U?.7 (NRST)
- net NRST: now also C?.1, J?.6 (Pin_6)
- net DRV_PIEZO_RHS: now reaches Q?.2 (D), R?.1
- net DRV_PIEZO_RHS: now also J?.2 (Pin_2)
- net DRV_PIEZO_LHS: now reaches Q?.2 (D), R?.1
- net DRV_PIEZO_LHS: now also J?.2 (Pin_2)
- net VSYS_SW: now reaches Q?.2 (D)
- net VSYS_SW: now also C?.2, D?.1 (K), J?.1 (Pin_1), J?.1 (Pin_1), R?.2, U?.6 (VIN), C?.2, D?.1 (K), J?.3 (Pin_3), J?.3 (Pin_3), J?.5 (Pin_5), R?.2, U?.6 (VIN)
- net FRONT_LED+ renamed FRONT_LED_P
- net FRONT_LED_P: now also J?.1 (Pin_1)
- net FRONT_LED- renamed FRONT_LED_N
- net FRONT_LED_N: now also J?.2 (Pin_2)
- net GPIO_SPR renamed SPR_PA8
- net SPR_PA8: now also J?.13 (Pin_13)
- net PWM_SPR renamed SPR_PB9
- net SPR_PB9: now also J?.14 (Pin_14)
- net SPR_ADC_IN0 renamed SPR_PA0
- net SPR_PA0: now also J?.15 (Pin_15)
- new net: D?.2 (A), L?.1, U?.7 (SW), U?.8 (SW)
- new net: D?.1 (K), R?.2
- new net: R?.1, U?.3 (SET)
- new net VSYS: C?.1, C?.2, C?.2, D?.1 (K), D?.1 (K), Q?.3 (S), R?.2, U?.2 (VIN)
- no-connect marks 0 -> 2
Other:
- note added: "0.4A"
- note added: "4A"
- note added: "AIN0"
- note added: "Also purchase 412mOhm"
- note added: "C_{STRAY}~=10pF Recommend C_{L}=20pF @ R_{S}=30k"
- note added: "C_{STRAY}~=5pF Recommend C_{L}=8pF @ R_{S}=30k"
- note added: "I_{out}=0.1V/R_{set} R_{set}=0.1V/0.2A ~=0.499R"
- note added: "LiPo Cell Balancing"
- note added: "LiPo Cell Voltage Sensing"
- note added: "Maybe use same inductor as 5.1V buck?"
- note added: "PWM"
- note added: "Phone"
- note added: "TO DO ------------------------------------ / Decide if/how to do low-batt shutdown/ship-mode / Decide how to handle power ORing / Crystals - JTAG conn, USB conn - Select passive component values - Select passive component values for LP LED bucks - Map MCU inputs (need dividers for ADC) - Select LP LDO - Select HP buck regulator - Select remaining passive component values - Select passive componen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"
- note added: "VDC_METERED"
- note added: "WAKE"
- note added: "t_{ON(MIN)}=500nS"
- note added: "t_{ON}=[L(0.26)(I_{LED})]/[V_{IN}-V_{LED}-I_{LED}(R_{SET}+R_{L}+R_{SW})] =[100uH(0.26)(0.2A)]/[14.8V-9.6V-0.2A(0.5+0.1+0.2)Ohms] =1.0317uS"
- note added: "t_{ON}=[L(0.26)(I_{LED})]/[V_{IN}-V_{LED}-I_{LED}(R_{SET}+R_{L}+R_{SW})] =[47uH(0.26)(1A)]/[16V-9.6V-1A(0.1+0.1+0.2)Ohms] =2.0366uS"
- note added: "t_{ON}=[L(0.26)(I_{LED})]/[V_{IN}-V_{LED}-I_{LED}(R_{SET}+R_{L}+R_{SW})] =[47uH(0.26)(3A)]/[14.8V-3V-3A(0.039+0.1+0.2)Ohms] =3.3997uS"
- note removed: "Front"
- note removed: "P=353uW"
- note removed: "Set total resistance between 0.8-1MOhm to reduce discharge"
- note removed: "TO DO ------------------------------------ - Decide if/how to do low-batt shutdown/ship-mode - Decide how to handle power ORing - JTAG conn - Select passive component values - Select passive component values for LP LED bucks - Map MCU inputs (need dividers for ADC) - Select LP LDO - Select HP buck regulator - Select remaining passive component values - Select passive components and MOSFETS (shoul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"
- moved on the sheet: C?, D?, F?, J?, L?, Q?, R?, U?
