File: faclon-main/FalconMain/FalconMain.kicad_sch (KiCad schematic)
At the start: 156 parts

Commit message: Select components, last power design wip
Parts:
- removed C?: 47uF, symbol Device:C_Polarized_Small
- removed C?: 620pF, symbol Device:C_Small
- removed C? (x3): 330nF, symbol Device:C_Small
- removed C?: 47nF, symbol Device:C_Small
- removed D? (x3): D_Schottky_Small, symbol Device:D_Schottky_Small
- removed F? (x5): Fuse_Small, symbol Device:Fuse_Small
- removed J? (x2): Conn_01x03, symbol Connector_Generic:Conn_01x03
- removed J?: Conn_02x05_Odd_Even, symbol Connector_Generic:Conn_02x05_Odd_Even
- removed J?: Conn_01x05, symbol Connector_Generic:Conn_01x05
- removed R?: 113k, symbol Device:R_Small
- added C30: DNP, symbol Device:C_Small
- added C39, C40, C41: 1uF, symbol Device:C_Small
- added C? (x10): ?????, symbol Device:C_Small
- added C?: 47nF, symbol Device:C_Small
- added C?: 620pF, symbol Device:C_Small
- added C? (x3): ?????, symbol Device:C_Polarized_Small
- added C?: 47uF, symbol Device:C_Polarized_Small
- added C?: 100nF, symbol Device:C_Small
- added D3, D? (x2): D_Schottky_Small, symbol Device:D_Schottky_Small
- added F1, F4: 6A, Resistor_SMD:R_0603_1608Metric, symbol Device:Fuse_Small
- added F2, F3: 3.5A, symbol Device:Fuse_Small
- added F6, F7, F8: 200mA, symbol Device:Fuse_Small
- added J3: Nano-Fit, symbol Connector_Generic:Conn_01x05
- added J6: Nano-Fit, symbol Connector_Generic:Conn_02x06_Odd_Even
- added L?: 3.3uH, symbol Device:L_Small
- added Q? (x4): Q_NMOS_GDS, symbol Device:Q_NMOS_GDS
- added Q? (x2): Q_PMOS_GDS, symbol Device:Q_PMOS_GDS
- added R30: DNP, symbol Device:R_Small
- added R31: 100k, symbol Device:R_Small
- added R48: 133k, Resistor_SMD:R_0402_1005Metric, symbol Device:R_Small
- added R5: 200R, symbol Device:R_Small
- added R? (x7): ????, symbol Device:R_Small
- added R?: 0R, symbol Device:R_Small
- added U?: NCP164ASN330T1G, JetkovKiCADLib:SOT-23-5_TSOP−5_ON, symbol JetkovKiCADLib:NCP164ASN330T1G
- added U?: LTC4412ES6#TRPBF, symbol JetkovKiCADLib:LTC4412ES6#TRPBF
- added U?: NCP3020BDR2G, symbol JetkovKiCADLib:NCP3020BDR2G
- C38: renamed from C?; value 330nF -> 1uF
- F5: renamed from F?; value Fuse_Small -> 200mA; Current 200mA -> (none)
- J1: renamed from J?; value Conn_01x02 -> Nano-Fit; Manufacturer (none) -> Molex; Part Number (none) -> 1053091102; Temp Range (none) -> -40°C +105°C
- J2: renamed from J?; value Conn_01x05 -> Nano-Fit; Manufacturer (none) -> Molex; Part Number (none) -> 1053091105; Temp Range (none) -> -40°C +105°C
- J4: renamed from J?; value Conn_01x02 -> PTH
- J5: renamed from J?; value Conn_02x15_Odd_Even -> 100mil; Manufacturer (none) -> Sullins Connector Solutions; Part Number (none) -> PREC015DAAN-RC; Temp Range (none) -> -40°C +105°C
- J7: renamed from J?; value Conn_01x05 -> JST-XH; Manufacturer (none) -> JST Sales America Inc.; Part Number (none) -> B5B-XH-AM(LF)(SN); Temp Range (none) -> -25°C +85°C
- J8: renamed from J?; value Conn_02x03_Odd_Even -> 100mil; Manufacturer (none) -> Sullins Connector Solutions; Part Number (none) -> PREC003DFAN-RC; Temp Range (none) -> -40°C +105°C
- J9: renamed from J?; value Conn_01x03 -> 100mil; Manufacturer (none) -> Sullins Connector Solutions; Part Number (none) -> PREC040SAAN-RC; Temp Range (none) -> -40°C +105°C
- R17: renamed from R?; footprint (none) -> Resistor_SMD:R_0402_1005Metric; Manufacturer (none) -> Stackpole Electronics Inc; Part Number (none) -> RMCF0402FT133K; Power (none) -> 0.063W; Temp Range (none) -> -55°C +155°C; Tolerance (none) -> 1%
- R18: renamed from R?; footprint (none) -> Resistor_SMD:R_0402_1005Metric; Manufacturer (none) -> Stackpole Electronics Inc; Part Number (none) -> RMCF0402FT49K9; Power (none) -> 0.063W; Temp Range (none) -> -55°C +155°C; Tolerance (none) -> 1%
- R36: renamed from R?; value 137k -> 243k
- R37: renamed from R?; value 28k -> 49.9
- R47: renamed from R?; value 383k -> 453k; footprint (none) -> Resistor_SMD:R_0402_1005Metric; Manufacturer (none) -> Stackpole Electronics Inc; Part Number (none) -> RMCF0402FT453K; Power (none) -> 0.063W; Temp Range (none) -> -55°C +155°C; Tolerance (none) -> 1%
- R51: renamed from R?; value 750k -> 221k
- R52: renamed from R?; value 169k -> 49.9k; footprint (none) -> Resistor_SMD:R_0402_1005Metric; Manufacturer (none) -> Stackpole Electronics Inc; Part Number (none) -> RMCF0402FT49K9; Power (none) -> 0.063W; Temp Range (none) -> -55°C +155°C; Tolerance (none) -> 1%
- R53: renamed from R?; value 698k -> 154k
- R54, R57: renamed from R?; value 226k -> 49.9k; footprint (none) -> Resistor_SMD:R_0402_1005Metric; Manufacturer (none) -> Stackpole Electronics Inc; Part Number (none) -> RMCF0402FT49K9; Power (none) -> 0.063W; Temp Range (none) -> -55°C +155°C; Tolerance (none) -> 1%
- R55: renamed from R?; value 576k -> 86.6k
- R56: renamed from R?; value 332k -> 49.9k; footprint (none) -> Resistor_SMD:R_0402_1005Metric; Manufacturer (none) -> Stackpole Electronics Inc; Part Number (none) -> RMCF0402FT49K9; Power (none) -> 0.063W; Temp Range (none) -> -55°C +155°C; Tolerance (none) -> 1%
- R58: renamed from R?; value 619k -> 133k; footprint (none) -> Resistor_SMD:R_0402_1005Metric; Manufacturer (none) -> Stackpole Electronics Inc; Part Number (none) -> RMCF0402FT133K; Power (none) -> 0.063W; Temp Range (none) -> -55°C +155°C; Tolerance (none) -> 1%
- gave numbers to parts that had none: 114
Connections:
- net VBAT_EN is gone; now on net EN_HIGH_POWER: Q3.1 (G), R11.2
- net +19V5: now also D3.2 (A), F4.2; no longer C1.1, C10.2, C11.2, C12.2, C13.2, C15.1, C16.1, C17.1, C18.2, C19.1, C2.1, C22.2, C23.2, C27.2, C28.1, C29.2, C3.2, C31.1, C32.1, C36.2, C37.2, C38.2, C4.1, C5.2, C6.2, C8.2, C9.2, D6.2 (A), J2.4 (Pin_4), J4.2 (Pin_2), J5.1 (Pin_1), J5.11 (Pin_11), J5.12 (Pin_12), J5.21 (Pin_21), J5.29 (Pin_29), J5.3 (Pin_3), J5.30 (Pin_30), J5.5 (Pin_5), J5.7 (Pin_7), J5.9 (Pin_9), J7.1 (Pin_1), J8.3 (Pin_3), J8.5 (Pin_5), Q1.3 (S), Q14.3 (S), Q2.3 (S), Q3.3 (S), Q6.3 (S), Q7.3 (S), Q8.3 (S), Q9.3 (S), R1.1, R11.1, R14.2, R18.2, R20.1, R3.1, R32.1, R33.1, R34.1, R35.1, R37.1, R45.2, R46.2, R49.1, R52.1, R54.1, R56.1, R58.1, R8.1, R9.1, U1.1 (GND), U1.2 (GND), U1.EPAD, U2.1 (GND), U2.2 (GND), U2.EPAD, U3.12 (GND), U4.23 (VSS_1), U4.35 (VSS_2), U4.47 (VSS_3), U4.8 (VSSA), U5.4 (GND), U5.7 (PGND)
- net +3V3: now also C?.2, R5.1, U?.5 (OUT)
- net +3V5: now also C?.2, U?.1 (IN), U?.3 (EN)
- net +5V1: now also J5.12 (Pin_12), C?.1, C?.1, C?.1, F2.2, F3.1, L?.2, R?.2, R?.2
- net CELL_1S: now also F8.1
- net CELL_1S_ADC: now also C41.1
- net CELL_2S: now also F7.1
- net CELL_2S_ADC: now also C40.1
- net CELL_3S: now also F6.1
- net CELL_3S_ADC: now also C39.1
- net DRV_PIEZO_RHS: now also J3.2 (Pin_2)
- net PWM_LED_REAR1: now also J6.9 (Pin_9)
- net PWM_LED_REAR2: now also J6.10 (Pin_10)
- net PWM_LED_RHS: now also J3.5 (Pin_5)
- net SPR_PB9: now also J5.16 (Pin_16); no longer J5.14 (Pin_14)
- net VBAT: now also F1.1, Q?.2 (D), U?.1 (VIN)
- net VDC: now also D3.1 (K)
- net VPIEZO: now also J3.1 (Pin_1)
- net VSYS: now also C?.1, D?.1 (K), Q?.3 (S), U?.6 (SENSE)
- net VSYS_SW: now also C?.1, C?.1, C?.1, C?.1, C?.1, J3.3 (Pin_3), J6.5 (Pin_5), Q?.2 (D), U?.1 (VCC); no longer Q4.2 (D)
- net at J7.4 (Pin_4): now also F6.2
- net at C35.2, R47.2, U5.5 (FB): now also R48.2
- net at J7.2 (Pin_2): now also F8.2
- net at U5.6 (COMP): now also C?.2
- net at J7.3 (Pin_3): now also F7.2
- net at U3.5 (CCI): now also C?.2
- net at R46.1: now also C?.1
- net VDC_METERED: now reaches Q5.3 (S), R27.2, R28.1
- net VDC_METERED: now also D?.2 (A)
- net at J4.1 (Pin_1): now also F1.2
- net EN_5V1 renamed EN_HIGH_POWER
- net SPR_PC13: no longer names the net of U4.2 (PC13_WKUP2)
- net SPR_PC13: now also C30.2, R30.2; no longer J5.16 (Pin_16)
- new net: J6.12 (Pin_12), R5.2
- new net: Q?.2 (D), Q?.2 (D)
- new net: C?.2, R?.1, R?.2, U?.3 (FB)
- new net: D?.2 (A), Q?.1 (G), R?.1, R?.2
- new net: C?.2, L?.1, Q?.2 (D), Q?.3 (S), R?.1, U?.6 (VSW)
- new net: D?.1 (K), R?.2, U?.7 (HSDR)
- new net: C?.1, R?.1
- new net: C?.1, R?.2, U?.2 (COMP)
- new net: C?.2, R?.1
- new net: Q?.1 (G), R?.2, U?.5 (LSDR)
- new net: R?.2, U?.3 (CTL)
- new net: Q?.1 (G), U?.5 (GATE)
- new net: C?.1, U?.8 (BST)
- new net 5V1_PHONE: F3.2, J6.2 (Pin_2)
- new net 5V1_REAR: F2.1, J6.1 (Pin_1)
- new net ACDC_IN: F4.1, J6.6 (Pin_6)
- new net BUTTON: J6.11 (Pin_11), R30.1, R31.2
- new net GND: C1.1, C10.2, C11.2, C12.2, C13.2, C15.1, C16.1, C17.1, C18.2, C19.1, C2.1, C22.2, C23.2, C27.2, C28.1, C29.2, C3.2, C30.1, C31.1, C32.1, C36.2, C37.2, C38.2, C39.2, C4.1, C40.2, C41.2, C5.2, C6.2, C8.2, C9.2, C?.1, C?.1, C?.1, C?.1, C?.2, C?.2, C?.2, C?.2, C?.2, C?.2, C?.2, C?.2, C?.2, C?.2, D6.2 (A), J2.4 (Pin_4), J3.4 (Pin_4), J4.2 (Pin_2), J5.1 (Pin_1), J5.11 (Pin_11), J5.21 (Pin_21), J5.29 (Pin_29), J5.3 (Pin_3), J5.30 (Pin_30), J5.5 (Pin_5), J5.7 (Pin_7), J5.9 (Pin_9), J6.3 (Pin_3), J6.4 (Pin_4), J6.7 (Pin_7), J6.8 (Pin_8), J7.1 (Pin_1), J8.3 (Pin_3), J8.5 (Pin_5), Q1.3 (S), Q14.3 (S), Q2.3 (S), Q3.3 (S), Q6.3 (S), Q7.3 (S), Q8.3 (S), Q9.3 (S), Q?.3 (S), R1.1, R11.1, R14.2, R18.2, R20.1, R3.1, R31.1, R32.1, R33.1, R34.1, R35.1, R37.1, R45.2, R46.2, R48.1, R49.1, R52.1, R54.1, R56.1, R58.1, R8.1, R9.1, R?.1, R?.1, R?.1, U1.1 (GND), U1.2 (GND), U1.EPAD, U2.1 (GND), U2.2 (GND), U2.EPAD, U3.12 (GND), U4.23 (VSS_1), U4.35 (VSS_2), U4.47 (VSS_3), U4.8 (VSSA), U5.4 (GND), U5.7 (PGND), U?.2 (GND), U?.2 (GND), U?.4 (GND)
- no-connect marks 2 -> 4
Other:
- note added: "4.2V"
- note added: "Alternatively remove these fuses and get current limiting buck"
- note added: "C_{OUT}>4.2(1+16.8/18.5)/((16.8)(300k)(62.6m))=25.4uF R_{ESR}<0.0626*12/4.2=0.179OHms"
- note added: "Current limiter"
- note added: "D_{MIN}~=5.1V/19V=0.268 D_{MAX}~=5.1V/12V=0.425"
- note added: "Front LED Driver"
- note added: "Keep divider above (n/4)*200k to reduce effect of R_{ds} and reduce power draw"
- note added: "L=V_{OUT}(1-D)/[(I_{OUT})(ra)(f_{SW})] =5.1(1-0.268)/[(10)(0.2)(600e3)] =3.11uH~=3.3uH ra=V_{OUT}(1-D)/[(I_{OUT})(L)(f_{SW})] ra_{MAX}=5.1(1-0.268)/[(10)(3.3e-6)(600e3)]=0.189 ra_{MIN}=5.1(1-0.425)/[(10)(3.3e-6)(600e3)]=0.148"
- note added: "Max LED power: (3.5V*3*0.25A*4+10W)=21W Max 5.1V power: 10A*5.1V/0.9=57W Max LED VSYS current: 21W/13.2V=1.6A Max VBAT current: (21W+57W)/13.2V=5.9A Min AC/DC current rating: (21W+57W)/18.5V=4.2A"
- note added: "NOTE CAPCITOR VOLTAGE RATINGS"
- note added: "Normal fuses have undesirable Vf Poly fuses are less temperature stable"
- note added: "R_{TH}=(R_{1}//R_{2}) R_{TH(MAX)}=42.7k"
- note added: "TO DO ------------------------------------ / Decide if/how to do low-batt shutdown/ship-mode / Decide how to handle power ORing / Crystals / JTAG conn, USB conn / Select passive component values / Select passive component values for LP LED bucks / Map MCU inputs (need dividers for ADC) / Select LP LDO - Select HP buck regulator - Select remaining passive component values - Select passive componen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"
- note added: "T_{RC}=(R1//R2)*C C<(1/42.7k)=23.4uF"
- note added: "Use murata or TDK for capacitors Beware of DC bias"
- note added: "V_{OUT}=0.8[(R_{1}+R_{2})/R_{2}] =0.8*[(453k+133k)/133k]=3.525V"
- note added: "f_{SW}=600kHz"
- note added: "ra=I_{RPL}/I_{OUT}=0.2 [0.1<ra<0.4]"
- note removed: "---> LDO --->"
- note removed: "--> BUCK -->"
- note removed: "AC/DC Adapter"
- note removed: "Batt "diode" Vf should be < 0.1V @ 5A (0.5W)"
- note removed: "Can use "ideal diode" or "power oring" IC to replace VBAT diode with MOSFET"
- note removed: "ESR < 1R"
- note removed: "LHS"
- note removed: "Lighting"
- note removed: "R_{TH}=(R_{1}//R_{2}) R_{TH(MAX)}=211k"
- note removed: "TO DO ------------------------------------ / Decide if/how to do low-batt shutdown/ship-mode / Decide how to handle power ORing / Crystals - JTAG conn, USB conn - Select passive component values - Select passive component values for LP LED bucks - Map MCU inputs (need dividers for ADC) - Select LP LDO - Select HP buck regulator - Select remaining passive component values - Select passive componen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"
- note removed: "T_{RC}=(R1//R2)*C C<(0.1/211k)=474nF"
- note removed: "VDC_METERED"
- note removed: "V_{OUT}=0.8[(R_{1}+R_{2})/R_{2}] =0.8[(383k+113k)/113k]=3.512V"
- note removed: "WAKE"
- note removed: "t_{ON}=[L(0.26)(I_{LED})]/[V_{IN}-V_{LED}-I_{LED}(R_{SET}+R_{L}+R_{SW})] =[47uH(0.26)(1A)]/[16V-9.6V-1A(0.1+0.1+0.2)Ohms] =2.0366uS"
- moved on the sheet: C1, C38, D1, F5, J1, J4, J5, J7, J8, J9, L1, Q1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

Commit message: Commit before 5V buck change
Parts:
- removed C? (x5): ?????, symbol Device:C_Small
- removed C? (x2): ?????, symbol Device:C_Polarized_Small
- removed R?: ????, symbol Device:R_Small
- added C? (x4): 22uF, symbol Device:C_Small
- added C?: DNP, symbol Device:C_Small
- added C? (x2): 470uF, symbol Device:C_Polarized_Small
- added C?: 8.2nF, symbol Device:C_Small
- added C?: DNP, symbol Device:C_Polarized_Small
- added C?: ?????, symbol Device:C_Small
- added Q?: Q_PMOS_GDS, symbol Device:Q_PMOS_GDS
- added Q?: Q_NMOS_GDS, symbol Device:Q_NMOS_GDS
- added R? (x2): 100k, symbol Device:R_Small
- added R?: 0R, symbol Device:R_Small
- added R?: ????, symbol Device:R_Small
- added R?: 4.75k, symbol Device:R_Small
- added R?: DNP, symbol Device:R_Small
- C30: value DNP -> 100nF
- C?: value ????? -> 22uF
- C?: value ????? -> 33pF
- C?: value ????? -> 470uF
- C?: value ????? -> 1.8nF
- R30: value DNP -> 0R
- R?: value ???? -> 7.5k
- R?: value ???? -> 2.49k
- R? (x2): value ???? -> 1k
- R?: value ???? -> 22.1k
- R?: value ???? -> 8.06
Connections:
- net +5V1: now also C?.1, C?.1, C?.1, C?.1, C?.1
- net EN_HIGH_POWER: now also Q?.1 (G), R?.2
- net GND: now also C?.2, C?.2, C?.2, C?.2, C?.2, C?.2, C?.2, C?.2, Q?.3 (S), R?.1, R?.1; no longer C?.2
- net VSYS: now also C?.1, Q?.3 (S), R?.2
- net VSYS_SW: now also C?.1, C?.1, C?.1
- net at C?.2, R?.1, R?.2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: now also R?.1
- net at C?.1, U?.2 (COMP): now also C?.2
- new net: Q?.2 (D), R?.1, R?.1
- new net: C?.2, R?.1, R?.2, R?.2
- new net: C?.2, Q?.1 (G), R?.2
- new net: C?.1, R?.2
Other:
- note added: "Derate polyfuses for 0-60C"
- note added: "Do not use tantalum due to high dI/dt"
- note added: "Get some 20W resistors for load testing"
- note added: "I_{COUT-RMS}=I_{OUT}(ra)/sqrt(12) =10(0.189)/sqrt(12)=0.546A V_{ESR-COUT}=I_{OUT}(ra)[ESR_{COUT}+1/((8)(f_{SW})(C_{OUT}))] V_{ESL-ON}=(ESL_{COUT})(I_{PP})(f_{SW})/D V_{ESL-OFF}=(ESL_{COUT})(I_{PP})(f_{SW})/(1-D) V_{TRAN-OUT-ESR}=I_{TRAN}(ESR_{COUT}) V_{TRAN-OUT-DISCHG}=[(I_{TRAN}^2)(L_{OUT})]/[(C_{OUT})(V_{IN}-V_{OUT})] V_{TRAN-OUT-CHG}=[(I_{TRAN}^2)(L_{OUT})]/[(C_{OUT})(V_{OUT})]"
- note added: "I_{RMS-CTRL}=I_{OUT}[sqrt(D(1+(ra^2)/12))] =10[sqrt(0.425(1+(0.148^2)/12))] =6.525A P_{COND}=(I_{RMS-CTRL}^2)(R_DS-ON-CTRL) t_{ON}= P_{SW}=0.5(I_{OUT})(V_{IN})(f_{SW})(t_{ON}+t_{OFF}) P_{D-CTRL}=P_{COND}+P_{SW-TOT}"
- note added: "I_{RMS}=I_{OUT}[sqrt(1+(ra^2)/12] =10[sqrt(1+(0.189^2)/12]=10.015A I_{PK}=I_{OUT}(1+ra/2) =10(1+0.189/2)=10.945A SR_{LOUT}=(V_{IN}-V_{OUT})/L_{OUT} =(12-5.1)/3.3e-6=2.091A/uS I_{PP}=V_{OUT}(1-D)/[(L_{OUT})(f_{SW})] =5.1(1-0.268)/[(3.3e-6)(600e3)]=1.885A"
- note added: "LP_{CU}=(I_{RMS}^2)(DCR) I_{IN-RMS}=I_{OUT}[sqrt(D(1-D))] =10[sqrt(0.425(1-0.425))]=4.94A P_{CIN}=ESR_{CIN}(I_{IN-RMS}^2) I_{INRUSH}=(C_{OUT})(V_{OUT})/t_{ss}"
- note added: "slew rate limit?"
- moved on the sheet: C?

Commit message: New buck controller WIP
Parts:
- removed C? (x5): 22uF, symbol Device:C_Small
- removed C?: DNP, symbol Device:C_Small
- removed C? (x3): 470uF, symbol Device:C_Polarized_Small
- removed C?: 8.2nF, symbol Device:C_Small
- removed C?: 33pF, symbol Device:C_Small
- removed C?: DNP, symbol Device:C_Polarized_Small
- removed C?: 1.8nF, symbol Device:C_Small
- removed C?: 100nF, symbol Device:C_Small
- removed D?: D_Schottky_Small, symbol Device:D_Schottky_Small
- removed L?: 3.3uH, symbol Device:L_Small
- removed Q? (x2): Q_NMOS_GDS, symbol Device:Q_NMOS_GDS
- removed R?: 7.5k, symbol Device:R_Small
- removed R?: 2.49k, symbol Device:R_Small
- removed R?: 0R, symbol Device:R_Small
- removed R?: 4.75k, symbol Device:R_Small
- removed R?: DNP, symbol Device:R_Small
- removed R? (x2): 1k, symbol Device:R_Small
- removed R?: 22.1k, symbol Device:R_Small
- removed R?: 8.06, symbol Device:R_Small
- removed U?: NCP3020BDR2G, symbol JetkovKiCADLib:NCP3020BDR2G
- added C? (x4): 10uF, symbol Device:C_Small
- added C? (x2): ?????, symbol Device:C_Small
- added C? (x4): 47uF, symbol Device:C_Small
- added C? (x2): DNP, symbol Device:C_Polarized_Small
- added C?: 51pF, symbol Device:C_Small
- added C?: 510pF, symbol Device:C_Small
- added C?: 1uF, symbol Device:C_Small
- added C? (x2): 100nF, symbol Device:C_Small
- added L?: 2.0uH, symbol Device:L_Small
- added Q? (x2): Q_NMOS_GDS, symbol Device:Q_NMOS_GDS
- added R?: 27.4k, symbol Device:R_Small
- added R? (x2): ????, symbol Device:R_Small
- added R?: 0R, symbol Device:R_Small
- added R?: 15k, symbol Device:R_Small
- added R?: 78.8, symbol Device:R_Small
- added U?: NCP164ASN330T1G, JetkovKiCADLib:SOT-23-5_TSOP−5_ON, symbol JetkovKiCADLib:NCP164ASN330T1G
- added U?: ADP1883ARMZ-0.6-R7, symbol JetkovKiCADLib:ADP1883ARMZ-0.6-R7
Connections:
- net +3V5: now also C?.2, U?.1 (IN)
- net +5V1: now also C?.1, C?.1, C?.1, C?.1, C?.1, L?.2, R?.2
- net EN_HIGH_POWER: now also U?.3 (EN)
- net GND: now also C?.1, C?.1, C?.1, C?.1, C?.1, C?.1, C?.1, C?.1, C?.2, C?.2, C?.2, C?.2, C?.2, C?.2, C?.2, Q?.3 (S), R?.1, R?.1, R?.1, U?.2 (GND), U?.4 (GND), U?.7 (PGND)
- net VSYS_SW: now also C?.1, C?.2, C?.2, C?.2, C?.2, Q?.2 (D), U?.1 (VIN)
- new net: Q?.1 (G), R?.1
- new net: C?.2, L?.1, Q?.2 (D), Q?.3 (S), R?.2, U?.9 (SW)
- new net: C?.1, C?.2, U?.2 (COMP/EN)
- new net: C?.2, R?.2
- new net: C?.2, C?.2, U?.5 (OUT), U?.5 (VDD)
- new net: Q?.1 (G), R?.2, U?.6 (DRVL)
- new net: C?.1, R?.1
- new net: R?.2, U?.8 (DRVH)
- new net: R?.1, R?.2, U?.3 (FB)
- new net: C?.1, U?.10 (BST)
- no-connect marks 4 -> 5
Other:
- note added: "VDD_5V1_BUCK"
- note removed: "D_{MIN}~=5.1V/19V=0.268 D_{MAX}~=5.1V/12V=0.425"
- note removed: "Do not use tantalum due to high dI/dt"
- note removed: "I_{COUT-RMS}=I_{OUT}(ra)/sqrt(12) =10(0.189)/sqrt(12)=0.546A V_{ESR-COUT}=I_{OUT}(ra)[ESR_{COUT}+1/((8)(f_{SW})(C_{OUT}))] V_{ESL-ON}=(ESL_{COUT})(I_{PP})(f_{SW})/D V_{ESL-OFF}=(ESL_{COUT})(I_{PP})(f_{SW})/(1-D) V_{TRAN-OUT-ESR}=I_{TRAN}(ESR_{COUT}) V_{TRAN-OUT-DISCHG}=[(I_{TRAN}^2)(L_{OUT})]/[(C_{OUT})(V_{IN}-V_{OUT})] V_{TRAN-OUT-CHG}=[(I_{TRAN}^2)(L_{OUT})]/[(C_{OUT})(V_{OUT})]"
- note removed: "I_{RMS-CTRL}=I_{OUT}[sqrt(D(1+(ra^2)/12))] =10[sqrt(0.425(1+(0.148^2)/12))] =6.525A P_{COND}=(I_{RMS-CTRL}^2)(R_DS-ON-CTRL) t_{ON}= P_{SW}=0.5(I_{OUT})(V_{IN})(f_{SW})(t_{ON}+t_{OFF}) P_{D-CTRL}=P_{COND}+P_{SW-TOT}"
- note removed: "I_{RMS}=I_{OUT}[sqrt(1+(ra^2)/12] =10[sqrt(1+(0.189^2)/12]=10.015A I_{PK}=I_{OUT}(1+ra/2) =10(1+0.189/2)=10.945A SR_{LOUT}=(V_{IN}-V_{OUT})/L_{OUT} =(12-5.1)/3.3e-6=2.091A/uS I_{PP}=V_{OUT}(1-D)/[(L_{OUT})(f_{SW})] =5.1(1-0.268)/[(3.3e-6)(600e3)]=1.885A"
- note removed: "L=V_{OUT}(1-D)/[(I_{OUT})(ra)(f_{SW})] =5.1(1-0.268)/[(10)(0.2)(600e3)] =3.11uH~=3.3uH ra=V_{OUT}(1-D)/[(I_{OUT})(L)(f_{SW})] ra_{MAX}=5.1(1-0.268)/[(10)(3.3e-6)(600e3)]=0.189 ra_{MIN}=5.1(1-0.425)/[(10)(3.3e-6)(600e3)]=0.148"
- note removed: "LP_{CU}=(I_{RMS}^2)(DCR) I_{IN-RMS}=I_{OUT}[sqrt(D(1-D))] =10[sqrt(0.425(1-0.425))]=4.94A P_{CIN}=ESR_{CIN}(I_{IN-RMS}^2) I_{INRUSH}=(C_{OUT})(V_{OUT})/t_{ss}"
- note removed: "f_{SW}=600kHz"
- note removed: "ra=I_{RPL}/I_{OUT}=0.2 [0.1<ra<0.4]"

Commit message: HP buck WIP
Parts:
- removed C?: ?????, symbol Device:C_Small
- removed U?: NCP164ASN330T1G, JetkovKiCADLib:SOT-23-5_TSOP−5_ON, symbol JetkovKiCADLib:NCP164ASN330T1G
- C? (x2): value ????? -> 1uF
- C?: value ????? -> 1.5nF
- R?: value 78.8 -> 80.6k
- R?: value ???? -> 2R
Connections:
- no-connect marks 5 -> 4
Other:
- note added: "170mV dropout max @ 3.3V/300mA"
- note added: "Duty Cycle --------- D_{MIN}=5.1/19=0.268 D_{MAX}=5.1/12=0.425 MOSFET Channel Conduction Loss ------------------------------- P_{N1,N2(CL)}=[D(R_{ON-UPPER})+(1-D)R_{ON-LOWER)}]I_{LOAD}^2 =[0.32(R_{ON-UPPER})+(1-0.32)R_{ON-LOWER}]10^2 MOSFET Driver Loss ------------------------------- P_{DR(LOSS)}=V_{DR}[(f_{SW})(C_{G-UPPER})(V_{DR})+I_{BIAS}]+V_{DD}[(f_{SW})(C_{G-LOWER})(V_{DD})+I_{BIAS}] =V_{DR}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"
- note added: "I_{VC-LIM}=I_{LOAD}(1-K_{I}) I_{VC-LIM}=1.5V/((A_{CS})(R_{ON}))"
- note added: "If there's space, double the MOSFET footprints"
- note added: "R_{T}=R_{B}(V_{OUT}-0.8V)/0.8V =15e3(5.1-0.8)/0.8 =80.625k~=80.6k"
- note added: "V_{DD}>=V_{IN}/8+1.5=20/8+1.5=4V V_{DD}>=V_{OuT}/4=5.1/4=1.275V"
- note added: "change to > 4V"
- note added: "dI_{L}=K_{I}(I_{LOAD}) ~=0.33(10)=3.3A L=[(V_{IN}-V_{OUT})/((dI_{L})(f_{SW}))][V_{OUT}/V_{IN}] =[(16-5.1)/((3.3)(600e3))][5.1/16]=1.755uH dI_{L}=[(16-5.1)/((2e-6)(600e3))][5.1/16]=2.895A K_{I}=2.895/10=0.29 dI_{L-MIN}=[(12-5.1)/((2e-6)(600e3))][5.1/12]=2.444A dI_{L-MAX}=[(19-5.1)/((2e-6)(600e3))][5.1/19]=3.109A I_{SAT}>16A"
- note added: "dV_{RR}=(0.01)*V_{OUT}=(0.01*5.1=0.051V C_{OUT}=dI_{L}/[(8)(f_{SW})(dV_{RR}-(dI_{L})(ESR))] =2.895/[(8)(600e3)(0.051-(2.895)(0.015))]=80uF C_{OUT}=[2(dI_{L})]/[(f_{SW})(V_{DROOP}-(I_{LOAD-STEP})(ESR))] =[2(2.895)]/[(600e3)(0.1-(3)(0.015))]=175uF"
- note added: "f_{CROSS}=f_{SW}/12=600e3/12=50kHz f_{ZERO}=f_{CROSS}/4=12.5kHz R_{COMP}=[(f_{CROSS}/(F_{CROSS}+F_{ZERO})][2(pi)(f_{CROSS})(C_{OUT})/((G_{M})(A_{CS}))][V_{OUT}/V_{REF}] =[50e3/(50e3+12.5e3)][(2)(pi)(50e3)(C_{OUT})/((500e-6)(A_{CS})][V_{OUT}/0.8] =[(C_{OUT})(V_{OUT})/(A_{CS})][628318530.718] =[(4*47e-6*0.67)(5.1)/13.4][628318530.718] =30.12kOhms C_{COMP}=1/[2(pi)(R_{COMP})(f_{ZERO})] =1/[2(pi)(27.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"
- note removed: "VDD_5V1_BUCK"
