File: faclon-main/FalconMain/FalconMain.kicad_sch (KiCad schematic)
At the start: 199 parts, among them J1 Nano-Fit, J2 Nano-Fit, J3 Nano-Fit, J4 PTH, J5 100mil, J6 Nano-Fit, J7 JST-XH, J8 100mil, J9 100mil, Q1 Q_NMOS_GDS, Q10 Q_PMOS_GDS, Q11 Q_PMOS_GDS, Q12 Q_PMOS_GDS, Q13 Q_PMOS_GDS, Q14 Q_NMOS_GDS, Q15 Q_PMOS_GDS, Q16 Q_PMOS_GDS, Q17 Q_PMOS_GDS, Q18 Q_PMOS_GDS, Q2 Q_NMOS_GDS, Q3 Q_NMOS_GDS, Q4 Q_PMOS_GDS, Q5 Q_PMOS_GDS, Q6 Q_NMOS_GDS, Q7 Q_NMOS_GDS, Q8 Q_NMOS_GDS, Q9 Q_NMOS_GDS, U1 AL8843QSP-13, U2 AL8843QSP-13, U3 MAX1873TEEE+, U4 STM32L152CBT6, U5 BD9E104FJ-E2, Y1 8MHz, Y2 32.768kHz

Commit message: Schematic organization WIP
Parts:
- removed C30: 100nF, symbol Device:C_Small
- removed C? (x3): 47uF, symbol Device:C_Small
- removed C? (x3): 10uF, symbol Device:C_Small
- removed C?: 1uF, symbol Device:C_Small
- removed Q14, Q3, Q? (x2): Q_NMOS_GDS, symbol Device:Q_NMOS_GDS
- removed Q15, Q16, Q17, Q4, Q?: Q_PMOS_GDS, symbol Device:Q_PMOS_GDS
- removed R10, R11, R49: 100k, symbol Device:R_Small
- added C40: 1uF, symbol Device:C_Small
- added C? (x3): 10uF, symbol Device:C_Small
- added C? (x3): 47uF, Capacitor_SMD:C_1210_3225Metric, symbol Device:C_Small
- added C?: 100nF, symbol Device:C_Small
- added L?: R0, symbol Device:L_Ferrite_Small
- added Q? (x4): Q_PMOS_GDS, symbol Device:Q_PMOS_GDS
- added Q?: Q_NMOS_GDS, symbol Device:Q_NMOS_GDS
- added R?: 100k, symbol Device:R_Small
- C49: renamed from C?; Manufacturer (none) -> TDK Corporation; Part Number (none) -> CGA6P3X7S1H106K250AB; Temp Range (none) -> -55°C +125°C; Tolerance (none) -> 10%; Voltage (none) -> 50V
- C56: renamed from C?; footprint (none) -> Capacitor_SMD:C_1210_3225Metric; Manufacturer (none) -> Murata Electronics; Part Number (none) -> GRM32EC81C476KE15K; Temp Range (none) -> -55°C +105°C; Tolerance (none) -> 10%; Voltage (none) -> 16V
- Q25, Q26: renamed from Q?; Part Number (none) -> PSMN4R1-30YLC,115
- R65: renamed from R?; value ???? -> 100k
- gave numbers to parts that had none: 30
- renumbered C9 to C10, C10 to C11, C11 to C12, C12 to C13, C13 to C14, C15 to C16, C16 to C17, C17 to C18, C18 to C19, C19 to C20, C20 to C21, C21 to C22, C22 to C23, C23 to C24, C24 to C25, C25 to C26, C31 to C32, C32 to C33, C33 to C34, C35 to C36, C36 to C37, C37 to C38, C3 to C4, C38 to C41, C39 to C42, C40 to C43, C41 to C44, C4 to C5, C5 to C6, C6 to C7, C7 to C8, C8 to C9, D6 to D5, D8 to D7, D9 to D8, Q7 to Q10, Q8 to Q11, Q9 to Q12, Q10 to Q13, Q11 to Q14, Q12 to Q15, Q13 to Q16, Q18 to Q22, Q5 to Q7, Q6 to Q9, R14 to R17, R15 to R18, R16 to R19, R17 to R20, R18 to R21, R19 to R22, R20 to R23, R21 to R24, R22 to R25, R23 to R26, R24 to R27, R25 to R28, R26 to R29, R27 to R30, R28 to R31, R29 to R32, R30 to R34, R31 to R35, R32 to R36, R33 to R37, R34 to R38, R35 to R39, R36 to R40, R37 to R41, R38 to R42, R39 to R43, R40 to R44, R41 to R45, R42 to R46, R43 to R47, R44 to R48, R45 to R49, R46 to R50, R47 to R51, R48 to R52, R50 to R54, R51 to R55, R52 to R56, R53 to R57, R54 to R58, R55 to R59, R56 to R60, R57 to R61, R58 to R62, U5 to U6
Connections:
- net +3V3: now also U4.29 (PA8), Q?.1 (G), R?.2
- net +5V1: now also C?.1, C?.1, C?.1
- net CELL_2S: now also Q?.3 (S)
- net CELL_3S: now also Q?.3 (S)
- net CELL_4S: now also Q?.3 (S)
- net GND: now also C40.2, C?.1, C?.1, C?.1, C?.2, C?.2, C?.2, C?.2, Q?.3 (S), R?.1
- net VSYS_SW: now also Q6.2 (D), C?.2, C?.2, C?.2
- net at R34.2, U4.2 (PC13_WKUP2): now also C?.1
- net at Q22.1 (G), R54.1: now also Q?.1 (G), Q?.1 (G), Q?.1 (G), Q?.2 (D)
- net at R59.2: now also Q?.2 (D)
- net at C39.2, U8.5 (VDD): now also C40.1, L?.2
- net at R57.2: now also Q?.2 (D)
- net at R55.2: now also Q?.2 (D)
- net at C3.2, Q6.1 (G), R16.2: now also Q?.1 (G)
- net SPR_PA8: no longer names the net of J5.13 (Pin_13)
- net SPR_PA8: no longer U4.29 (PA8)
- new net +4V: Q?.3 (S)
- new net +4V_SW: L?.1, Q?.2 (D)
- no-connect marks 4 -> 5
Other:
- note added: "12-19.5V/0.7A to 4V/0.2A Buck Regulator"
- note added: "12-19.5V/4.7A to 5.1V/10A Buck Regulator"
- note added: "170mV dropout @ 3.3V/300mA"
- note added: "19.5V supply enables power to the MCU. MCU should maintain 4V_EN high"
- note added: "4V to 3.3V LDO"
- note added: "AC/DC Adapter Current Limiting -------------------- I_{IN(MAX)}=0.1V/R_{CSS} =0.1V/22.6mOhms =4.43A"
- note added: "AC/DC and Battery Power OR-ing"
- note added: "Accounting for DC bias: C_{OUT}=47*(1-0.424)*4=108uF"
- note added: "BATTERY BALANCING"
- note added: "BATTERY CHARGING"
- note added: "Cell Voltage Cutoff Set -------------------- V_{VADJ}=9.5(V_{CELL})-9(V_{REF}) =9.5(4.1V)-9(4.2V)=1.15V R_{2}=R_{1}[V_{VADJ}/(V_{REF}-V_{VADJ})] =133k*(1.15/(4.2-1.15)~=49.9k V_{VADJ}=1.14587V V_{CELL}=(1.14587V+9(4.2V))/9.5=4.0996V"
- note added: "Charge Current Sense Output -------------------- V_{Iout}=20(R_{CSB} * I_{chg}) C_{load} < 5nF Charge Current Set -------------------- V_{ICH-EN}=I_{CHG} * 1.3146"
- note added: "Check MOSFET pins numbers!"
- note added: "Duty Cycle --------- D_{MIN}=5.1/19=0.268 D_{MAX}=5.1/12=0.425"
- note added: "Enable 4V_SW with VSYS_SW to power the 5.1V buck regulator LV circuits"
- note added: "HIGH POWER 5.1V REGULATION"
- note added: "HIGH POWER SWITCH"
- note added: "LOW POWER 4V AND 3.3V REGULATION"
- note added: "LV PMOS will turn on later, and turn off earlier, than HV"
- note added: "Li-ion 4S Charge Regulator Controller"
- note added: "Li-ion Cell Balancing FETs"
- note added: "Li-ion Cell Voltage Sensing"
- note added: "Loop Compensation ---------------- f_{CROSS}=f_{SW}/12=600e3/12=50kHz f_{ZERO}=f_{CROSS}/4=12.5kHz R_{COMP}=[(f_{CROSS}/(F_{CROSS}+F_{ZERO})][2(pi)(f_{CROSS})(C_{OUT})/((G_{M})(A_{CS}))][V_{OUT}/V_{REF}] =[50e3/(50e3+12.5e3)][(2)(pi)(50e3)(C_{OUT})/((500e-6)(A_{CS})][V_{OUT}/0.8] =[(C_{OUT})(V_{OUT})/(A_{CS})][628318530.718] =[(108e-6)(5.1)/13.4][628318530.718] =25.83kOhms~=26.1kOhms -> 27.4kOhms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"
- note added: "Loop Compensation ------------------------ R_{4}=[(2pi)(V_{OUT})(f_{CRS})(C_{OUT})]/[(V_{FB})(G_{MP})(G_{MA})] =[(2pi)(V_{OUT})(f_{CRS})(C_{OUT})]/[(0.8V)(7A/V)(82uA/V)] =13682.8948(V_{OUT})(f_{CRS})(C_{OUT}) =13682.8948(3.5)(40k)(20u) =38.312kOhms~=38.3kOhms C_{4}=1/[(2pi)(R_{4})(f_{CRS}/6)] =1/[(2pi)(3.83k)(40k/6) =623.32pF~=620pF"
- note added: "MICROCONTROLLER"
- note added: "MOSFET Channel Conduction Loss --------------------- P_{N1,N2(CL)}=[D(R_{ON-UPPER})+(1-D)R_{ON-LOWER)}]I_{LOAD}^2 =[0.32(5e-3)+(1-0.32)(5e-3)]10^2 =0.16+0.34=0.5W MOSFET Driver Loss --------------------- V_{DR}=V_{DD}-V_{F(RECT)}=4-0.320=3.68V P_{DR(LOSS)}=V_{DR}[(f_{SW})(C_{G-UPPER})(V_{DR})+I_{BIAS}]+V_{DD}[(f_{SW})(C_{G-LOWER})(V_{DD})+I_{BIAS}] =3.68[(600e3)(2.5e-9)(3.68)+2e-3]+4[(600e3)(2.5e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"
- note added: "MOSFET PSMN4R1-30YLC -------------------- R_{DS(ON)@4V}=5mOhms V_{f(DIODE)@10A}=0.75V Q_{G(TOT)@4V}=10nC C_{G(TOT)@4V)=10nC/4V=2.5nF C_{iss}=1.5nF R_{G}=1.9Ohms"
- note added: "Max Charge Current Set -------------------- R_{CSB}=0.2V(V_{ICH-EN}/V_{REF})/I_{CHG} =0.2V(3.3V/4.2V)/2.5A ~=62.6mOhms I_{CHG}=0.2V(3.3V/4.2V)/0.0626R=2.5103A"
- note added: "Maximum Inductor Ripple Current -------------------------------- dI_{L}=K_{I}(I_{LOAD}) ~=0.33(10)=3.3A Minimum Inductance -------------------------------- L=[(V_{IN}-V_{OUT})/((dI_{L})(f_{SW}))][V_{OUT}/V_{IN}] =[(16-5.1)/((3.3)(600e3))][5.1/16]=1.755uH Inductor Ripple Current with Selected Inductance -------------------------------- dI_{L}=[(16-5.1)/((2e-6)(600e3))][5.1/16]=2.895A K_{I}=2.895/1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"
- note added: "Minimum Inductance -------------------- L>{V_{BATT}[V_{DCIN(MAX)}-V_{BATT}]}/{[V_{DCIN(MAX)}][f_{SW}][I_{CHG}][LIR]} >((14.8V)(19.5V-14.8V))/((19.5V)(300kHz)(2.5A)(0.3)) >15.85uH"
- note added: "Minimum Input Capacitance -------------------- V_{CIN-MAX-RPL}=0.01(V_{IN-MIN})+([I_{LOAD-MAX})(ESR_{CIN}) =0.01(12)-(10)(0.001)=110mV C_{IN-MIN}=[I_{LOAD-MAX}/V_{MAX-RPL}][D(1-D)/f_{SW}] =[10/0.11][0.425(1-0.425)/600e3]=37uF Minimum Output Capacitance ------------------------- dV_{OUTRR}=(0.01)V_{OUT}=(0.01)5.1=0.051V C_{OUT}>dI_{L}/[(8)(f_{SW})(dV_{OUTRR}-(dI_{L})(ESR_{COUT}))] >2.895/[(8)(600e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"
- note added: "Minimum Output Capacitance -------------------- C_{OUT}>4.2(1+16.8/18.5)/((16.8)(300k)(62.6m))=25.4uF R_{ESR}<0.0626*12/4.2=179mOhms"
- note added: "ON-BOARD LOAD DRIVERS"
- note added: "Output Voltage Set ----------- R_{T}=R_{B}(V_{OUT}-0.8V)/0.8V =15e3(5.1-0.8)/0.8 =80.625k~=80.6k"
- note added: "Output Voltage Set ------------------------ V_{OUT}=0.8[(R_{1}+R_{2})/R_{2}] =0.8*[(453k+133k)/133k]=3.525V"
- note added: "Place as close to MOSFETs as possible"
- note added: "Ripple Current at Selected Inductance ------------------------ I_{RPL}=(V_{OUT})(V_{IN}-V_{OUT})/[(V_{IN})(f_{OSC})(L)] =(3.5V)(15V-3.5V)/[(15V)(570kHz)(10uH)] =0.471A Ripple Voltage at Selected Output Capacitance ------------------------ V_{RPL}=I_{RPL}[R_{ESR}+1/(8(C_{OUT})(f_{OSC}))] =(0.471A)[10mOhm+1/(8(20uF)(570kHz))] =9.87mV"
- note added: "STM32L1 MCU"
- note added: "STM32L1 MCU POWER"
- note added: "Use murata or TDK for capacitors Beware of DC bias NOTE CAPCITOR VOLTAGE RATINGS Get some 20W resistors for load testing"
- note added: "V_{DD}>=V_{IN}/8+1.5 =20/8+1.5=4V V_{DD}>=V_{OuT}/4 =5.1/4=1.275V"
- note added: "Valley Current Limiting -------------- I_{VC-LIM}=1.5V/((A_{CS})(R_{ON})) =1.5/((26.7)(5e-3)) =11.23 I_{LOAD-LIM}=I_{VC-LIM}/(1-K_{I}) =11.23/(1-0.29)=15.8A"
- note removed: "170mV dropout max @ 3.3V/300mA"
- note removed: "19.5V supply enables power to the MCU MCU should maintain 3V5_EN high"
- note removed: "C_{4}=1/[(2pi)(R_{4})(f_{CRS}/6)] =1/[(2pi)(3.83k)(40k/6) =623.32pF~=620pF"
- note removed: "C_{OUT}>4.2(1+16.8/18.5)/((16.8)(300k)(62.6m))=25.4uF R_{ESR}<0.0626*12/4.2=0.179OHms"
- note removed: "Duty Cycle --------- D_{MIN}=5.1/19=0.268 D_{MAX}=5.1/12=0.425 MOSFET Channel Conduction Loss ------------------------------- P_{N1,N2(CL)}=[D(R_{ON-UPPER})+(1-D)R_{ON-LOWER)}]I_{LOAD}^2 =[0.32(R_{ON-UPPER})+(1-0.32)R_{ON-LOWER}]10^2 MOSFET Driver Loss ------------------------------- P_{DR(LOSS)}=V_{DR}[(f_{SW})(C_{G-UPPER})(V_{DR})+I_{BIAS}]+V_{DD}[(f_{SW})(C_{G-LOWER})(V_{DD})+I_{BIAS}] =V_{DR}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"
- note removed: "Get some 20W resistors for load testing"
- note removed: "I_{IN(MAX)}=0.1V/R_{CSS} =0.1V/22.6mOhms =4.43A"
- note removed: "I_{RPL}=(V_{OUT})(V_{IN}-V_{OUT})/[(V_{IN})(f_{OSC})(L)] =(3.5V)(15V-3.5V)/[(15V)(570kHz)(10uH)] =0.471A"
- note removed: "I_{VC-LIM}=I_{LOAD}(1-K_{I}) I_{VC-LIM}=1.5V/((A_{CS})(R_{ON}))"
- note removed: "If there's space, double the MOSFET footprints"
- note removed: "L>{V_{BATT}[V_{DCIN(MAX)}-V_{BATT}]}/{[V_{DCIN(MAX)}][f_{SW}][I_{CHG}][LIR]} >((14.8V)(19.5V-14.8V))/((19.5V)(300kHz)(2.5A)(0.3)) >15.85uH"
- note removed: "LiPo Cell Balancing"
- note removed: "LiPo Cell Voltage Sensing"
- note removed: "Maybe use same inductor as 5.1V buck?"
- note removed: "NOTE CAPCITOR VOLTAGE RATINGS"
- note removed: "R_{4}=[(2pi)(V_{OUT})(f_{CRS})(C_{OUT})]/[(V_{FB})(G_{MP})(G_{MA})] =[(2pi)(V_{OUT})(f_{CRS})(C_{OUT})]/[(0.8V)(7A/V)(82uA/V)] =13682.8948(V_{OUT})(f_{CRS})(C_{OUT}) =13682.8948(3.5)(40k)(20u) =38.312kOhms~=38.3kOhms"
- note removed: "R_{CSB}=0.2V(V_{ICH-EN}/V_{REF})/I_{CHG} =0.2V(3.3V/4.2V)/2.5A ~=62.6mOhms I_{CHG}=0.2V(3.3V/4.2V)/0.0626R=2.5103A"
- note removed: "R_{T}=R_{B}(V_{OUT}-0.8V)/0.8V =15e3(5.1-0.8)/0.8 =80.625k~=80.6k"
- note removed: "Use murata or TDK for capacitors Beware of DC bias"
- note removed: "V_{DD}>=V_{IN}/8+1.5=20/8+1.5=4V V_{DD}>=V_{OuT}/4=5.1/4=1.275V"
- note removed: "V_{ICH-EN}=I_{CHG} * 1.3146"
- note removed: "V_{Iout}=20(R_{CSB} * I_{chg}) C_{load} < 5nF"
- note removed: "V_{OUT}=0.8[(R_{1}+R_{2})/R_{2}] =0.8*[(453k+133k)/133k]=3.525V"
- note removed: "V_{RPL}=I_{RPL}[R_{ESR}+1/(8(C_{OUT})(f_{OSC}))] =(0.471A)[10mOhm+1/(8(20uF)(570kHz))] =9.87mV"
- note removed: "V_{VADJ}=9.5(V_{CELL})-9(V_{REF}) =9.5(4.1V)-9(4.2V)=1.15V R_{2}=R_{1}[V_{VADJ}/(V_{REF}-V_{VADJ})] =133k*(1.15/(4.2-1.15)~=49.9k V_{VADJ}=1.14587V V_{CELL}=(1.14587V+9(4.2V))/9.5=4.0996V"
- note removed: "dI_{L}=K_{I}(I_{LOAD}) ~=0.33(10)=3.3A L=[(V_{IN}-V_{OUT})/((dI_{L})(f_{SW}))][V_{OUT}/V_{IN}] =[(16-5.1)/((3.3)(600e3))][5.1/16]=1.755uH dI_{L}=[(16-5.1)/((2e-6)(600e3))][5.1/16]=2.895A K_{I}=2.895/10=0.29 dI_{L-MIN}=[(12-5.1)/((2e-6)(600e3))][5.1/12]=2.444A dI_{L-MAX}=[(19-5.1)/((2e-6)(600e3))][5.1/19]=3.109A I_{SAT}>16A"
- note removed: "dV_{RR}=(0.01)*V_{OUT}=(0.01*5.1=0.051V C_{OUT}=dI_{L}/[(8)(f_{SW})(dV_{RR}-(dI_{L})(ESR))] =2.895/[(8)(600e3)(0.051-(2.895)(0.015))]=80uF C_{OUT}=[2(dI_{L})]/[(f_{SW})(V_{DROOP}-(I_{LOAD-STEP})(ESR))] =[2(2.895)]/[(600e3)(0.1-(3)(0.015))]=175uF"
- note removed: "f_{CROSS}=f_{SW}/12=600e3/12=50kHz f_{ZERO}=f_{CROSS}/4=12.5kHz R_{COMP}=[(f_{CROSS}/(F_{CROSS}+F_{ZERO})][2(pi)(f_{CROSS})(C_{OUT})/((G_{M})(A_{CS}))][V_{OUT}/V_{REF}] =[50e3/(50e3+12.5e3)][(2)(pi)(50e3)(C_{OUT})/((500e-6)(A_{CS})][V_{OUT}/0.8] =[(C_{OUT})(V_{OUT})/(A_{CS})][628318530.718] =[(4*47e-6*0.67)(5.1)/13.4][628318530.718] =30.12kOhms C_{COMP}=1/[2(pi)(R_{COMP})(f_{ZERO})] =1/[2(pi)(27.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"
- note removed: "slew rate limit?"
- moved on the sheet: C10, C11, C12, C13, C14, C15, C16, C17, C18, C19, C2, C20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

Commit message: Organization and start side project
Parts:
- J9: value 100mil -> DNP
Other:
- note added: "CONNECTORS"
- note added: "Diagnostic"
- note added: "Front LED"
- note added: "Left Side Indication"
- note added: "Li-ion Balance"
- note added: "Li-ion Power"
- note added: "Rear Panel"
- note added: "Right Side Indication"
- note added: "SWD"
- note added: "rPi/Arducam"
- note removed: "LiPo Balance"
- note removed: "LiPo Main"
- moved on the sheet: C1, C21, C22, C25, C26, D1, D4, F1, F2, F3, F4, F5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

Commit message: Some capacitor selection
Parts:
- removed C1, C2, C32, C37, C38: 10uF, symbol Device:C_Small
- removed C47: DNP, symbol Device:C_Polarized_Small
- removed L?: R0, symbol Device:L_Ferrite_Small
- added C? (x5): 10uF, symbol Device:C_Small
- added C?: 33uF, Capacitor_THT:CP_Radial_D6.3mm_P2.50mm, symbol Device:C_Polarized_Small
- added R?: 0R, symbol Device:R_Small
- C27: footprint (none) -> Capacitor_THT:CP_Radial_D6.3mm_P2.50mm; ESR (none) -> 40mOhm @ 100kHz; Manufacturer (none) -> KEMET; Part Number (none) -> A758EK336M1EAAE040; Temp Range (none) -> -55°C +105°C; Tolerance (none) -> 20%; Voltage (none) -> 25V
- C35: value 620pF -> 44.2k
- C60: footprint (none) -> Capacitor_THT:CP_Radial_D8.0mm_P3.50mm; ESR (none) -> 7mOhm @ 100kHz; Manufacturer (none) -> Nichicon; Part Number (none) -> RR71A101MDN1; Temp Range (none) -> -55°C +105°C; Tolerance (none) -> 20%; Voltage (none) -> 10V
- R50: value 38.3k -> 510pF
- R51: value 453k -> 402k
- R52: value 133k -> 100k
- R6: value ???? -> 0R
- R7: value ???? -> DNP
Connections:
- net +3V5 is gone; now on net +4V: C36.1, C46.2, L9.2, R51.1, U7.1 (IN), U7.3 (EN)
- net EN_3V5 is gone; now on net EN_4V: J9.1 (Pin_1), U4.42 (PB6)
- net +4V: now also C?.2, C?.2
- net +4V_SW: now also R?.2
- net GND: now also C?.1, C?.1, C?.1, C?.1, C?.1, C?.2
- net VSYS: now also C?.2
- net VSYS_SW: now also C?.1, C?.2, C?.2
- net at C39.2, C40.1, U8.5 (VDD): now also R?.1
- net 3V5_EN renamed EN_4V
Other:
- note added: "170mV dropout @ 3.3V/300mA ±2% Accuracy"
- note added: "5A"
- note added: "Alt: C_{OUT}=30uF, R_{4}=64.9kOhms, C_{4}=360pF"
- note added: "C@19V=6uF"
- note added: "C@5.1V=27uF"
- note added: "Check Min On-Time Spec -------------------- 250ns<=1.75(V_{OUT}/V_{IN}) 250ns<=1.75(4/19)=368ms"
- note added: "Loop Compensation ------------------------ R_{4}=[(2pi)(V_{OUT})(f_{CRS})(C_{OUT})]/[(V_{FB})(G_{MP})(G_{MA})] =[(2pi)(V_{OUT})(f_{CRS})(C_{OUT})]/[(0.8V)(7A/V)(82uA/V)] =13682.8948(V_{OUT})(f_{CRS})(C_{OUT}) =13682.8948(4)(40e3)(20e-6) =43.785kOhms~=44.2kOhms C_{4}=1/[(2pi)(R_{4})(f_{CRS}/6)] =1/[(2pi)(44.2e3)(40e3/6)] =540pF~=510pF"
- note added: "MOSFET PSMN4R1-30YLC -------------------- R_{DS(ON)@4V}=5mOhms V_{f(DIODE)@10A}=0.75V Q_{G(TOT)@4V}=10nC C_{G(TOT)@4V}=10nC/4V=2.5nF C_{iss}=1.5nF R_{G}=1.9Ohms"
- note added: "Maximum Load Capacitance ----------------- C_{LOAD-MAX}=[(t_{ss})(I_{LIM}-I_{OUTMAX}-I_{RPL}/2)/V_{OUT}]-C_{OUT} =[(1.2e-3)(2.1-0.2-0.526/2)/4]-20e-6 =471uF"
- note added: "Minimum Input Capacitance -------------------- V_{CIN-MAX-RPL}=0.01(V_{IN-MIN})+([I_{LOAD-MAX})(ESR_{CIN}) =0.01(12)-(10)(0.005)=70mV C_{IN-MIN}=[I_{LOAD-MAX}/V_{MAX-RPL}][D(1-D)/f_{SW}] =[10/0.07][0.425(1-0.425)/600e3]=58.1uF Minimum Output Capacitance ------------------------- dV_{OUTRR}=(0.01)V_{OUT}=(0.005)5.1=0.051V C_{OUT}>dI_{L}/[(8)(f_{SW})(dV_{OUTRR}-(dI_{L})(ESR_{COUT}))] >2.895/[(8)(60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"
- note added: "Minimum Output Capacitance -------------------- C_{OUT}>4.2(1+16.8/18.5)/[(16.8)(300e3)(62.6e-3)]=25.4uF R_{ESR}<0.0626*12/4.2=179mOhms"
- note added: "Output Voltage Set ------------------------ V_{OUT}=0.8[(R_{1}+R_{2})/R_{2}] =0.8*[(402+100)/100]=4.016V"
- note added: "Ripple Current at Selected Inductance ------------------------ I_{RPL}=(V_{OUT})(V_{IN}-V_{OUT})/[(V_{IN})(f_{OSC})(L)] =(4V)(16V-4V)/[(16V)(570kHz)(10uH)] =0.526A Ripple Voltage at Selected Output Capacitance ------------------------ V_{RPL}=I_{RPL}[R_{ESR}+1/(8(C_{OUT})(f_{OSC}))] =(0.526A)[0.005Ohm+1/(8(20uF)(570kHz))] =8.40mV"
- note added: "f_{OSC}=570kHz f_{CRS}=40kHz"
- note removed: "-> C_{OUT}=20uF, R_{4}=38.3kOhms, C_{4}=620pF Alt: C_{OUT}=30uF, R_{4}=57.6kOhms, C_{4}=430pF Alt: L=22uH"
- note removed: "170mV dropout @ 3.3V/300mA"
- note removed: "Loop Compensation ------------------------ R_{4}=[(2pi)(V_{OUT})(f_{CRS})(C_{OUT})]/[(V_{FB})(G_{MP})(G_{MA})] =[(2pi)(V_{OUT})(f_{CRS})(C_{OUT})]/[(0.8V)(7A/V)(82uA/V)] =13682.8948(V_{OUT})(f_{CRS})(C_{OUT}) =13682.8948(3.5)(40k)(20u) =38.312kOhms~=38.3kOhms C_{4}=1/[(2pi)(R_{4})(f_{CRS}/6)] =1/[(2pi)(3.83k)(40k/6) =623.32pF~=620pF"
- note removed: "MOSFET PSMN4R1-30YLC -------------------- R_{DS(ON)@4V}=5mOhms V_{f(DIODE)@10A}=0.75V Q_{G(TOT)@4V}=10nC C_{G(TOT)@4V)=10nC/4V=2.5nF C_{iss}=1.5nF R_{G}=1.9Ohms"
- note removed: "Minimum Input Capacitance -------------------- V_{CIN-MAX-RPL}=0.01(V_{IN-MIN})+([I_{LOAD-MAX})(ESR_{CIN}) =0.01(12)-(10)(0.001)=110mV C_{IN-MIN}=[I_{LOAD-MAX}/V_{MAX-RPL}][D(1-D)/f_{SW}] =[10/0.11][0.425(1-0.425)/600e3]=37uF Minimum Output Capacitance ------------------------- dV_{OUTRR}=(0.01)V_{OUT}=(0.01)5.1=0.051V C_{OUT}>dI_{L}/[(8)(f_{SW})(dV_{OUTRR}-(dI_{L})(ESR_{COUT}))] >2.895/[(8)(600e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"
- note removed: "Minimum Output Capacitance -------------------- C_{OUT}>4.2(1+16.8/18.5)/((16.8)(300k)(62.6m))=25.4uF R_{ESR}<0.0626*12/4.2=179mOhms"
- note removed: "Output Voltage Set ------------------------ V_{OUT}=0.8[(R_{1}+R_{2})/R_{2}] =0.8*[(453k+133k)/133k]=3.525V"
- note removed: "Ripple Current at Selected Inductance ------------------------ I_{RPL}=(V_{OUT})(V_{IN}-V_{OUT})/[(V_{IN})(f_{OSC})(L)] =(3.5V)(15V-3.5V)/[(15V)(570kHz)(10uH)] =0.471A Ripple Voltage at Selected Output Capacitance ------------------------ V_{RPL}=I_{RPL}[R_{ESR}+1/(8(C_{OUT})(f_{OSC}))] =(0.471A)[10mOhm+1/(8(20uF)(570kHz))] =9.87mV"
- note removed: "change to > 4V"
- note removed: "f_{CRS}=40kHz"
- note removed: "f_{OSC}=570kHz"
- moved on the sheet: D2, L2, Q1, Q2, R12, R13, R3, R4, R6, R7, R8, R9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

Commit message: Jelly bean selection WIP
Parts:
- removed C31: 47uF, symbol Device:C_Polarized_Small
- removed C35: 44.2k, symbol Device:C_Small
- removed C5: 2.2uF, symbol Device:C_Small
- removed D4: D_Schottky_Small, symbol Device:D_Schottky_Small
- removed R18: 0R, symbol Device:R_Small
- added C51: 510pF, Capacitor_SMD:C_0402_1005Metric, symbol Device:C_Small
- added C? (x2): 10uF, Capacitor_SMD:C_1210_3225Metric, symbol Device:C_Small
- added R?: 0R, symbol Device:R_Small
- C12: renamed from C49; footprint (none) -> Capacitor_SMD:C_1210_3225Metric
- C16: renamed from C20; footprint (none) -> Capacitor_SMD:C_0402_1005Metric; Manufacturer (none) -> Würth Elektronik; Part Number (none) -> 885012205061; Temp Range (none) -> -55°C +125°C; Tolerance (none) -> 10%; Voltage (none) -> 50V
- C17, C18, C21, C45, C46, C55, C56, C57: renamed from C?; footprint (none) -> Capacitor_SMD:C_1210_3225Metric
- C19: renamed from C53; footprint (none) -> Capacitor_SMD:C_0402_1005Metric; Manufacturer (none) -> Würth Elektronik; Part Number (none) -> 885012205061; Temp Range (none) -> -55°C +125°C; Tolerance (none) -> 10%; Voltage (none) -> 50V
- C22: renamed from C55; footprint (none) -> Capacitor_SMD:C_0402_1005Metric; Manufacturer (none) -> Würth Elektronik; Part Number (none) -> 885012205045; Temp Range (none) -> -55°C +125°C; Tolerance (none) -> 10%; Voltage (none) -> 25V
- C23: renamed from C6; footprint (none) -> Capacitor_SMD:C_0402_1005Metric; Manufacturer (none) -> Würth Elektronik; Part Number (none) -> 885012205061; Temp Range (none) -> -55°C +125°C; Tolerance (none) -> 10%; Voltage (none) -> 50V
- C25: renamed from C10; footprint (none) -> Capacitor_SMD:C_0402_1005Metric; Manufacturer (none) -> Würth Elektronik; Part Number (none) -> 885012205061; Temp Range (none) -> -55°C +125°C; Tolerance (none) -> 10%; Voltage (none) -> 50V
- C29: renamed from C11; footprint (none) -> Capacitor_SMD:C_0402_1005Metric; Manufacturer (none) -> Würth Elektronik; Part Number (none) -> 885012205061; Temp Range (none) -> -55°C +125°C; Tolerance (none) -> 10%; Voltage (none) -> 50V
- C3: renamed from C7; footprint (none) -> Capacitor_SMD:C_0603_1608Metric; Manufacturer (none) -> TDK Corporation; Part Number (none) -> CGA3E1X7R1E105K080AC; Temp Range (none) -> -55°C +125°C; Tolerance (none) -> 10%; Voltage (none) -> 25V
- C32: renamed from C12; footprint (none) -> Capacitor_SMD:C_0603_1608Metric; Manufacturer (none) -> TDK Corporation; Part Number (none) -> CGA3E1X7R1E105K080AC; Temp Range (none) -> -55°C +125°C; Tolerance (none) -> 10%; Voltage (none) -> 25V
- C34: renamed from C19; footprint (none) -> Capacitor_SMD:C_0402_1005Metric; Manufacturer (none) -> Würth Elektronik; Part Number (none) -> 885012205061; Temp Range (none) -> -55°C +125°C; Tolerance (none) -> 10%; Voltage (none) -> 50V
- C36: renamed from C23; footprint (none) -> Capacitor_SMD:C_0402_1005Metric; Manufacturer (none) -> Würth Elektronik; Part Number (none) -> 885012205061; Temp Range (none) -> -55°C +125°C; Tolerance (none) -> 10%; Voltage (none) -> 50V
- C39: renamed from C?; footprint (none) -> Capacitor_SMD:C_0402_1005Metric; Manufacturer (none) -> Würth Elektronik; Part Number (none) -> 885012205061; Temp Range (none) -> -55°C +125°C; Tolerance (none) -> 10%; Voltage (none) -> 50V
- C40: renamed from C41; footprint (none) -> Capacitor_SMD:C_0603_1608Metric; Manufacturer (none) -> TDK Corporation; Part Number (none) -> CGA3E1X7R1E105K080AC; Temp Range (none) -> -55°C +125°C; Tolerance (none) -> 10%; Voltage (none) -> 25V
- C41: renamed from C42; footprint (none) -> Capacitor_SMD:C_0603_1608Metric; Manufacturer (none) -> TDK Corporation; Part Number (none) -> CGA3E1X7R1E105K080AC; Temp Range (none) -> -55°C +125°C; Tolerance (none) -> 10%; Voltage (none) -> 25V
- C42: renamed from C43; footprint (none) -> Capacitor_SMD:C_0603_1608Metric; Manufacturer (none) -> TDK Corporation; Part Number (none) -> CGA3E1X7R1E105K080AC; Temp Range (none) -> -55°C +125°C; Tolerance (none) -> 10%; Voltage (none) -> 25V
- C43: renamed from C44; footprint (none) -> Capacitor_SMD:C_0603_1608Metric; Manufacturer (none) -> TDK Corporation; Part Number (none) -> CGA3E1X7R1E105K080AC; Temp Range (none) -> -55°C +125°C; Tolerance (none) -> 10%; Voltage (none) -> 25V
- C47: renamed from C33; footprint (none) -> Capacitor_SMD:C_0402_1005Metric; Manufacturer (none) -> Würth Elektronik; Part Number (none) -> 885012205061; Temp Range (none) -> -55°C +125°C; Tolerance (none) -> 10%; Voltage (none) -> 50V
- C48: renamed from C34; footprint (none) -> Capacitor_SMD:C_0402_1005Metric; Manufacturer (none) -> Würth Elektronik; Part Number (none) -> 885012205061; Temp Range (none) -> -55°C +125°C; Tolerance (none) -> 10%; Voltage (none) -> 50V
- C5: renamed from C39; footprint (none) -> Capacitor_SMD:C_0402_1005Metric; Manufacturer (none) -> Würth Elektronik; Part Number (none) -> 885012205061; Temp Range (none) -> -55°C +125°C; Tolerance (none) -> 10%; Voltage (none) -> 50V
- C58: renamed from C46; footprint (none) -> Capacitor_SMD:C_0603_1608Metric; Manufacturer (none) -> TDK Corporation; Part Number (none) -> CGA3E1X7R1E105K080AC; Temp Range (none) -> -55°C +125°C; Tolerance (none) -> 10%; Voltage (none) -> 25V
- C59: renamed from C51; footprint (none) -> Capacitor_SMD:C_0603_1608Metric; Manufacturer (none) -> TDK Corporation; Part Number (none) -> CGA3E1X7R1E105K080AC; Temp Range (none) -> -55°C +125°C; Tolerance (none) -> 10%; Voltage (none) -> 25V
- C6: renamed from C40; footprint (none) -> Capacitor_SMD:C_0603_1608Metric; Manufacturer (none) -> TDK Corporation; Part Number (none) -> CGA3E1X7R1E105K080AC; Temp Range (none) -> -55°C +125°C; Tolerance (none) -> 10%; Voltage (none) -> 25V
- C7: renamed from C45; footprint (none) -> Capacitor_SMD:C_0402_1005Metric; Manufacturer (none) -> Murata Electronics; Part Number (none) -> GRM1555C1H510GA01D; Temp Range (none) -> -55°C +125°C; Tolerance (none) -> 2%; Voltage (none) -> 50V
- C9: renamed from C48; footprint (none) -> Capacitor_SMD:C_0402_1005Metric; Manufacturer (none) -> Murata Electronics; Part Number (none) -> GRM1555C1H511JA01D; Temp Range (none) -> -55°C +125°C; Tolerance (none) -> 5%; Voltage (none) -> 50V
- R60: renamed from R50; value 510pF -> 44.2k
- gave numbers to parts that had none: 11
- renumbered C4 to C1, C13 to C10, C14 to C11, C15 to C13, C16 to C14, C17 to C15, C27 to C20, C56 to C26, C18 to C27, C24 to C31, C60 to C35, C28 to C37, C29 to C38, C8 to C4, C9 to C44, C21 to C49, C22 to C50, C25 to C52, C26 to C53, C36 to C54, C3 to C60, D3 to D1, D5 to D2, D6 to D3, D7 to D4, D8 to D5, D1 to D6, D2 to D8, F5 to F4, F6 to F5, F7 to F6, F8 to F7, F4 to F8, J2 to J1, J4 to J2, J6 to J3, J8 to J4, J1 to J5, J5 to J6, J3 to J7, J9 to J8, J7 to J9, L4 to L1, L2 to L10, L10 to L2, L1 to L4, L9 to L5, L5 to L6, L6 to L7, L7 to L8, L8 to L9, Q7 to Q1, Q14 to Q10, Q15 to Q11, Q16 to Q12, Q22 to Q17, Q1 to Q18, Q2 to Q19, Q25 to Q2, Q6 to Q20, Q5 to Q21, Q26 to Q3, Q8 to Q4, Q9 to Q5, Q10 to Q6, Q11 to Q7, Q12 to Q8, Q13 to Q9, R17 to R1, R30 to R10, R31 to R11, R32 to R12, R5 to R13, R64 to R14, R65 to R15, R33 to R16, R66 to R17, R67 to R18, R68 to R19, R36 to R20, R37 to R21, R38 to R22, R39 to R23, R42 to R24, R43 to R25, R44 to R26, R45 to R27, R46 to R28, R47 to R29, R19 to R3, R48 to R30, R49 to R31, R54 to R32, R55 to R34, R56 to R35, R57 to R36, R58 to R37, R59 to R38, R60 to R39, R20 to R4, R61 to R40, R62 to R41, R34 to R42, R35 to R43, R22 to R44, R23 to R45, R1 to R46, R6 to R47, R7 to R48, R40 to R49, R21 to R5, R41 to R50, R8 to R51, R9 to R52, R12 to R53, R13 to R54, R2 to R55, R24 to R56, R25 to R57, R26 to R58, R27 to R59, R51 to R61, R52 to R62, R3 to R63, R4 to R64, R14 to R65, R16 to R66, R15 to R67, R63 to R7, R28 to R8, R29 to R9, U3 to U1, U8 to U2, U5 to U3, U1 to U5, U2 to U7, U7 to U8
Connections:
- net GND: now also C?.1, C?.1
- net ~{CHG_EN}: now also R?.2
- net at R1.1, R3.1, U1.6 (ICHG/EN): now also R?.1
- net at R60.1: now also C51.2
- net at U6.6 (COMP): now also C51.1
- net at U1.16 (VL): now also C?.2, C?.2
