File: faclon-main/FalconMain/FalconMain.kicad_sch (KiCad schematic)
At the start: 193 parts, among them J1 Nano-Fit, J2 PTH, J3 Nano-Fit, J4 100mil, J5 Nano-Fit, J6 100mil, J7 Nano-Fit, J8 DNP, J9 JST-XH, Q1 Q_PMOS_GDS, Q10 Q_PMOS_GDS, Q11 Q_PMOS_GDS, Q12 Q_PMOS_GDS, Q13 Q_NMOS_GDS, Q14 Q_PMOS_GDS, Q15 Q_PMOS_GDS, Q16 Q_PMOS_GDS, Q17 Q_PMOS_GDS, Q18 Q_NMOS_GDS, Q19 Q_NMOS_GDS, Q2 Q_NMOS_GDS, Q20 Q_PMOS_GDS, Q21 Q_NMOS_GDS, Q22 Q_PMOS_GDS, Q3 Q_NMOS_GDS, Q4 Q_PMOS_GDS, Q5 Q_NMOS_GDS, Q6 Q_NMOS_GDS, Q7 Q_NMOS_GDS, Q8 Q_NMOS_GDS, Q9 Q_PMOS_GDS, U1 MAX1873TEEE+, U2 ADP1883ARMZ-0.6-R7, U3 LTC4412ES6#TRPBF, U4 STM32L152CBT6, U5 AL8843QSP-13, U6 BD9E104FJ-E2, U7 AL8843QSP-13, U8 NCP164ASN330T1G, Y1 8MHz, Y2 32.768kHz

Commit message: WIP
Parts:
- removed C44: DNP, symbol Device:C_Small
- removed C49, C50, C52, C53, C60: ?????, symbol Device:C_Small
- removed L6, L7, L8, L9: ?????, symbol Device:L_Small
- removed R56, R57, R59, R66: ????, symbol Device:R_Small
- added C25: 100uF, Capacitor_THT:CP_Radial_D8.0mm_P3.50mm, symbol Device:C_Polarized_Small
- added C45: DNP, Capacitor_SMD:C_0402_1005Metric, symbol Device:C_Small
- added C57: 10nF, Capacitor_SMD:C_0402_1005Metric, symbol Device:C_Small
- C1, C4: footprint (none) -> Capacitor_SMD:C_0603_1608Metric; Manufacturer (none) -> TDK Corporation; Part Number (none) -> C1608X7R1H224K080AB; Temp Range (none) -> -55°C +125°C; Tolerance (none) -> 10%; Voltage (none) -> 50V
- C11: renamed from C10; footprint (none) -> Capacitor_SMD:C_0402_1005Metric; Manufacturer (none) -> Würth Elektronik; Part Number (none) -> 885012205067; Temp Range (none) -> -55°C +125°C; Tolerance (none) -> 10%; Voltage (none) -> 50V
- C12: renamed from C11; footprint (none) -> Capacitor_SMD:C_0402_1005Metric; Manufacturer (none) -> Würth Elektronik; Part Number (none) -> 885012205067; Temp Range (none) -> -55°C +125°C; Tolerance (none) -> 10%; Voltage (none) -> 50V
- C14: renamed from C13; footprint (none) -> Capacitor_SMD:C_0402_1005Metric; Manufacturer (none) -> Murata Electronics; Part Number (none) -> GRM155R71H473KE14D; Temp Range (none) -> -55°C +125°C; Tolerance (none) -> 10%; Voltage (none) -> 50V
- C15: renamed from C14; footprint (none) -> Capacitor_SMD:C_0402_1005Metric; Manufacturer (none) -> Murata Electronics; Part Number (none) -> GRM155R71H473KE14D; Temp Range (none) -> -55°C +125°C; Tolerance (none) -> 10%; Voltage (none) -> 50V
- C16: renamed from C15; footprint (none) -> Capacitor_SMD:C_0402_1005Metric; Manufacturer (none) -> Würth Elektronik; Part Number (none) -> 885012205061; Temp Range (none) -> -55°C +125°C; Tolerance (none) -> 10%; Voltage (none) -> 50V
- C21: renamed from C20; HF Ripple Current (none) -> 3.1 A @ 100 kHz
- C28: renamed from C27; value ????? -> 15pF; footprint (none) -> Capacitor_SMD:C_0402_1005Metric; Manufacturer (none) -> Würth Elektronik; Part Number (none) -> 885012005056; Temp Range (none) -> -55°C +125°C; Tolerance (none) -> 5%; Voltage (none) -> 50V
- C32: renamed from C31; value ????? -> 15pF; footprint (none) -> Capacitor_SMD:C_0402_1005Metric; Manufacturer (none) -> Würth Elektronik; Part Number (none) -> 885012005056; Temp Range (none) -> -55°C +125°C; Tolerance (none) -> 5%; Voltage (none) -> 50V
- C36: renamed from C35; HF Ripple Current (none) -> 5.6 A @ 100 kHz
- C38: renamed from C37; value ????? -> 6pF; footprint (none) -> Capacitor_SMD:C_0402_1005Metric; Manufacturer (none) -> TDK Corporation; Part Number (none) -> CGA2B2C0G1H060D050BA; Temp Range (none) -> -55°C +125°C; Tolerance (none) -> 0.5pF; Voltage (none) -> 50V
- C39: renamed from C38; value ????? -> 6pF; footprint (none) -> Capacitor_SMD:C_0402_1005Metric; Manufacturer (none) -> TDK Corporation; Part Number (none) -> CGA2B2C0G1H060D050BA; Temp Range (none) -> -55°C +125°C; Tolerance (none) -> 0.5pF; Voltage (none) -> 50V
- C51: renamed from C54; footprint (none) -> Capacitor_SMD:C_0402_1005Metric; Manufacturer (none) -> Murata Electronics; Part Number (none) -> GCM1555C1H120JA16D; Temp Range (none) -> -55°C +125°C; Tolerance (none) -> 5%; Voltage (none) -> 50V
- C9: renamed from C8; value 33uF -> 100uF; footprint Capacitor_THT:CP_Radial_D6.3mm_P2.50mm -> Capacitor_THT:CP_Radial_D8.0mm_P3.50mm; ESR 40mOhm @ 100kHz -> 25mOhm @ 100kHz; HF Ripple Current (none) -> 1.817 A @ 100 kHz; Part Number A758EK336M1EAAE040 -> A759KS107M1EAAE025; Temp Range -55°C +105°C -> -55°C +125°C
- D1, D2, D3: Manufacturer (none) -> STMicroelectronics; Part Number (none) -> FERD2045SB-TR; Temp Range (none) -> -40°C +150°C; Voltage (none) -> 45V
- D4, D5, D6: value D_Schottky_Small -> 500mA; Manufacturer (none) -> Toshiba Semiconductor and Storage; Part Number (none) -> CUS551V30,H3F; Temp Range (none) -> -55°C +125°C; Voltage (none) -> 30V
- D7: renamed from D8; Manufacturer (none) -> STMicroelectronics; Part Number (none) -> FERD2045SB-TR; Temp Range (none) -> -40°C +150°C; Voltage (none) -> 45V
- F1, F8: value 6A -> 7A; Part Number 0686F6000-01 -> 0686F7000-01; Power 0.64W -> 0.75W; Voltage (none) -> 32V
- F2, F3: value 3.5A -> 4A; footprint (none) -> Resistor_SMD:R_0402_1005Metric; Manufacturer (none) -> Schurter Inc.; Part Number (none) -> 3414.0123.26; Power (none) -> 0.23W; Temp Range (none) -> -55°C +125°C; Voltage (none) -> 32V
- F4, F5, F6, F7: value 200mA -> 300mA; footprint (none) -> Resistor_SMD:R_0603_1608Metric; Manufacturer (none) -> Bel Fuse Inc.; Part Number (none) -> C2Q 300; Power (none) -> 0.07W; Temp Range (none) -> -55°C +125°C; Voltage (none) -> 32V
- R28, R29, R30, R31: value 47 -> 47R
- R32: value 100K -> 100k
- R49: value 243k -> 442k
- R50: value 49.9 -> 100k
- R57: renamed from R61; footprint Resistor_SMD:R_0402_1005Metric -> (none); Manufacturer Stackpole Electronics Inc -> (none); Part Number RMCF0402FT453K -> (none); Power 0.063W -> (none); Temp Range -55°C +155°C -> (none); Tolerance 1% -> (none)
- R58: value ???? -> 100k
- R62: footprint Resistor_SMD:R_0402_1005Metric -> (none); Manufacturer Stackpole Electronics Inc -> (none); Part Number RMCF0402FT133K -> (none); Power 0.063W -> (none); Temp Range -55°C +155°C -> (none); Tolerance 1% -> (none)
- Y1: ESR (none) -> 40 Ohms; Load Capacitance ?pF -> 18pF; Manufacturer (none) -> Würth Elektronik; Part Number (none) -> 830050510; Temp Range (none) -> -40°C +85°C; Tolerance (none) -> 30ppm
- Y2: ESR (none) -> 50 kOhms; Load Capacitance ?pF -> 6pF; Manufacturer (none) -> Würth Elektronik; Part Number (none) -> 830014219B; Temp Range (none) -> -40°C +85°C; Tolerance (none) -> 20ppm
- gave numbers to parts that had none: 3
- renumbered C9 to C10, C12 to C13, C16 to C17, C17 to C18, C18 to C19, C19 to C20, C21 to C22, C22 to C23, C23 to C24, C25 to C26, C26 to C27, C28 to C29, C29 to C30, C30 to C31, C32 to C33, C33 to C34, C34 to C35, C36 to C37, C39 to C40, C40 to C41, C41 to C42, C42 to C43, C43 to C44, C45 to C46, C46 to C47, C47 to C48, C48 to C49, C51 to C50, C55 to C52, C56 to C53, C57 to C54, C58 to C55, C59 to C56, C5 to C6, C6 to C7, C7 to C8, L10 to L6, R60 to R56, R63 to R59, R64 to R60, R65 to R61, R67 to R63
Connections:
- net GND: now also R58.1, C25.2, C45.2; no longer R62.1
- net NRST: now also C45.1
- net VSYS: now also C25.1, C57.1
- net at R58.2: now also C51.2, R57.2, U6.5 (FB)
- net at Q21.2 (D), R61.1: now also R62.1
- net at Q20.1 (G), Q22.1 (G): now also R62.2, C57.2
Other:
- note added: "C_{L1}=C_{L2}=2(C_{L}-C_{stray} =2(18pF-10pF)=16pF~=15pF"
- note added: "C_{L1}=C_{L2}=2(C_{L}-C_{stray} =2(6pF-3pF)=6pF~=6pF"
- note added: "LV PMOS will turn on later and turn off earlier than HV"
- note added: "MLCCC @19V C=6uF"
- note added: "Max LED power: (3.5V*3*0.25A*4+10W)=21W Max 5.1V power: 10A*5.1V/0.9=57W Max LED VSYS current: 21W/13.2V=1.6A Max VBAT current: (21W+57W)/13.2V=5.9A Max AC/DC current: (21W+57W)/18.5V=4.2A"
- note added: "Note: Measured voltage may be 50mV lower than true if measured while a discharge FET is conducting (due to parasitic resistance)"
- note removed: "C@19V=6uF"
- note removed: "LV PMOS will turn on later, and turn off earlier, than HV"
- note removed: "Max LED power: (3.5V*3*0.25A*4+10W)=21W Max 5.1V power: 10A*5.1V/0.9=57W Max LED VSYS current: 21W/13.2V=1.6A Max VBAT current: (21W+57W)/13.2V=5.9A Min AC/DC current rating: (21W+57W)/18.5V=4.2A"

Commit message: Select all main board components
Parts:
- removed C46: 10uF, Capacitor_SMD:C_1210_3225Metric, symbol Device:C_Small
- removed D6: 500mA, symbol Device:D_Schottky_Small
- removed L4: 100uH, symbol Device:L_Small
- removed Q10, Q11, Q12, Q14, Q15, Q16, Q17, Q22, Q9: Q_PMOS_GDS, symbol Device:Q_PMOS_GDS
- removed Q13, Q18, Q19, Q21, Q5, Q6, Q7, Q8: Q_NMOS_GDS, symbol Device:Q_NMOS_GDS
- removed R46: 1M, symbol Device:R_Small
- removed R48: DNP, symbol Device:R_Small
- removed R55: 499m, symbol Device:R_Small
- removed U5: AL8843QSP-13, JetkovKiCADLib:8-SOIC_SO-8EP_DIO, symbol JetkovKiCADLib:AL8843QSP-13
- added Q10, Q11, Q12, Q14, Q15, Q16, Q17, Q22, Q9: Q_PMOS_GSD, symbol Device:Q_PMOS_GSD
- added Q13, Q18, Q19, Q21, Q5, Q6, Q7, Q8: Q_NMOS_GSD, symbol Device:Q_NMOS_GSD
- added R47: DNP, Resistor_SMD:R_0402_1005Metric, symbol Device:R_Small
- L1: value ????? -> 22uH; Manufacturer (none) -> Eaton - Electronics Division; Part Number (none) -> DR125-220-R; Temp Range (none) -> -40°C +125°C; Tolerance (none) -> 20%
- L2: Manufacturer (none) -> Würth Elektronik; Part Number (none) -> 7443551200; Temp Range (none) -> -40°C +155°C; Tolerance (none) -> 20%
- L3: value L_Ferrite_Small -> 600 Ohms @ 100 MHz; footprint (none) -> Inductor_SMD:L_0402_1005Metric; Manufacturer (none) -> Murata Electronics; Part Number (none) -> BLM15AX601SN1D; Temp Range (none) -> -55°C +125°C
- L4: renamed from L5; footprint (none) -> Inductor_SMD:L_1008_2520Metric; Manufacturer (none) -> Taiyo Yuden; Part Number (none) -> LBC2518T100K; Temp Range (none) -> -40°C +105°C; Tolerance (none) -> 10%
- L5: renamed from L6; Manufacturer (none) -> Abracon LLC; Part Number (none) -> AMDLA1306S-470MT; Temp Range (none) -> -40°C +155°C; Tolerance (none) -> 20%
- Q1, Q20, Q4: Part Number (none) -> BUK6Y19-30PX alt DMG4407SSS-13
- R1, R15, R20, R21, R22, R23, R24, R25, R26, R27, R32, R33, R43, R44, R45: footprint (none) -> Resistor_SMD:R_0402_1005Metric; Manufacturer (none) -> YAGEO; Part Number (none) -> RC0402FR-13100KL; Power (none) -> 0.063W; Temp Range (none) -> -55°C +155°C; Tolerance (none) -> 1%
- R10: value 22.6m -> 22m; footprint (none) -> Resistor_SMD:R_1206_3216Metric; Manufacturer (none) -> Susumu; Part Number (none) -> KRL1632E-M-R022-F-T5; Power (none) -> 0.75W; Temp Range (none) -> -55°C +155°C; Tolerance (none) -> 1%
- R11, R8: footprint (none) -> Resistor_SMD:R_0402_1005Metric; Manufacturer (none) -> Stackpole Electronics Inc; Part Number (none) -> RMCF0402FT4R70; Power (none) -> 0.063W; Temp Range (none) -> -55°C +155°C; Tolerance (none) -> 1%
- R12: value 62.6m -> 68m; footprint (none) -> Resistor_SMD:R_1206_3216Metric; Manufacturer (none) -> Susumu; Part Number (none) -> KRL1632E-M-R068-F-T5; Power (none) -> 0.75W; Temp Range (none) -> -55°C +155°C; Tolerance (none) -> 1%
- R13: footprint (none) -> Resistor_SMD:R_0603_1608Metric; Manufacturer (none) -> Stackpole Electronics Inc; Part Number (none) -> RMCF0603JT200R; Power (none) -> 0.1W; Temp Range (none) -> -55°C +155°C; Tolerance (none) -> 5%
- R14, R16, R2, R42, R6: footprint (none) -> Resistor_SMD:R_0402_1005Metric; Manufacturer (none) -> Stackpole Electronics Inc; Part Number (none) -> RMCF0402ZT0R00; Power (none) -> 0.063W; Temp Range (none) -> -55°C +155°C; Tolerance (none) -> Jumper
- R17: footprint (none) -> Resistor_SMD:R_0402_1005Metric; Manufacturer (none) -> Stackpole Electronics Inc; Part Number (none) -> RMCF0402JT2R00; Power (none) -> 0.063W; Temp Range (none) -> -55°C +155°C; Tolerance (none) -> 5%
- R18: footprint (none) -> Resistor_SMD:R_0402_1005Metric; Manufacturer (none) -> Stackpole Electronics Inc; Part Number (none) -> RMCF0402FT80K6; Power (none) -> 0.063W; Temp Range (none) -> -55°C +155°C; Tolerance (none) -> 1%
- R19: footprint (none) -> Resistor_SMD:R_0402_1005Metric; Manufacturer (none) -> Stackpole Electronics Inc; Part Number (none) -> RMCF0402FT15K0; Power (none) -> 0.063W; Temp Range (none) -> -55°C +155°C; Tolerance (none) -> 1%
- R28, R29, R30, R31: footprint (none) -> Resistor_SMD:R_2512_6332Metric; Manufacturer (none) -> Stackpole Electronics Inc; Part Number (none) -> RMCF2512JT47R0; Power 0.75W -> 1W; Temp Range (none) -> -55°C +155°C; Tolerance (none) -> 5%
- R3, R7: footprint (none) -> Resistor_SMD:R_0402_1005Metric; Manufacturer (none) -> Stackpole Electronics Inc; Part Number (none) -> RMCF0402FT27K4; Power (none) -> 0.063W; Temp Range (none) -> -55°C +155°C; Tolerance (none) -> 1%
- R34: footprint (none) -> Resistor_SMD:R_0402_1005Metric; Manufacturer (none) -> Stackpole Electronics Inc; Part Number (none) -> RMCF0402FT221K; Power (none) -> 0.063W; Temp Range (none) -> -55°C +155°C; Tolerance (none) -> 1%
- R36: footprint (none) -> Resistor_SMD:R_0402_1005Metric; Manufacturer (none) -> Stackpole Electronics Inc; Part Number (none) -> RMCF0402FT154K; Power (none) -> 0.063W; Temp Range (none) -> -55°C +155°C; Tolerance (none) -> 1%
- R38: footprint (none) -> Resistor_SMD:R_0402_1005Metric; Manufacturer (none) -> Stackpole Electronics Inc; Part Number (none) -> RMCF0402FT86K6; Power (none) -> 0.063W; Temp Range (none) -> -55°C +155°C; Tolerance (none) -> 1%
- R46: renamed from R47; footprint (none) -> Resistor_SMD:R_0402_1005Metric; Manufacturer (none) -> Stackpole Electronics Inc; Part Number (none) -> RMCF0402ZT0R00; Power (none) -> 0.063W; Temp Range (none) -> -55°C +155°C; Tolerance (none) -> Jumper
- R48: renamed from R49; footprint (none) -> Resistor_SMD:R_0402_1005Metric; Manufacturer (none) -> Stackpole Electronics Inc; Part Number (none) -> RMCF0402FT442K; Power (none) -> 0.063W; Temp Range (none) -> -55°C +155°C; Tolerance (none) -> 1%
- R49: renamed from R50; footprint (none) -> Resistor_SMD:R_0402_1005Metric; Manufacturer (none) -> YAGEO; Part Number (none) -> RC0402FR-13100KL; Power (none) -> 0.063W; Temp Range (none) -> -55°C +155°C; Tolerance (none) -> 1%
- R50: renamed from R51; footprint (none) -> Resistor_SMD:R_0402_1005Metric; Manufacturer (none) -> YAGEO; Part Number (none) -> RC0402FR-13100KL; Power (none) -> 0.063W; Temp Range (none) -> -55°C +155°C; Tolerance (none) -> 1%
- R51: renamed from R52; footprint (none) -> Resistor_SMD:R_0402_1005Metric; Manufacturer (none) -> YAGEO; Part Number (none) -> RC0402FR-13100KL; Power (none) -> 0.063W; Temp Range (none) -> -55°C +155°C; Tolerance (none) -> 1%
- R52: renamed from R53; footprint (none) -> Resistor_SMD:R_0402_1005Metric; Manufacturer (none) -> Stackpole Electronics Inc; Part Number (none) -> RMCF0402FT2K00; Power (none) -> 0.063W; Temp Range (none) -> -55°C +155°C; Tolerance (none) -> 1%
- R53: renamed from R54; footprint (none) -> Resistor_SMD:R_0402_1005Metric; Manufacturer (none) -> Stackpole Electronics Inc; Part Number (none) -> RMCF0402FT2K00; Power (none) -> 0.063W; Temp Range (none) -> -55°C +155°C; Tolerance (none) -> 1%
- R54: renamed from R56; footprint (none) -> Resistor_SMD:R_0402_1005Metric; Manufacturer (none) -> Stackpole Electronics Inc; Part Number (none) -> RMCF0402FT44K2; Power (none) -> 0.063W; Temp Range (none) -> -55°C +155°C; Tolerance (none) -> 1%
- R55: renamed from R57; footprint (none) -> Resistor_SMD:R_0402_1005Metric; Manufacturer (none) -> Stackpole Electronics Inc; Part Number (none) -> RMCF0402FT402K; Power (none) -> 0.063W; Temp Range (none) -> -55°C +155°C; Tolerance (none) -> 1%
- R56: renamed from R58; footprint (none) -> Resistor_SMD:R_0402_1005Metric; Manufacturer (none) -> YAGEO; Part Number (none) -> RC0402FR-13100KL; Power (none) -> 0.063W; Temp Range (none) -> -55°C +155°C; Tolerance (none) -> 1%
- R57: renamed from R59; footprint (none) -> Resistor_SMD:R_0402_1005Metric; Manufacturer (none) -> Stackpole Electronics Inc; Part Number (none) -> RMCF0402FT1M00; Power (none) -> 0.063W; Temp Range (none) -> -55°C +155°C; Tolerance (none) -> 1%
- R58: renamed from R60; footprint (none) -> Resistor_SMD:R_1206_3216Metric; Manufacturer (none) -> Susumu; Part Number (none) -> KRL1632E-M-R039-F-T5; Power (none) -> 0.75W; Temp Range (none) -> -55°C +155°C; Tolerance (none) -> 1%
- R59: renamed from R61; footprint (none) -> Resistor_SMD:R_0402_1005Metric; Manufacturer (none) -> YAGEO; Part Number (none) -> RC0402FR-13100KL; Power (none) -> 0.063W; Temp Range (none) -> -55°C +155°C; Tolerance (none) -> 1%
- R60: renamed from R62; footprint (none) -> Resistor_SMD:R_0402_1005Metric; Manufacturer (none) -> YAGEO; Part Number (none) -> RC0402FR-13100KL; Power (none) -> 0.063W; Temp Range (none) -> -55°C +155°C; Tolerance (none) -> 1%
- R61: renamed from R63; footprint (none) -> Resistor_SMD:R_0402_1005Metric; Manufacturer (none) -> YAGEO; Part Number (none) -> RC0402FR-13100KL; Power (none) -> 0.063W; Temp Range (none) -> -55°C +155°C; Tolerance (none) -> 1%
- R9: footprint (none) -> Resistor_SMD:R_0402_1005Metric; Manufacturer (none) -> Stackpole Electronics Inc; Part Number (none) -> RMCF0402FT10K0; Power (none) -> 0.063W; Temp Range (none) -> -55°C +155°C; Tolerance (none) -> 1%
- renumbered C47 to C46, C48 to C47, C49 to C48, C50 to C49, C51 to C50, C52 to C51, C53 to C52, C54 to C53, C55 to C54, C56 to C55, C57 to C56, D7 to D6, U6 to U5, U7 to U6, U8 to U7
Connections:
- net +3V3: now also Q13.1 (G)
- net +4V: now also Q22.2 (S)
- net +4V_SW: now also Q22.3 (D)
- net CELL_1S: now also Q12.2 (S), Q17.2 (S)
- net CELL_1S_DIS_EN: now also Q8.1 (G)
- net CELL_2S: now also Q11.2 (S), Q16.2 (S)
- net CELL_2S_DIS_EN: now also Q7.1 (G)
- net CELL_3S: now also Q10.2 (S), Q15.2 (S)
- net CELL_3S_DIS_EN: now also Q6.1 (G)
- net CELL_4S: now also Q14.2 (S), Q9.2 (S)
- net CELL_4S_DIS_EN: now also Q5.1 (G)
- net DRV_PIEZO_LHS: now also Q18.3 (D)
- net DRV_PIEZO_RHS: now also Q19.3 (D)
- net EN_HIGH_POWER: now also Q21.1 (G)
- net GND: now also Q13.2 (S), Q18.2 (S), Q19.2 (S), Q21.2 (S), Q5.2 (S), Q6.2 (S), Q7.2 (S), Q8.2 (S)
- net PWM_PIEZO_LHS: now also Q18.1 (G)
- net PWM_PIEZO_RHS: now also Q19.1 (G)
- net VBAT: now also R47.2
- net VPIEZO: now also R47.1
- net ~{CELL_1S_DIS_EN}: now also Q12.1 (G), Q8.3 (D)
- net ~{CELL_2S_DIS_EN}: now also Q11.1 (G), Q7.3 (D)
- net ~{CELL_3S_DIS_EN}: now also Q10.1 (G), Q6.3 (D)
- net ~{CELL_4S_DIS_EN}: now also Q5.3 (D), Q9.1 (G)
- net at R40.2: now also Q17.3 (D)
- net at R32.1: now also Q13.3 (D), Q14.1 (G), Q15.1 (G), Q16.1 (G), Q17.1 (G)
- net at C56.2, Q20.1 (G), R60.2: now also Q22.1 (G)
- net at R34.2: now also Q14.3 (D)
- net at R1.1, R2.1, U1.6 (ICHG/EN): now also R3.2; no longer R3.1
- net at C3.1, R4.1, U1.9 (REF): now also R3.1; no longer R3.2
- net at R38.2: now also Q16.3 (D)
- net at R30.1: now also Q11.3 (D)
- net at R59.1, R60.1: now also Q21.3 (D)
- net at R31.1: now also Q12.3 (D)
- net at R29.1: now also Q10.3 (D)
- net at R36.2: now also Q15.3 (D)
- net at R28.1: now also Q9.3 (D)
Other:
- note added: "AC/DC Adapter Current Limiting -------------------- I_{IN(MAX)}=0.1V/R_{CSS} =0.1V/22mOhms =4.55A"
- note added: "Make footprint compatible with ETQ-P5M2R0YLC"
- note added: "P=CV^{2}(f_{SW}) =(1.5e-9)(5.1^2)(600e3)=0.023"
- note removed: "0.4A"
- note removed: "AC/DC Adapter Current Limiting -------------------- I_{IN(MAX)}=0.1V/R_{CSS} =0.1V/22.6mOhms =4.43A"
- note removed: "Also purchase 412mOhm"
- note removed: "I_{out}=0.1V/R_{set} R_{set}=0.1V/0.2A ~=0.499R"
- note removed: "t_{ON}=[L(0.26)(I_{LED})]/[V_{IN}-V_{LED}-I_{LED}(R_{SET}+R_{L}+R_{SW})] =[100uH(0.26)(0.2A)]/[14.8V-9.6V-0.2A(0.5+0.1+0.2)Ohms] =1.0317uS"

Commit message: PMOS diode replacement
Parts:
- removed D3: D_Schottky_Small, symbol Device:D_Schottky_Small
- added D?: DNP, symbol Device:D_Schottky_Small
- added F9: 4A, Resistor_SMD:R_0402_1005Metric, symbol Device:Fuse_Small
- added Q1, Q?: Q_PMOS_GDS, symbol Device:Q_PMOS_GDS
- added R1: 100k, Resistor_SMD:R_0402_1005Metric, symbol Device:R_Small
- added R2: 10k, Resistor_SMD:R_0402_1005Metric, symbol Device:R_Small
- added R44, R?: 0R, Resistor_SMD:R_0402_1005Metric, symbol Device:R_Small
- added R?: 442k, Resistor_SMD:R_0402_1005Metric, symbol Device:R_Small
- D1: value D_Schottky_Small -> DNP
- renumbered C13 to C11, C11 to C12, C12 to C13, C18 to C17, C17 to C18, Q9 to Q10, Q10 to Q11, Q11 to Q12, Q12 to Q13, Q13 to Q14, Q14 to Q15, Q15 to Q16, Q16 to Q17, Q17 to Q18, Q18 to Q19, Q1 to Q2, Q19 to Q20, Q20 to Q21, Q21 to Q22, Q22 to Q23, Q2 to Q3, Q3 to Q4, Q4 to Q5, Q5 to Q6, Q6 to Q7, Q7 to Q8, Q8 to Q9, R8 to R10, R9 to R11, R10 to R12, R11 to R13, R13 to R14, R12 to R15, R14 to R16, R15 to R17, R16 to R18, R17 to R19, R18 to R20, R19 to R21, R20 to R22, R21 to R23, R22 to R24, R23 to R25, R24 to R26, R25 to R27, R26 to R28, R27 to R29, R1 to R3, R28 to R30, R29 to R31, R30 to R32, R31 to R33, R32 to R34, R33 to R35, R34 to R36, R35 to R37, R36 to R38, R37 to R39, R2 to R4, R38 to R40, R39 to R41, R40 to R42, R41 to R43, R42 to R45, R43 to R46, R44 to R47, R45 to R48, R46 to R49, R3 to R5, R47 to R50, R48 to R51, R49 to R52, R50 to R53, R51 to R54, R52 to R55, R53 to R56, R54 to R57, R55 to R58, R56 to R59, R4 to R6, R57 to R60, R58 to R61, R59 to R62, R60 to R63, R61 to R64, R5 to R7, R6 to R8, R7 to R9
Connections:
- net +19V5: now also Q1.2 (D)
- net CHG_IOUT: now also R?.2
- net GND: now also R2.2
- net SPR_PA0: now also R?.1
- net SPR_PB9: now also R44.2
- net VDC: now also Q1.3 (S), R1.2
- net VDC_METERED: now also D?.2 (A), Q?.2 (D)
- net VSYS: now also D?.1 (K), Q?.3 (S), R?.2
- net VSYS_SW: now also F9.2; no longer J1.3 (Pin_3), J3.5 (Pin_5), J7.3 (Pin_3)
- net at U3.4 (STAT): now also Q?.1 (G), R?.1
- new net: Q1.1 (G), R1.1, R2.1
- new net VSYS_SW_FUSED: F9.1, J1.3 (Pin_3), J3.5 (Pin_5), J7.3 (Pin_3)
- new net ~{19V5_PRESENT}: R44.1
Other:
- added sheet Battery (FaclonMain-Battery.kicad_sch)
- added sheet High Power 5V1 (FalconMain-HP5V1.kicad_sch)
- added sheet Low Power and Drivers (FalconMain-LPDrivers.kicad_sch)
- note added: "Charge Current Sense Output -------------------- V_{Iout}=20(R_{CSB} * I_{chg}) =20(0.068)(2.3)=3.2V C_{load} < 5nF Charge Current Set -------------------- V_{ICH-EN}=I_{CHG} * 1.3146"
- note added: "High: VSYS Low: 4.42V"
- note added: "Max Charge Current Set -------------------- R_{CSB}=0.2V(V_{ICH-EN}/V_{REF})/I_{CHG} =0.2V(3.3V/4.2V)/2.5A ~=62.6mOhms I_{CHG}=0.2V(3.3V/4.2V)/0.068Ohms=2.311A"
- note removed: "5A"
- note removed: "Charge Current Sense Output -------------------- V_{Iout}=20(R_{CSB} * I_{chg}) C_{load} < 5nF Charge Current Set -------------------- V_{ICH-EN}=I_{CHG} * 1.3146"
- note removed: "Derate polyfuses for 0-60C"
- note removed: "Max Charge Current Set -------------------- R_{CSB}=0.2V(V_{ICH-EN}/V_{REF})/I_{CHG} =0.2V(3.3V/4.2V)/2.5A ~=62.6mOhms I_{CHG}=0.2V(3.3V/4.2V)/0.0626R=2.5103A"
- note removed: "Normal fuses have undesirable Vf Poly fuses are less temperature stable"
- note removed: "TO DO ------------------------------------ / Decide if/how to do low-batt shutdown/ship-mode / Decide how to handle power ORing / Crystals / JTAG conn, USB conn / Select passive component values / Select passive component values for LP LED bucks / Map MCU inputs (need dividers for ADC) / Select LP LDO - Select HP buck regulator - Select remaining passive component values - Select passive componen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"
- company: (none) -> University of Waterloo
- title: (none) -> Project Falcon
- moved on the sheet: C1, C12, C13, C14, C15, C16, C18, C2, C21, C25, C3, C4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

Commit message: Review WIP
Parts:
- removed C2: 10uF, Capacitor_SMD:C_1210_3225Metric, symbol Device:C_Small
- removed R44, R?: 0R, Resistor_SMD:R_0402_1005Metric, symbol Device:R_Small
- removed R62: 100k, Resistor_SMD:R_0402_1005Metric, symbol Device:R_Small
- added C?: 100uF, Capacitor_THT:CP_Radial_D8.0mm_P3.50mm, symbol Device:C_Polarized_Small
- added D?: DNP, symbol Device:D_Schottky_Small
- added Q? (x2): Q_PMOS_GDS, symbol Device:Q_PMOS_GDS
- added R38: DNP, Resistor_SMD:R_0402_1005Metric, symbol Device:R_Small
- added R39, R66: 49.9k, Resistor_SMD:R_0402_1005Metric, symbol Device:R_Small
- added R4, R?: 0R, Resistor_SMD:R_0402_1005Metric, symbol Device:R_Small
- added R40: 80.6k, Resistor_SMD:R_0402_1005Metric, symbol Device:R_Small
- added R69: 2k, Resistor_SMD:R_0402_1005Metric, symbol Device:R_Small
- added R?: 442k, Resistor_SMD:R_0402_1005Metric, symbol Device:R_Small
- added U?: LTC4412ES6#TRPBF, symbol JetkovKiCADLib:LTC4412ES6#TRPBF
- Q1, Q2, Q5: Voltage (none) -> 20Vgs/30Vds/3Vth
- Q10: renamed from Q9; Voltage 20Vgs/60Vds -> 20Vgs/60Vds/1Vth
- Q11: renamed from Q10; Voltage 20Vgs/30Vds -> 20Vgs/30Vds/2.5Vth
- Q12: renamed from Q11; Voltage 20Vgs/30Vds -> 20Vgs/30Vds/2.5Vth
- Q13: renamed from Q12; Voltage 20Vgs/30Vds -> 20Vgs/30Vds/2.5Vth
- Q14: renamed from Q13; Voltage 20Vgs/30Vds -> 20Vgs/30Vds/2.5Vth
- Q15: renamed from Q14; Voltage 20Vgs/60Vds -> 20Vgs/60Vds/1Vth
- Q16: renamed from Q15; Voltage 20Vgs/30Vds -> 20Vgs/30Vds/2.5Vth
- Q17: renamed from Q16; Voltage 20Vgs/30Vds -> 20Vgs/30Vds/2.5Vth
- Q18: renamed from Q17; Voltage 20Vgs/30Vds -> 20Vgs/30Vds/2.5Vth
- Q19: renamed from Q18; Voltage 20Vgs/30Vds -> 20Vgs/30Vds/2.5Vth
- Q20: renamed from Q19; Voltage 20Vgs/60Vds -> 20Vgs/60Vds/1Vth
- Q21: renamed from Q20; Voltage 20Vgs/60Vds -> 20Vgs/60Vds/1Vth
- Q22: renamed from Q21; Voltage (none) -> 20Vgs/30Vds/3Vth
- Q23: renamed from Q22; Voltage 20Vgs/60Vds -> 20Vgs/60Vds/1Vth
- Q24: renamed from Q23; Voltage 20Vgs/30Vds -> 20Vgs/30Vds/2.5Vth
- Q6: renamed from Q?; Voltage (none) -> 20Vgs/30Vds/3Vth
- Q7: renamed from Q6; Voltage 20Vgs/60Vds -> 20Vgs/60Vds/1Vth
- Q8: renamed from Q7; Voltage 20Vgs/60Vds -> 20Vgs/60Vds/1Vth
- Q9: renamed from Q8; Voltage 20Vgs/60Vds -> 20Vgs/60Vds/1Vth
- R1: value 100k -> 1M; Manufacturer YAGEO -> Stackpole Electronics Inc; Part Number RC0402FR-13100KL -> RMCF0402FT1M00
- R2: value 10k -> 100k; Manufacturer Stackpole Electronics Inc -> YAGEO; Part Number RMCF0402FT10K0 -> RC0402FR-13100KL
- gave numbers to parts that had none: 2
- renumbered C11 to C10, C12 to C11, C13 to C12, C14 to C13, C15 to C14, C16 to C15, C17 to C16, C18 to C17, C19 to C18, C20 to C19, C4 to C2, C21 to C20, C22 to C21, C23 to C22, C24 to C23, C25 to C24, C26 to C25, C27 to C26, C28 to C27, C29 to C28, C30 to C29, C5 to C3, C31 to C30, C32 to C31, C33 to C32, C34 to C33, C35 to C34, C36 to C35, C37 to C36, C38 to C37, C39 to C38, C41 to C39, C3 to C4, C42 to C40, C43 to C41, C44 to C42, C40 to C43, C45 to C44, C46 to C45, C47 to C46, C48 to C47, C49 to C48, C50 to C49, C6 to C5, C51 to C50, C52 to C51, C53 to C52, C54 to C53, C55 to C54, C56 to C55, C7 to C6, C8 to C7, C9 to C8, C10 to C9, R9 to R10, R10 to R11, R11 to R12, R12 to R13, R13 to R14, R14 to R15, R15 to R16, R16 to R17, R17 to R19, R19 to R20, R20 to R22, R21 to R23, R22 to R24, R23 to R25, R24 to R26, R25 to R27, R26 to R28, R27 to R29, R28 to R30, R29 to R31, R30 to R32, R31 to R33, R32 to R34, R33 to R35, R34 to R36, R35 to R37, R36 to R41, R37 to R42, R38 to R43, R39 to R44, R40 to R45, R41 to R46, R42 to R47, R43 to R48, R45 to R49, R4 to R5, R46 to R50, R47 to R51, R48 to R52, R49 to R53, R50 to R54, R51 to R55, R52 to R56, R53 to R57, R54 to R58, R55 to R59, R5 to R6, R56 to R60, R57 to R61, R58 to R62, R59 to R63, R60 to R64, R61 to R65, R63 to R67, R64 to R68, R6 to R7, R7 to R8, R8 to R9
Connections:
- net CELL_1S_ADC is gone; now on net VSENSE_CELL_1S: C42.1, R47.1, R48.2
- net CELL_1S_DIS_EN is gone; now on net EN_CELL_1S_DIS: Q10.1 (G), R27.2
- net CELL_2S_ADC is gone; now on net VSENSE_CELL_2S: C41.1, R45.1, R46.2
- net CELL_2S_DIS_EN is gone; now on net EN_CELL_2S_DIS: Q9.1 (G), R26.2
- net CELL_3S_ADC is gone; now on net VSENSE_CELL_3S: C40.1, R43.1, R44.2
- net CELL_3S_DIS_EN is gone; now on net EN_CELL_3S_DIS: Q8.1 (G), R25.2
- net CELL_4S_ADC is gone; now on net VSENSE_CELL_4S: C39.1, R41.1, R42.2
- net CELL_4S_DIS_EN is gone; now on net EN_CELL_4S_DIS: Q7.1 (G), R24.2
- net ~{CHG_EN} is gone; now on net VSET_ICHG: R5.2
- net +19V5: now also D?.2 (A), Q?.2 (D)
- net +3V3: no longer Q15.1 (G), R37.2, U4.29 (PA8)
- net +5V1: now also R39.1
- net CHG_IOUT: now also U4.10 (PA0-WKUP1), R4.2; no longer U1.7 (IOUT)
- net GND: now also R2.1, C?.2, R40.1, R?.1, U?.2 (GND); no longer R2.2
- net VBAT: now also Q?.2 (D), U?.1 (VIN)
- net VDC: now also C?.1, D?.1 (K), Q?.3 (S), Q?.3 (S), R?.2, U?.6 (SENSE)
- net VSENSE_5V1: now also J6.15 (Pin_15), R38.1, R39.2, R40.2
- net VSYS: now also R66.1
- net VSYS_SW: now also R38.2
- net at Q1.1 (G), R1.1: now also R2.2; no longer R2.1
- net at R67.1: now also R66.2, R69.1; no longer Q23.3 (D)
- removed net SPR_PA0: J6.15 (Pin_15), U4.10 (PA0-WKUP1)
- net ~{CELL_1S_DIS_EN} renamed ~{EN_CELL_1S_DIS}
- net ~{CELL_2S_DIS_EN} renamed ~{EN_CELL_2S_DIS}
- net ~{CELL_3S_DIS_EN} renamed ~{EN_CELL_3S_DIS}
- net ~{CELL_4S_DIS_EN} renamed ~{EN_CELL_4S_DIS}
- new net: Q?.1 (G), R?.1, U?.4 (STAT)
- new net: R4.1, U1.7 (IOUT)
- new net: Q23.3 (D), R69.2
- new net: Q?.1 (G), U?.5 (GATE)
- new net: R?.2, U?.3 (CTL)
- new net EN_CELL_SENSE: Q15.1 (G), R37.2, U4.29 (PA8)
Other:
- note added: "Can we just use the one ideal diode controller here?"
- note added: "Checklist -------- - No MOSFET gate is ever floating wrt. source - No MOSFET voltage rating exceeded - No capacitor voltage rating exceeded - Symbol pins correspond to package pins - Symbol/package pins correspond to footprint pins - Resistor wattage rating not exceeded - Diodes do not dissipate excessive heat - Unintentional wire junctions - Check MCU pins support functions - No MCU pin is be po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"
- note added: "DNP divider to use AIN0 as spare"
- note added: "Heatsink"
- note added: "High: VSYS Low: VSYS-4.42V"
- note added: "LV PMOS will turn on after HV, and turn off before HV"
- note added: "MLCC @19V C=6uF"
- note added: "Note: Measured voltage may be 50mV lower than true if measured while a discharge FET is conducting (due to parasitic fuse, etc. resistance)"
- note added: "charger"
- note removed: "AIN0"
- note removed: "High: VSYS Low: 4.42V"
- note removed: "LV PMOS will turn on later and turn off earlier than HV"
- note removed: "MLCCC @19V C=6uF"
- note removed: "Note: Measured voltage may be 50mV lower than true if measured while a discharge FET is conducting (due to parasitic resistance)"
- note removed: "Use murata or TDK for capacitors Beware of DC bias NOTE CAPCITOR VOLTAGE RATINGS Get some 20W resistors for load testing"
- moved on the sheet: C24, C39, C4, C40, C41, C42, D3, Q15, Q16, Q17, Q18, Q19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
