File: faclon-main/FalconMain/FalconMain.kicad_pcb (KiCad board)
At the start: 2 copper layers, 181 parts, among them J1 Nano-Fit, J2 PTH, J3 Nano-Fit, J4 100mil, J5 Nano-Fit, J6 100mil, J7 Nano-Fit, J8 DNP, J9 JST-XH, Q1 Q_PMOS_LFPAK, Q10 Q_PMOS_GSD, Q11 Q_PMOS_GSD, Q12 Q_PMOS_GSD, Q13 Q_PMOS_GSD, Q14 Q_NMOS_GSD, Q15 Q_PMOS_GSD, Q16 Q_PMOS_GSD, Q17 Q_PMOS_GSD, Q18 Q_PMOS_GSD, Q19 Q_NMOS_GSD, Q2 Q_NMOS_LFPAK, Q20 Q_NMOS_GSD, Q21 Q_PMOS_LFPAK, Q22 Q_NMOS_GSD, Q23 Q_PMOS_GSD, Q3 Q_NMOS_LFPAK, Q4 Q_PMOS_LFPAK, Q5 Q_PMOS_LFPAK, Q6 Q_NMOS_GSD, Q7 Q_NMOS_GSD, Q8 Q_NMOS_GSD, Q9 Q_NMOS_GSD, U1 MAX1873TEEE+, U2 ADP1883ARMZ-0.6-R7, U3 LTC4412ES6#TRPBF, U4 STM32L152CBT6, U5 BD9E104FJ-E2, U6 AL8843QSP-13, U7 NCP164ASN330T1G, Y1 8MHz, Y2 32.768kHz

Commit message: Reorganize
Parts:
- removed the C1 at (12.9, 66.7)
- removed the C10 at (-92.0, 48.2)
- removed the C11 at (-36.8, 147.5)
- removed the C12 at (13.4, 79.1)
- removed the C2 at (-65.3, 171.2)
- removed the C3 at (-41.5, 169.0)
- removed the C4 at (-33.6, 149.6)
- removed the C5 at (10.9, 81.0)
- removed the C6 at (24.5, 58.5)
- removed the C7 at (21.6, 72.3)
- removed the C8 at (-127.5, 57.3)
- removed the C9 at (4.14, 89.6)
- removed the L1 at (-75.2, 159.1)
- removed the R1 at (18.7, 72.6)
- removed the R2 at (15.8, 72.6)
- removed the R3 at (-9.77, 94.3)
- removed the R4 at (-4.53, 90.6)
- removed the R5 at (-38.6, 151.5)
- removed the U1 at (-45.2, 156.4)
- added C24: 47nF, Capacitor_SMD:C_0402_1005Metric, F.Cu at (-88.2, 54.1)
- added C25: 33uF, Capacitor_THT:CP_Radial_D6.3mm_P2.50mm, F.Cu at (-99.9, 45.8)
- added C27: 1nF, Capacitor_SMD:C_0402_1005Metric, F.Cu at (-82.3, 48.0)
- added C29: 100nF, Capacitor_SMD:C_0402_1005Metric, F.Cu at (-19.6, 37.2)
- added C31: 10uF, Capacitor_SMD:C_1210_3225Metric, F.Cu at (-46.2, 47.2)
- added C32: 10uF, Capacitor_SMD:C_1210_3225Metric, F.Cu at (-33.9, 31.6)
- added C34: 1uF, Capacitor_SMD:C_0603_1608Metric, F.Cu at (-32.8, 44.9)
- added C36: 100nF, Capacitor_SMD:C_0402_1005Metric, F.Cu at (-22.5, 39.3)
- added C37: 10nF, Capacitor_SMD:C_0402_1005Metric, F.Cu at (-29.4, 46.2)
- added C38: 510pF, Capacitor_SMD:C_0402_1005Metric, F.Cu at (-22.5, 37.4)
- added C43: 10uF, Capacitor_SMD:C_1210_3225Metric, F.Cu at (-28.1, 70.5)
- added C44: 10uF, Capacitor_SMD:C_1210_3225Metric, F.Cu at (-19.4, 62.0)
- added L3: 10uH, Inductor_SMD:L_1008_2520Metric, F.Cu at (-28.6, 31.6)
- added R13: 47R, Resistor_SMD:R_2512_6332Metric, F.Cu at (-88.9, 25.4)
- added R47: 44.2k, Resistor_SMD:R_0402_1005Metric, F.Cu at (-16.4, 31.6)
- added R48: 2k, Resistor_SMD:R_0402_1005Metric, F.Cu at (-41.9, 48.9)
- added R49: 100k, Resistor_SMD:R_0402_1005Metric, F.Cu at (-13.5, 29.6)
- added R50: 0R, Resistor_SMD:R_0402_1005Metric, F.Cu at (-16.4, 29.6)
- added U4: BD9E104FJ-E2, JetkovKiCADLib:8-SOIC_8-SOP-J_ROHM, F.Cu at (-24.1, 26.4)
- C13: value 47nF -> 220nF; footprint Capacitor_SMD:C_0402_1005Metric -> Capacitor_SMD:C_0603_1608Metric
- C14: value 47nF -> 100uF; footprint Capacitor_SMD:C_0402_1005Metric -> Capacitor_THT:CP_Radial_D8.0mm_P3.50mm
- C15: value 1nF -> 1uF; footprint Capacitor_SMD:C_0402_1005Metric -> Capacitor_SMD:C_0603_1608Metric
- C16: value 10uF -> 220nF; footprint Capacitor_SMD:C_1210_3225Metric -> Capacitor_SMD:C_0603_1608Metric
- C17, C19: value 100nF -> 10nF
- C20: value 100uF -> 1uF; footprint Capacitor_THT:CP_Radial_D8.0mm_P3.50mm -> Capacitor_SMD:C_0603_1608Metric
- C21: value 33uF -> 47nF; footprint Capacitor_THT:CP_Radial_D6.3mm_P2.50mm -> Capacitor_SMD:C_0402_1005Metric
- C22: value 10uF -> 1uF; footprint Capacitor_SMD:C_1210_3225Metric -> Capacitor_SMD:C_0603_1608Metric
- C23: value 1.5nF -> 1uF; footprint Capacitor_SMD:C_0402_1005Metric -> Capacitor_SMD:C_0603_1608Metric
- C26: value 47uF -> 100nF; footprint Capacitor_SMD:C_1210_3225Metric -> Capacitor_SMD:C_0402_1005Metric
- C28, C33: value 47uF -> 1uF; footprint Capacitor_SMD:C_1210_3225Metric -> Capacitor_SMD:C_0603_1608Metric
- C30: value 47uF -> 12pF; footprint Capacitor_SMD:C_1210_3225Metric -> Capacitor_SMD:C_0402_1005Metric
- C35: value DNP -> 10uF; footprint Capacitor_THT:CP_Radial_D8.0mm_P3.50mm -> Capacitor_SMD:C_1210_3225Metric
- C39, C41, C42: value 1uF -> 10uF; footprint Capacitor_SMD:C_0603_1608Metric -> Capacitor_SMD:C_1210_3225Metric
- C40, C53: value 1uF -> 100uF; footprint Capacitor_SMD:C_0603_1608Metric -> Capacitor_THT:CP_Radial_D8.0mm_P3.50mm
- C45: value 10uF -> 100nF; footprint Capacitor_SMD:C_1210_3225Metric -> Capacitor_SMD:C_0402_1005Metric
- C46: value 100nF -> 1uF; footprint Capacitor_SMD:C_0402_1005Metric -> Capacitor_SMD:C_0603_1608Metric
- C49: value 12pF -> 47uF; footprint Capacitor_SMD:C_0402_1005Metric -> Capacitor_SMD:C_1210_3225Metric
- C50, C51, C52: value 10uF -> 47uF
- C54: value 1uF -> 51pF; footprint Capacitor_SMD:C_0603_1608Metric -> Capacitor_SMD:C_0402_1005Metric
- C55: value 10nF -> 1.5nF
- L2: value 2.0uH -> 22uH; footprint JetkovKiCADLib:WE-HCI_1365_7443551 -> JetkovKiCADLib:DR125-220-R_Handsolder
- L4: value 10uH -> 47uH; footprint Inductor_SMD:L_1008_2520Metric -> JetkovKiCADLib:AMDLA1306S
- L5: value 47uH -> 2.0uH; footprint JetkovKiCADLib:AMDLA1306S -> JetkovKiCADLib:WE-HCI_1365_7443551
- Q1, Q4: value Q_PMOS_LFPAK -> Q_PMOS_GSD; footprint JetkovKiCADLib:LFPACK56-S08_SOT669_NXP -> JetkovKiCADLib:SC-96_TSMT3_ROM
- Q10, Q13: value Q_PMOS_GSD -> Q_NMOS_GSD; footprint JetkovKiCADLib:SC-96_TSMT3_ROM -> JetkovKiCADLib:SOT-323_SC-70
- Q15, Q16, Q17: value Q_PMOS_GSD -> Q_PMOS_LFPAK; footprint JetkovKiCADLib:SC-96_TSMT3_ROM -> JetkovKiCADLib:LFPACK56-S08_SOT669_NXP
- Q2: value Q_NMOS_LFPAK -> Q_PMOS_GSD; footprint JetkovKiCADLib:LFPACK56-S08_SOT669_NXP -> JetkovKiCADLib:SC-96_TSMT3_ROM
- Q21: value Q_PMOS_LFPAK -> Q_NMOS_GSD; footprint JetkovKiCADLib:LFPACK56-S08_SOT669_NXP -> JetkovKiCADLib:SOT-323_SC-70
- Q22: value Q_NMOS_GSD -> Q_NMOS_LFPAK; footprint JetkovKiCADLib:SOT-323_SC-70 -> JetkovKiCADLib:LFPACK56-S08_SOT669_NXP
- Q23: value Q_PMOS_GSD -> Q_NMOS_LFPAK; footprint JetkovKiCADLib:SC-96_TSMT3_ROM -> JetkovKiCADLib:LFPACK56-S08_SOT669_NXP
- Q3: value Q_NMOS_LFPAK -> Q_NMOS_GSD; footprint JetkovKiCADLib:LFPACK56-S08_SOT669_NXP -> JetkovKiCADLib:SOT-323_SC-70
- Q6, Q8, Q9: value Q_NMOS_GSD -> Q_PMOS_GSD; footprint JetkovKiCADLib:SOT-323_SC-70 -> JetkovKiCADLib:SC-96_TSMT3_ROM
- R10: value 10k -> 4.7R
- R11: value 22m -> 4.7R; footprint Resistor_SMD:R_1206_3216Metric -> Resistor_SMD:R_0402_1005Metric
- R12: value 4.7R -> 49.9k
- R14: value 68m -> 100k; footprint Resistor_SMD:R_0612_1632Metric -> Resistor_SMD:R_0402_1005Metric
- R15: value 0R -> 100k
- R16: value 0R -> 154k
- R17, R26, R34, R61: value 100k -> 49.9k
- R18: value 2R -> 0R
- R19: value 442k -> 47R; footprint Resistor_SMD:R_0402_1005Metric -> Resistor_SMD:R_2512_6332Metric
- R20: value 80.6k -> 0R
- R21: value 15k -> 100k
- R22: value 100k -> 68m; footprint Resistor_SMD:R_0402_1005Metric -> Resistor_SMD:R_0612_1632Metric
- R24: value 100k -> 86.6k
- R25: value 100k -> DNP
- R28: value 100k -> 47R; footprint Resistor_SMD:R_0402_1005Metric -> Resistor_SMD:R_2512_6332Metric
- R29, R35: value 100k -> 133k
- R30, R33: value 47R -> 100k; footprint Resistor_SMD:R_2512_6332Metric -> Resistor_SMD:R_0402_1005Metric
- R31: value 47R -> 10k; footprint Resistor_SMD:R_2512_6332Metric -> Resistor_SMD:R_0402_1005Metric
- R32: value 47R -> 49.9k; footprint Resistor_SMD:R_2512_6332Metric -> Resistor_SMD:R_0402_1005Metric
- R36: value DNP -> 47R; footprint Resistor_SMD:R_0402_1005Metric -> Resistor_SMD:R_2512_6332Metric
- R37, R44, R6: value 49.9k -> 100k
- R38: value 80.6k -> 100k
- R39: value 221k -> 442k
- R40: value 49.9k -> 0R
- R41: value 154k -> 442k
- R42: value 49.9k -> 402k
- R43: value 86.6k -> 100k
- R46: value 133k -> 100k
- R51: value 0R -> DNP
- R52: value DNP -> 2k
- R53: value 442k -> 39m; footprint Resistor_SMD:R_0402_1005Metric -> Resistor_SMD:R_1206_3216Metric
- R55: value 100k -> 1M
- R56: value 100k -> 2k
- R57: value 2k -> 100k
- R58: value 2k -> 0R
- R59: value 44.2k -> 0R
- R60: value 402k -> DNP
- R62: value 1M -> 2R
- R63: value 39m -> 80.6k; footprint Resistor_SMD:R_1206_3216Metric -> Resistor_SMD:R_0402_1005Metric
- R64: value 49.9k -> 80.6k
- R65: value 100k -> 27.4k
- R67: value 2k -> 15k
- R7: value 0R -> 221k
- R8: value 27.4k -> 100k
- R9: value 4.7R -> 22m; footprint Resistor_SMD:R_0402_1005Metric -> Resistor_SMD:R_1206_3216Metric
- U2: value ADP1883ARMZ-0.6-R7 -> MAX1873TEEE+; footprint JetkovKiCADLib:10-MSOP_RM-10_AD -> JetkovKiCADLib:16-SSOP_16-QSOP_MAX
- U5: value BD9E104FJ-E2 -> NCP164ASN330T1G; footprint JetkovKiCADLib:8-SOIC_8-SOP-J_ROHM -> JetkovKiCADLib:SOT-23-5_TSOP−5_ON
- U7: value NCP164ASN330T1G -> ADP1883ARMZ-0.6-R7; footprint JetkovKiCADLib:SOT-23-5_TSOP−5_ON -> JetkovKiCADLib:10-MSOP_RM-10_AD
- moved Q15 181.8 mm to (-80.5, 26.4)
- moved R40 169.2 mm to (-74.0, 32.9)
- moved R22 162.7 mm to (-92.7, 48.8)
- moved R35 162.3 mm to (-78.9, 40.4)
- moved R31 160.6 mm to (-66.3, 26.5)
- moved R32 158.1 mm to (-70.8, 35.0)
- moved Q18 157.9 mm to (-17.7, 25.6)
- moved R53 156.8 mm to (-33.9, 35.4)
- moved R30 155.8 mm to (-91.4, 52.3)
- moved Q16 153.8 mm to (-89.2, 31.3)
- moved R29 151.6 mm to (-67.1, 29.0)
- moved R19 150.7 mm to (-115.7, 47.5)
- moved Q4 149.5 mm to (-82.1, 32.2)
- moved R28 148.6 mm to (-115.7, 52.4)
- moved R43 148.2 mm to (-10.1, 25.9)
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- renumbered C43 to C1, C32 to C10, C34 to C11, C36 to C12, C27 to C2, C31 to C3, C37 to C4, C38 to C5, C44 to C6, C24 to C7, C25 to C8, C29 to C9, F4 to F1, F5 to F2, F1 to F3, F6 to F4, F7 to F5, F9 to F6, F2 to F7, F3 to F8, F8 to F9, J2 to J1, J9 to J2, J6 to J3, J8 to J5, J5 to J6, J1 to J7, J7 to J8, J3 to J9, L3 to L1, R47 to R1, R48 to R2, R49 to R3, R50 to R4, R13 to R5, U4 to U1
Connections:
- C13 pad 1: GND -> VDC
- C13 pad 2: Net-(C13-Pad2) -> GND
- C14 pad 1: GND -> VSYS
- C14 pad 2: Net-(C14-Pad2) -> GND
- C15 pad 1: GND -> VSENSE_CELL_4S
- C15 pad 2: Net-(C15-Pad2) -> GND
- C16 pad 1: GND -> Net-(C16-Pad1)
- C16 pad 2: VSYS_SW -> VDC
- C17 pad 1: GND -> Net-(C17-Pad1)
- C17 pad 2: Net-(C17-Pad2) -> GND
- C18 pad 2: VSYS_SW -> Net-(C18-Pad2)
- C19 pad 2: Net-(C19-Pad2) -> GND
- C20 pad 1: VSYS -> VSENSE_CELL_3S
- C21 pad 1: VBAT -> GND
- C21 pad 2: GND -> Net-(C21-Pad2)
- C22 pad 1: GND -> VSENSE_CELL_2S
- C22 pad 2: VSYS_SW -> GND
- C26 pad 1: +5V1 -> GND
- C26 pad 2: GND -> Net-(C26-Pad2)
- C28 pad 1: +5V1 -> VSENSE_CELL_1S
- C30 pad 1: +5V1 -> +4V
- C30 pad 2: GND -> Net-(C30-Pad2)
- C33 pad 1: +5V1 -> GND
- C33 pad 2: GND -> +4V
- C35 pad 1: +5V1 -> GND
- C35 pad 2: GND -> VSYS
- C39 pad 1: VSENSE_CELL_4S -> GND
- C39 pad 2: GND -> VSYS_SW
- C40 pad 1: VSENSE_CELL_3S -> VSYS_SW
- C41 pad 1: VSENSE_CELL_2S -> GND
- C41 pad 2: GND -> VSYS_SW
- C42 pad 1: VSENSE_CELL_1S -> GND
- C42 pad 2: GND -> VSYS_SW
- C45 pad 2: VSYS -> Net-(C45-Pad2)
- C46 pad 1: GND -> Net-(C45-Pad2)
- C46 pad 2: VSYS -> GND
- C49 pad 1: +4V -> +5V1
- C49 pad 2: Net-(C49-Pad2) -> GND
- C50 pad 1: GND -> +5V1
- C50 pad 2: VSYS_SW -> GND
- C51 pad 1: GND -> +5V1
- C51 pad 2: +4V -> GND
- C52 pad 1: GND -> +5V1
- C52 pad 2: +4V -> GND
- C53 pad 1: GND -> +5V1
- C53 pad 2: +4V -> GND
- C54 pad 2: +3V3 -> Net-(C48-Pad1)
- C55 pad 1: VSYS -> Net-(C55-Pad1)
- C55 pad 2: Net-(C55-Pad2) -> GND
- D1 pad 1: Net-(D1-Pad1) -> GND
- D1 pad 3: (no net) -> Net-(D1-Pad3)
- D2 pad 2: EN_4V -> +19V5
- D3 pad 2: +19V5 -> EN_4V
- D4 pad 1: VSYS_SW -> Net-(D4-Pad1)
- D4 pad 2: Net-(D4-Pad2) -> Net-(D4-Pad1)
- D4 pad 3: (no net) -> VSYS_SW
- L2 pad 1: Net-(C19-Pad2) -> Net-(D1-Pad3)
- L2 pad 2: +5V1 -> Net-(L2-Pad2)
- L4 pad 1: Net-(C47-Pad2) -> Net-(D4-Pad1)
- L4 pad 2: +4V -> /Low Power and Drivers/FRONT_LED_N
- L5 pad 1: Net-(D4-Pad2) -> Net-(C47-Pad2)
- L5 pad 2: /FRONT_LED_N -> +5V1
- Q1 pad 1: VSYS -> Net-(Q1-Pad1)
- Q1 pad 2: VSYS -> /Battery/CELL_4S
- Q1 pad 3: VSYS -> Net-(Q1-Pad3)
- Q10 pad 1: /~{EN_CELL_4S_DIS} -> EN_CELL_2S_DIS
- Q10 pad 2: /CELL_4S -> GND
- Q10 pad 3: Net-(Q10-Pad3) -> /Battery/~{EN_CELL_2S_DIS}
- Q11 pad 1: /~{EN_CELL_3S_DIS} -> Net-(Q1-Pad1)
- Q11 pad 2: /CELL_3S -> /Battery/CELL_1S
- Q12 pad 1: /~{EN_CELL_2S_DIS} -> /Battery/~{EN_CELL_1S_DIS}
- Q12 pad 2: /CELL_2S -> /Battery/CELL_1S
- Q13 pad 1: /~{EN_CELL_1S_DIS} -> EN_CELL_1S_DIS
- Q13 pad 2: /CELL_1S -> GND
- Q13 pad 3: Net-(Q13-Pad3) -> /Battery/~{EN_CELL_1S_DIS}
- Q14 pad 3: Net-(Q14-Pad3) -> Net-(Q1-Pad1)
- Q15 pad 1: Net-(Q14-Pad3) -> VDC
- Q15 pad 2: /CELL_4S -> VDC
- Q15 pad 3: Net-(Q15-Pad3) -> VDC
- Q16 pad 1: Net-(Q14-Pad3) -> VDC
- Q16 pad 2: /CELL_3S -> VDC
- Q16 pad 3: Net-(Q16-Pad3) -> VDC
- Q17 pad 1: Net-(Q14-Pad3) -> VSYS
- Q17 pad 2: /CELL_2S -> VSYS
- Q17 pad 3: Net-(Q17-Pad3) -> VSYS
- Q18 pad 1: Net-(Q14-Pad3) -> Net-(C37-Pad2)
- Q18 pad 2: /CELL_1S -> +4V
- Q18 pad 3: Net-(Q18-Pad3) -> +4V_SW
- Q19 pad 1: PWM_PIEZO_LHS -> EN_HIGH_POWER
- Q19 pad 3: DRV_PIEZO_LHS -> Net-(Q19-Pad3)
- Q2 pad 1: Net-(C19-Pad2) -> /Battery/~{EN_CELL_4S_DIS}
- Q2 pad 2: Net-(C19-Pad2) -> /Battery/CELL_4S
- Q2 pad 3: Net-(C19-Pad2) -> Net-(Q2-Pad3)
- Q20 pad 1: PWM_PIEZO_RHS -> PWM_PIEZO_LHS
- Q20 pad 3: DRV_PIEZO_RHS -> DRV_PIEZO_LHS
- Q21 pad 1: VSYS -> PWM_PIEZO_RHS
- Q21 pad 2: VSYS -> GND
- Q21 pad 3: VSYS -> DRV_PIEZO_RHS
- Q22 pad 1: EN_HIGH_POWER -> Net-(C47-Pad2)
- Q22 pad 2: GND -> Net-(C47-Pad2)
- Q22 pad 3: Net-(Q22-Pad3) -> Net-(C47-Pad2)
- Q23 pad 1: Net-(C55-Pad2) -> GND
- Q23 pad 2: +4V -> GND
- Q23 pad 3: +4V_SW -> GND
- Q3 pad 1: GND -> EN_CELL_4S_DIS
- Q3 pad 3: GND -> /Battery/~{EN_CELL_4S_DIS}
- Q4 pad 1: VDC -> Net-(Q1-Pad1)
- Q4 pad 2: VDC -> /Battery/CELL_3S
- Q4 pad 3: VDC -> Net-(Q4-Pad3)
- Q5 pad 1: VDC -> VSYS
- Q5 pad 2: VDC -> VSYS
- Q5 pad 3: VDC -> VSYS
- Q5 pad 5: +19V5 -> Net-(D1-Pad3)
- Q6 pad 1: EN_CELL_4S_DIS -> /Battery/~{EN_CELL_3S_DIS}
- Q6 pad 2: GND -> /Battery/CELL_3S
- Q6 pad 3: /~{EN_CELL_4S_DIS} -> Net-(Q6-Pad3)
- Q7 pad 3: /~{EN_CELL_3S_DIS} -> /Battery/~{EN_CELL_3S_DIS}
- Q8 pad 1: EN_CELL_2S_DIS -> Net-(Q1-Pad1)
- Q8 pad 2: GND -> /Battery/CELL_2S
- Q8 pad 3: /~{EN_CELL_2S_DIS} -> Net-(Q8-Pad3)
- Q9 pad 1: EN_CELL_1S_DIS -> /Battery/~{EN_CELL_2S_DIS}
- Q9 pad 2: GND -> /Battery/CELL_2S
- Q9 pad 3: /~{EN_CELL_1S_DIS} -> Net-(Q9-Pad3)
- R10 pad 1: Net-(C17-Pad2) -> VDC
- R10 pad 2: Net-(C15-Pad2) -> Net-(C17-Pad1)
- R11 pad 1: VDC -> VSYS
- R11 pad 2: VSYS -> Net-(C19-Pad1)
- R12 pad 1: VSYS -> GND
- R12 pad 2: Net-(C12-Pad1) (its old number) -> VSENSE_CELL_4S
- R14 pad 1: VBAT -> GND
- R14 pad 2: Net-(L1-Pad2) -> EN_CELL_4S_DIS
- R15 pad 1: Net-(Q2-Pad4) -> /Battery/~{EN_CELL_3S_DIS}
- R15 pad 2: Net-(R15-Pad2) -> /Battery/CELL_3S
- R16 pad 1: GND -> VSENSE_CELL_3S
- R16 pad 2: Net-(R16-Pad2) -> Net-(Q4-Pad3)
- R17 pad 2: Net-(Q3-Pad4) -> VSENSE_CELL_3S
- R18 pad 1: Net-(C23-Pad1) -> Net-(R18-Pad1)
- R18 pad 2: Net-(C19-Pad2) -> CHG_IOUT
- R19 pad 1: Net-(Q5-Pad4) -> Net-(Q6-Pad3)
- R19 pad 2: VDC -> /Battery/CELL_2S
- R20 pad 2: +5V1 -> VSET_ICHG
- R21 pad 2: Net-(R20-Pad1) -> EN_CELL_3S_DIS
- R22 pad 1: GND -> VBAT
- R22 pad 2: EN_CELL_4S_DIS -> Net-(L2-Pad2)
- R23 pad 1: GND -> /Battery/~{EN_CELL_2S_DIS}
- R23 pad 2: EN_CELL_3S_DIS -> /Battery/CELL_2S
- R24 pad 1: GND -> VSENSE_CELL_2S
- R24 pad 2: EN_CELL_2S_DIS -> Net-(Q8-Pad3)
- R25 pad 1: GND -> Net-(C23-Pad1)
- R25 pad 2: EN_CELL_1S_DIS -> Net-(R20-Pad1)
- R26 pad 1: /~{EN_CELL_4S_DIS} -> GND
- R26 pad 2: /CELL_4S -> VSENSE_CELL_2S
- R27 pad 1: /~{EN_CELL_3S_DIS} -> Net-(R20-Pad1)
- R27 pad 2: /CELL_3S -> GND
- R28 pad 1: /~{EN_CELL_2S_DIS} -> Net-(Q9-Pad3)
- R28 pad 2: /CELL_2S -> /Battery/CELL_1S
- R29 pad 1: /~{EN_CELL_1S_DIS} -> Net-(C23-Pad1)
- R29 pad 2: /CELL_1S -> Net-(R29-Pad2)
- R30 pad 1: Net-(Q10-Pad3) -> GND
- R30 pad 2: /CELL_3S -> EN_CELL_2S_DIS
- R31 pad 1: Net-(Q11-Pad3) -> Net-(C26-Pad2)
- R31 pad 2: /CELL_2S -> Net-(C27-Pad2)
- R32 pad 1: Net-(Q12-Pad3) -> Net-(R29-Pad2)
- R32 pad 2: /CELL_1S -> GND
- R33 pad 1: Net-(Q13-Pad3) -> /Battery/~{EN_CELL_1S_DIS}
- R33 pad 2: GND -> /Battery/CELL_1S
- R34 pad 1: Net-(Q14-Pad3) -> VSENSE_CELL_1S
- R34 pad 2: /CELL_4S -> Net-(Q11-Pad3)
- R35 pad 2: EN_CELL_SENSE -> VSENSE_CELL_1S
- R36 pad 1: VSENSE_5V1 -> Net-(Q12-Pad3)
- R36 pad 2: VSYS_SW -> GND
- R37 pad 1: +5V1 -> GND
- R37 pad 2: VSENSE_5V1 -> EN_CELL_1S_DIS
- R38 pad 2: VSENSE_5V1 -> EN_CELL_SENSE
- R39 pad 1: VSENSE_CELL_4S -> Net-(Q15-Pad4)
- R39 pad 2: Net-(Q15-Pad3) -> VDC
- R40 pad 2: VSENSE_CELL_4S -> Net-(R40-Pad2)
- R41 pad 1: VSENSE_CELL_3S -> Net-(D3-Pad1)
- R41 pad 2: Net-(Q16-Pad3) -> Net-(D2-Pad1)
- R42 pad 1: GND -> +4V
- R42 pad 2: VSENSE_CELL_3S -> Net-(C30-Pad2)
- R43 pad 1: VSENSE_CELL_2S -> GND
- R43 pad 2: Net-(Q17-Pad3) -> Net-(D3-Pad1)
- R44 pad 2: VSENSE_CELL_2S -> Net-(C30-Pad2)
- R45 pad 1: VSENSE_CELL_1S -> VSYS
- R45 pad 2: Net-(Q18-Pad3) -> Net-(R45-Pad2)
- R46 pad 1: GND -> Net-(R45-Pad2)
- R46 pad 2: VSENSE_CELL_1S -> Net-(C37-Pad2)
- R51 pad 1: /VPIEZO -> /Low Power and Drivers/VPIEZO
- R51 pad 2: +5V1 -> VBAT
- R52 pad 1: /VPIEZO -> DRV_PIEZO_LHS
- R52 pad 2: VBAT -> /Low Power and Drivers/VPIEZO
- R53 pad 1: Net-(D2-Pad1) -> /Low Power and Drivers/FRONT_LED_P
- R53 pad 2: Net-(D3-Pad1) -> VSYS_SW
- R54 pad 2: Net-(D2-Pad1) -> PWM_PIEZO_LHS
- R55 pad 2: PWM_PIEZO_LHS -> PWM_LED_FRONT
- R56 pad 1: GND -> DRV_PIEZO_RHS
- R56 pad 2: PWM_PIEZO_RHS -> /Low Power and Drivers/VPIEZO
- R57 pad 1: DRV_PIEZO_LHS -> GND
- R57 pad 2: /VPIEZO -> PWM_PIEZO_RHS
- R58 pad 1: DRV_PIEZO_RHS -> Net-(Q22-Pad4)
- R58 pad 2: /VPIEZO -> Net-(R58-Pad2)
- R59 pad 1: Net-(C48-Pad2) -> Net-(C45-Pad2)
- R59 pad 2: GND -> +4V_SW
- R6 pad 1: Net-(R5-Pad2) -> /Battery/~{EN_CELL_4S_DIS}
- R6 pad 2: GND -> /Battery/CELL_4S
- R60 pad 1: +4V -> VSENSE_5V1
- R60 pad 2: Net-(C49-Pad2) -> VSYS_SW
- R61 pad 1: GND -> +5V1
- R61 pad 2: Net-(C49-Pad2) -> VSENSE_5V1
- R62 pad 1: GND -> Net-(C55-Pad1)
- R62 pad 2: PWM_LED_FRONT -> Net-(C47-Pad2)
- R63 pad 1: /FRONT_LED_P -> Net-(R63-Pad1)
- R63 pad 2: VSYS_SW -> +5V1
- R64 pad 1: VSYS -> GND
- R64 pad 2: Net-(R64-Pad2) -> VSENSE_5V1
- R65 pad 1: Net-(R64-Pad2) -> GND
- R65 pad 2: Net-(C55-Pad2) -> Net-(C48-Pad2)
- R66 pad 2: EN_HIGH_POWER -> Net-(Q23-Pad4)
- R67 pad 1: Net-(R64-Pad2) -> GND
- R67 pad 2: Net-(Q22-Pad3) -> Net-(R63-Pad1)
- R7 pad 1: Net-(C5-Pad2) -> VSENSE_CELL_4S
- R7 pad 2: +4V_SW -> Net-(Q1-Pad3)
- R8 pad 1: GND -> Net-(Q1-Pad1)
- R8 pad 2: Net-(C9-Pad2) -> /Battery/CELL_4S
- R9 pad 2: Net-(C11-Pad1) -> VSYS
- U2 pad 1: VSYS_SW -> Net-(C19-Pad1)
- U2 pad 10: Net-(C19-Pad1) -> VBAT
- U2 pad 2: Net-(C7-Pad2) -> Net-(C17-Pad1)
- U2 pad 3: Net-(R20-Pad1) -> Net-(C24-Pad2)
- U2 pad 4: GND -> Net-(C27-Pad2)
- U2 pad 5: Net-(C5-Pad2) -> Net-(C21-Pad2)
- U2 pad 6: Net-(Q3-Pad4) -> Net-(R20-Pad1)
- U2 pad 7: GND -> Net-(R18-Pad1)
- U2 pad 8: Net-(R15-Pad2) -> Net-(R29-Pad2)
- U2 pad 9: Net-(C19-Pad2) -> Net-(C23-Pad1)
- U3 pad 3: Net-(R16-Pad2) -> Net-(R40-Pad2)
- U3 pad 4: Net-(Q5-Pad4) -> Net-(Q15-Pad4)
- U3 pad 5: Net-(Q4-Pad4) -> Net-(Q16-Pad4)
- U5 pad 1: Net-(C47-Pad1) -> +4V
- U5 pad 2: VSYS -> GND
- U5 pad 3: Net-(D2-Pad1) -> +4V
- U5 pad 4: GND -> unconnected-(U5-Pad4)
- U5 pad 5: Net-(C49-Pad2) -> +3V3
- U6 pad 3: /FRONT_LED_P -> /Low Power and Drivers/FRONT_LED_P
- U6 pad 7: Net-(D4-Pad2) -> Net-(D4-Pad1)
- U6 pad 8: Net-(D4-Pad2) -> Net-(D4-Pad1)
- U7 pad 1: +4V -> VSYS_SW
- U7 pad 2: GND -> Net-(C48-Pad1)
- U7 pad 3: +4V -> Net-(R63-Pad1)
- U7 pad 4: unconnected-(U7-Pad4) -> GND
- U7 pad 5: +3V3 -> Net-(C45-Pad2)

Commit message: Layout WIP
Parts:
- C2, C3, C4, C5, Y1, Y2: moved to B.Cu
- moved C48 166.2 mm to (-74.2, 207.4), turned to 180 degrees
- moved R63 164.3 mm to (-67.7, 210.9)
- moved R62 163.8 mm to (-62.9, 210.2), turned to 180 degrees
- moved R59 161.2 mm to (-69.8, 211.2), turned to 180 degrees
- moved R66 159.6 mm to (-66.1, 209.8), turned to 180 degrees
- moved C45 159.3 mm to (-69.8, 210.2), turned to 180 degrees
- moved C44 154.3 mm to (-80.4, 203.8)
- moved Q23 147.5 mm to (-64.6, 198.4), turned to 180 degrees
- moved C54 147.0 mm to (-72.7, 207.8), turned to 90 degrees
- moved C41 143.0 mm to (-80.4, 193.9)
- moved R65 141.6 mm to (-74.2, 208.4), turned to 180 degrees
- moved C43 140.1 mm to (-80.4, 200.5)
- moved R58 138.8 mm to (-64.7, 208.2), turned to 180 degrees
- moved C47 138.3 mm to (-65.2, 206.7), turned to -90 degrees
- moved C55 137.9 mm to (-61.0, 210.2)
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Connections:
- net Net-(D1-Pad3) renamed /Battery/CHG_DRN
Routing:
- net (no net): track 35.0 -> 0.00 mm

Commit message: Layout WIP
Parts:
- moved Q15 200.6 mm to (-32.5, 191.7)
- moved Q16 200.6 mm to (-38.0, 191.7)
- moved R39 200.6 mm to (-30.4, 196.2)
- moved R40 200.6 mm to (-47.3, 196.4)
- moved U3 200.6 mm to (-44.6, 195.9)
- moved R2 101.3 mm to (-23.2, 159.8)
- moved R3 99.3 mm to (-18.2, 154.9)
- moved U6 94.9 mm to (-43.9, 120.4)
- moved C28 92.3 mm to (-117.7, 100.4)
- moved C6 91.5 mm to (-20.4, 157.9)
- moved Q11 91.3 mm to (-128.9, 98.5), turned to 180 degrees
- moved R24 86.4 mm to (-118.0, 90.0)
- moved R53 84.5 mm to (-26.7, 119.6)
- moved R1 84.5 mm to (-21.6, 152.8)
- moved L4 81.6 mm to (-37.0, 111.2)
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