File: faclon-main/FalconMain/FalconMain.kicad_pcb (KiCad board)
At the start: 2 copper layers, 181 parts, among them J1 PTH, J2 JST-XH, J3 100mil, J4 100mil, J5 DNP, J6 Nano-Fit, J7 Nano-Fit, J8 Nano-Fit, J9 Nano-Fit, Q1 Q_PMOS_GSD, Q10 Q_NMOS_GSD, Q11 Q_PMOS_GSD, Q12 Q_PMOS_GSD, Q13 Q_NMOS_GSD, Q14 Q_NMOS_GSD, Q15 Q_PMOS_LFPAK, Q16 Q_PMOS_LFPAK, Q17 Q_PMOS_LFPAK, Q18 Q_PMOS_GSD, Q19 Q_NMOS_GSD, Q2 Q_PMOS_GSD, Q20 Q_NMOS_GSD, Q21 Q_NMOS_GSD, Q22 Q_NMOS_LFPAK, Q23 Q_NMOS_LFPAK, Q3 Q_NMOS_GSD, Q4 Q_PMOS_GSD, Q5 Q_PMOS_LFPAK, Q6 Q_PMOS_GSD, Q7 Q_NMOS_GSD, Q8 Q_PMOS_GSD, Q9 Q_PMOS_GSD, U1 STM32L152CBT6, U2 MAX1873TEEE+, U3 LTC4412ES6#TRPBF, U4 BD9E104FJ-E2, U5 NCP164ASN330T1G, U6 AL8843QSP-13, U7 ADP1883ARMZ-0.6-R7, Y1 8MHz, Y2 32.768kHz

Commit message: Layout WIP
Parts:
- R55: moved to B.Cu
- moved C13 218.0 mm to (-26.0, 236.7)
- moved C14 218.0 mm to (-44.5, 231.4)
- moved C16 218.0 mm to (-26.2, 239.7)
- moved C17 218.0 mm to (-31.9, 236.9)
- moved C18 218.0 mm to (-29.1, 236.2)
- moved C19 218.0 mm to (-35.5, 237.8)
- moved C21 218.0 mm to (-35.5, 241.9)
- moved C23 218.0 mm to (-28.6, 244.2)
- moved C24 218.0 mm to (-35.5, 238.9)
- moved C25 218.0 mm to (-14.4, 224.8)
- moved C26 218.0 mm to (-36.5, 239.9)
- moved C27 218.0 mm to (-36.5, 240.9)
- moved D1 218.0 mm to (-39.9, 218.3)
- moved L2 218.0 mm to (-28.2, 224.5)
- moved Q5 218.0 mm to (-39.1, 228.7)
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Connections:
- R51 pad 2: VBAT -> VSYS
Routing:
- net +5V1: track 0.00 -> 44.0 mm
- net /5V1_PHONE: track 0.00 -> 6.20 mm
- net /5V1_REAR: track 0.00 -> 2.05 mm
- net Net-(Q16-Pad4): vias 0 -> 1

Commit message: Layout WIP
Parts:
- moved C45 244.4 mm to (121.9, 80.2)
- moved C47 244.4 mm to (126.6, 76.8)
- moved C48 244.4 mm to (117.5, 77.5)
- moved C55 244.4 mm to (130.8, 80.2)
- moved R58 244.4 mm to (127.0, 78.2)
- moved R59 244.4 mm to (122.0, 81.2)
- moved R62 244.4 mm to (128.9, 80.2)
- moved R63 244.4 mm to (124.0, 81.0)
- moved R65 244.4 mm to (117.5, 78.5)
- moved R66 244.4 mm to (125.6, 79.8)
- moved R67 244.4 mm to (124.0, 82.0)
- moved C46 244.4 mm to (119.5, 80.2)
- moved C54 244.4 mm to (119.0, 77.9)
- moved U7 244.4 mm to (122.8, 77.9)
- moved C44 209.4 mm to (64.2, 68.5), turned to 180 degrees
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Connections:
- net Net-(C17-Pad1) renamed /Battery/CHG_CSSP
- net Net-(C19-Pad1) renamed /Battery/CHG_CSSN
- net Net-(C45-Pad2) renamed /High Power 5V1/5V1_BVDD
- net Net-(C47-Pad2) renamed /High Power 5V1/5V1_BSW
- net Net-(C48-Pad1) renamed /High Power 5V1/5V1_BCOMP
- net Net-(L2-Pad2) renamed /Battery/CHG_CSB
- net Net-(Q15-Pad4) renamed /Battery/PWR_OR_STAT
- net Net-(Q16-Pad4) renamed /Battery/PWR_OR_GATE
- net Net-(Q22-Pad4) renamed /High Power 5V1/5V1_BDRVH
- net Net-(Q23-Pad4) renamed /High Power 5V1/5V1_BDRVL
- net Net-(Q5-Pad4) renamed /Battery/CHG_DRV
- J9 pad 10: PWM_LED_REAR2 -> GND
- J9 pad 11: BUTTON -> PWM_LED_REAR2
- J9 pad 2: /5V1_PHONE -> GND
- J9 pad 3: GND -> /VSYS_SW_FUSED
- J9 pad 5: /VSYS_SW_FUSED -> PWM_LED_REAR1
- J9 pad 6: /ACDC_IN -> BUTTON
- J9 pad 7: GND -> /5V1_PHONE
- J9 pad 9: PWM_LED_REAR1 -> /ACDC_IN
Routing:
- net +5V1: track 44.0 -> 12.7 mm
- net /Battery/PWR_OR_STAT: track 0.00 -> 15.2 mm
- net /Battery/PWR_OR_GATE: track 0.00 -> 7.48 mm, vias 1 -> 0
- net /5V1_PHONE: track 6.20 -> 0.00 mm
- net /5V1_REAR: track 2.05 -> 0.00 mm

Commit message: Large component rough placement
Parts:
- added H1: MountingHole, MountingHole:MountingHole_2.7mm_M2.5, F.Cu at (130.0, 61.0)
- added H2: MountingHole, MountingHole:MountingHole_2.7mm_M2.5, F.Cu at (188.0, 61.0)
- added H3: MountingHole, MountingHole:MountingHole_2.7mm_M2.5, F.Cu at (130.0, 110.0)
- added H4: MountingHole, MountingHole:MountingHole_2.7mm_M2.5, F.Cu at (188.0, 110.0)
- added H5: MountingHole, MountingHole:MountingHole_2.7mm_M2.5, F.Cu at (110.0, 135.0)
- added H6: MountingHole, MountingHole:MountingHole_2.7mm_M2.5, F.Cu at (188.0, 135.0)
- C1: renamed from C7; moved to B.Cu
- C10: renamed from C5; moved to F.Cu
- C2: renamed from C8; moved to B.Cu
- C24: renamed from C25; footprint Capacitor_THT:CP_Radial_D6.3mm_P2.50mm -> JetkovKiCADLib:CP_Radial_D6.3mm_P2.50mm
- C3: renamed from C2; moved to F.Cu
- C4: renamed from C9; moved to B.Cu
- C40: renamed from C45; moved to B.Cu
- C41: renamed from C46; moved to B.Cu
- C42: renamed from C54; moved to B.Cu
- C44: renamed from C48; moved to B.Cu
- C48: renamed from C47; moved to B.Cu
- C5: renamed from C3; moved to F.Cu
- C6: renamed from C10; moved to B.Cu
- C7: renamed from C11; moved to B.Cu
- C8: renamed from C12; moved to B.Cu
- C9: renamed from C4; moved to F.Cu
- F4: renamed from F1; moved to B.Cu
- F5: renamed from F2; moved to B.Cu
- F6: renamed from F4; moved to B.Cu
- F7: renamed from F5; moved to B.Cu
- J9: renamed from J2; footprint Connector_JST:JST_XH_B5B-XH-AM_1x05_P2.50mm_Vertical -> JetkovKiCADLib:JST_XH_B5B-XH-AM_1x05_P2.50mm_Vertical
- L1, R63, U1, U7: moved to B.Cu
- R58: renamed from R59; moved to B.Cu
- R59: renamed from R65; moved to B.Cu
- R60: renamed from R58; moved to B.Cu
- R61: renamed from R66; moved to B.Cu
- R64: renamed from R67; moved to B.Cu
- Y1: moved to F.Cu
- Y2: footprint Crystal:Crystal_DS26_D2.0mm_L6.0mm_Horizontal -> JetkovKiCADLib:Crystal_DS26_D2.0mm_L6.0mm_Horizontal; moved to F.Cu
- moved Q17 219.5 mm to (187.2, 149.8)
- moved Q18 219.5 mm to (182.4, 144.7)
- moved R48 219.2 mm to (184.4, 145.1), turned to -90 degrees
- moved R41 217.9 mm to (181.2, 149.1)
- moved R47 217.1 mm to (189.2, 150.2), turned to -90 degrees
- moved D1 216.6 mm to (147.6, 109.8), turned to 180 degrees
- moved R45 216.4 mm to (185.1, 150.2), turned to 90 degrees
- moved R53 215.5 mm to (169.4, 93.6), turned to 180 degrees
- moved R42 215.1 mm to (181.2, 150.2)
- moved U5 214.5 mm to (169.4, 97.6), turned to 180 degrees
- moved R46 213.2 mm to (180.3, 145.1), turned to 90 degrees
- moved Q1 212.2 mm to (137.2, 110.6), turned to 0 degrees
- moved L4 209.6 mm to (172.6, 106.9)
- moved R52 209.4 mm to (166.4, 94.1), turned to -90 degrees
- moved C23 204.1 mm to (124.2, 116.7), turned to 0 degrees
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- renumbered C1 to C11, C6 to C12, C16 to C14, C18 to C15, C23 to C16, C19 to C18, C21 to C19, C24 to C20, C27 to C21, C26 to C22, C14 to C23, C15 to C25, C20 to C26, C22 to C27, C35 to C29, C36 to C30, C29 to C31, C38 to C32, C30 to C33, C39 to C34, C31 to C35, C32 to C36, C33 to C37, C34 to C38, C37 to C39, C40 to C43, C41 to C45, C42 to C46, C43 to C47, C44 to C49, C55 to C50, C49 to C51, C50 to C52, C51 to C53, C52 to C54, C53 to C55, D3 to D2, D2 to D3, F3 to F1, F7 to F2, F8 to F3, F9 to F8, F6 to F9, J7 to J1, J1 to J2, J9 to J3, J6 to J5, J3 to J6, J8 to J7, J5 to J8, Q5 to Q1, Q9 to Q10, Q12 to Q11, Q14 to Q12, Q1 to Q13, Q4 to Q14, Q8 to Q15, Q11 to Q16, Q20 to Q17, Q21 to Q18, Q17 to Q19, Q16 to Q2, Q19 to Q20, Q18 to Q21, Q15 to Q3, Q3 to Q4, Q7 to Q5, Q10 to Q6, Q13 to Q7, Q2 to Q8, Q6 to Q9, R5 to R1, R29 to R10, R32 to R11, R10 to R12, R31 to R13, R9 to R14, R11 to R15, R22 to R16, R40 to R17, R39 to R18, R14 to R19, R1 to R2, R21 to R20, R30 to R21, R37 to R22, R6 to R23, R15 to R24, R23 to R25, R33 to R26, R13 to R27, R19 to R28, R28 to R29, R2 to R3, R36 to R30, R8 to R31, R38 to R32, R7 to R33, R12 to R34, R16 to R35, R17 to R36, R24 to R37, R26 to R38, R34 to R39, R3 to R4, R35 to R40, R50 to R41, R51 to R42, R41 to R43, R43 to R44, R54 to R45, R57 to R46, R52 to R47, R56 to R48, R47 to R49, R4 to R5, R42 to R50, R44 to R51, R55 to R52, R45 to R54, R46 to R55, R49 to R56, R48 to R57, R27 to R6, R60 to R65, R61 to R66, R64 to R67, R18 to R7, R20 to R8, R25 to R9, U6 to U5, U5 to U6
Connections:
- J3 pad 1: /5V1_REAR -> Net-(J3-Pad1)
- J3 pad 10: GND -> /VSYS_SW_FUSED
- J3 pad 11: PWM_LED_REAR2 -> GND
- J3 pad 12: Net-(R5-Pad2) -> /5V1_REAR
- J3 pad 2: GND -> PWM_LED_REAR2
- J3 pad 3: /VSYS_SW_FUSED -> GND
- J3 pad 4: GND -> /ACDC_IN
- J3 pad 5: PWM_LED_REAR1 -> GND
- J3 pad 6: BUTTON -> /5V1_PHONE
- J3 pad 7: /5V1_PHONE -> BUTTON
- J3 pad 8: GND -> PWM_LED_REAR1
- J3 pad 9: /ACDC_IN -> GND
- R1 pad 2: Net-(R5-Pad2) -> Net-(J3-Pad1)
Routing:
- net /Battery/PWR_OR_STAT: track 15.2 -> 13.2 mm
Other:
- board outline added: 85 x 81 mm
