File: faclon-main/FalconMain/FalconMain.kicad_pcb (KiCad board)
At the start: 2 copper layers, 85 x 81 mm, 187 parts, among them J1 Nano-Fit, J2 PTH, J3 Nano-Fit, J4 100mil, J5 Nano-Fit, J6 100mil, J7 Nano-Fit, J8 DNP, J9 JST-XH, Q1 Q_PMOS_LFPAK, Q10 Q_PMOS_GSD, Q11 Q_PMOS_GSD, Q12 Q_NMOS_GSD, Q13 Q_PMOS_GSD, Q14 Q_PMOS_GSD, Q15 Q_PMOS_GSD, Q16 Q_PMOS_GSD, Q17 Q_NMOS_GSD, Q18 Q_NMOS_GSD, Q19 Q_PMOS_LFPAK, Q2 Q_PMOS_LFPAK, Q20 Q_NMOS_GSD, Q21 Q_PMOS_GSD, Q22 Q_NMOS_LFPAK, Q23 Q_NMOS_LFPAK, Q3 Q_PMOS_LFPAK, Q4 Q_NMOS_GSD, Q5 Q_NMOS_GSD, Q6 Q_NMOS_GSD, Q7 Q_NMOS_GSD, Q8 Q_PMOS_GSD, Q9 Q_PMOS_GSD, U1 STM32L152CBT6, U2 MAX1873TEEE+, U3 LTC4412ES6#TRPBF, U4 BD9E104FJ-E2, U5 AL8843QSP-13, U6 NCP164ASN330T1G, U7 ADP1883ARMZ-0.6-R7, Y1 8MHz, Y2 32.768kHz

Commit message: Rought placement done
Parts:
- added C13: 1uF, Capacitor_SMD:C_0603_1608Metric, B.Cu at (136.4, 121.9)
- added C17: 1uF, Capacitor_SMD:C_0603_1608Metric, B.Cu at (136.4, 123.4)
- added J7: 100mil, Connector_PinHeader_2.54mm:PinHeader_2x07_P2.54mm_Vertical, F.Cu at (162.8, 116.0)
- C14: renamed from C13; moved to B.Cu
- C15: value 10uF -> 1uF; footprint Capacitor_SMD:C_1210_3225Metric -> Capacitor_SMD:C_0603_1608Metric; moved to B.Cu
- C16: renamed from C14; moved to B.Cu
- C18: renamed from C16; moved to B.Cu
- C19: renamed from C17; moved to B.Cu
- C20: renamed from C18; moved to B.Cu
- C21: renamed from C19; moved to B.Cu
- C22: renamed from C20; moved to B.Cu
- C23: renamed from C21; moved to B.Cu
- C24: renamed from C22; moved to B.Cu
- J6: footprint Connector_PinHeader_2.54mm:PinHeader_2x15_P2.54mm_Vertical -> Connector_PinHeader_2.54mm:PinHeader_2x05_P2.54mm_Vertical
- R10, R11, R12, R13, R15, R6, R65, R66, R67, R7, R8, R9, U2: moved to B.Cu
- moved R56 111.5 mm to (171.5, 82.1), turned to -90 degrees
- moved D2 110.7 mm to (169.6, 66.2)
- moved D3 110.7 mm to (170.8, 69.0)
- moved R43 110.7 mm to (168.9, 67.8)
- moved R44 110.7 mm to (168.9, 68.8)
- moved Q20 108.4 mm to (169.4, 82.0), turned to 180 degrees
- moved R57 105.3 mm to (166.9, 81.2), turned to 180 degrees
- moved R54 103.4 mm to (167.4, 82.8), turned to 90 degrees
- moved R55 101.8 mm to (166.4, 82.8), turned to -90 degrees
- moved C41 100.7 mm to (166.9, 84.3), turned to 180 degrees
- moved R30 98.8 mm to (140.5, 79.0), turned to 0 degrees
- moved R22 98.6 mm to (142.7, 75.6), turned to -90 degrees
- moved Q21 98.3 mm to (163.7, 82.3), turned to 90 degrees
- moved J9 98.0 mm to (175.2, 66.1), turned to 90 degrees
- moved Q7 96.1 mm to (140.7, 75.6), turned to 180 degrees
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- renumbered C23 to C25, C24 to C26, C25 to C27, C26 to C28, C27 to C29, C28 to C30, C29 to C31, C30 to C32, C31 to C33, C32 to C34, C33 to C35, C34 to C36, C35 to C37, C36 to C38, C37 to C39, C38 to C40, C39 to C41, C40 to C42, C41 to C43, C42 to C44, C43 to C45, C44 to C46, C45 to C47, C46 to C48, C47 to C49, C48 to C50, C49 to C51, C50 to C52, C51 to C53, C52 to C54, C53 to C55, C54 to C56, C55 to C57, J9 to J10, J7 to J8, J8 to J9
Connections:
- net Net-(C39-Pad2) renamed /Low Power and Drivers/~{EN_HIGH_POWER}
- C15 pad 1: GND -> Net-(C13-Pad1)
- C15 pad 2: Net-(C15-Pad2) -> GND
- J6 pad 1: GND -> +5V1
- J6 pad 10: +5V1 -> GND
- J6 pad 2: +5V1 -> GND
- J6 pad 3: GND -> +5V1
- J6 pad 4: +5V1 -> GND
- J6 pad 5: GND -> +5V1
- J6 pad 6: +5V1 -> GND
- J6 pad 7: GND -> +5V1
- J6 pad 8: +5V1 -> GND
- J6 pad 9: GND -> +5V1
- R42 pad 2: VSYS -> /Low Power and Drivers/VSYS_SW_FUSED
- U2 pad 16: Net-(C15-Pad2) -> Net-(C13-Pad1)
Routing:
- net +5V1: track 12.7 -> 204.0 mm
- net /FRONT_LED_P: track 0.00 -> 50.9 mm
- net VSYS_SW: track 0.00 -> 45.6 mm
- net /Low Power and Drivers/FRONT_LED_N: track 0.00 -> 35.2 mm
- net VSYS: track 0.00 -> 25.2 mm
- net /Battery/PWR_OR_STAT: track 13.2 -> 14.0 mm
Other:
- outline, holes or cut-outs redrawn

Commit message: Layout WIP
Parts:
- H1, H2, H3, H4, H5, H6: footprint MountingHole:MountingHole_2.7mm_M2.5 -> JetkovKiCADLib:MountingHole_2.7mm_M2.5_Clearanced
- moved J8 10.7 mm to (158.3, 130.2), turned to 90 degrees
- moved Q18 10.4 mm to (158.2, 136.2), turned to 180 degrees
- moved R46 10.2 mm to (160.3, 136.6), turned to -90 degrees
- moved R48 9.14 mm to (157.7, 134.3), turned to 180 degrees
- moved R42 7.36 mm to (166.1, 136.6)
- moved R41 6.15 mm to (167.2, 136.6)
- moved R45 4.99 mm to (185.9, 130.8), turned to -90 degrees
- moved R47 2.59 mm to (181.8, 130.1), turned to 90 degrees
- moved Q17 2.03 mm to (183.8, 130.5), turned to 180 degrees
- moved D4 1.33 mm to (160.4, 106.3)
- moved Q23 1.16 mm to (117.0, 96.6)
- moved J4 1.13 mm to (162.8, 122.9)
- moved C55 0.94 mm to (126.2, 85.6)
- moved C53 0.94 mm to (132.8, 85.6)
- moved C54 0.94 mm to (129.4, 85.6)
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Connections:
- net Net-(F1-Pad2) renamed /BATT_P
Routing:
- net +5V1: track 204.0 -> 0.00 mm
- net VSYS_SW: track 45.6 -> 0.00 mm
- net VSYS: track 25.2 -> 0.00 mm
- net +19V5: track 0.22 -> 4.89 mm
- added copper zone on F.Cu, net +19V5
- added copper zone on F.Cu, net +5V1
- added copper zone on F.Cu, net /5V1_PHONE
- added copper zone on F.Cu, net /5V1_REAR
- added copper zone on F.Cu, net /ACDC_IN
- added copper zone on F.Cu, net /BATT_P
- added copper zone on F.Cu, net /Battery/CHG_CSB
- added copper zone on F.Cu, net VBAT
- added copper zone on F.Cu, net VDC
- added copper zone on F.Cu, net VSYS
- added copper zone on F.Cu, net VSYS_SW
Other:
- board text added: "BATT 4S"

Commit message: Reviewed again
Parts:
- moved F4 10.0 mm to (142.5, 131.1)
- moved F7 5.00 mm to (150.0, 131.1)
- moved F5 5.00 mm to (145.0, 131.1)
- moved C14 3.29 mm to (139.9, 127.6), turned to 0 degrees
- moved C13 1.02 mm to (136.6, 122.6)
- moved C15 1.02 mm to (136.5, 125.7)
- moved C17 1.02 mm to (136.6, 124.2)
- moved F6 0.06 mm to (147.5, 131.1)
Connections:
- net Net-(C18-Pad1) renamed /Battery/CHG_VREF
- net Net-(C33-Pad1) renamed /Low Power and Drivers/4VB_BOOT
- net Net-(C33-Pad2) renamed /Low Power and Drivers/4VB_SW
- net Net-(C34-Pad1) renamed /Low Power and Drivers/4VB_CMP
- net Net-(C35-Pad2) renamed /Low Power and Drivers/4VB_FB
- net Net-(D2-Pad1) renamed /Low Power and Drivers/4VB_EN
- net Net-(R10-Pad2) renamed /Battery/CHG_VADJ
- J10 pad 1: GND -> Net-(F4-Pad2)
- J10 pad 2: Net-(F7-Pad2) -> Net-(F5-Pad2)
- J10 pad 4: Net-(F5-Pad2) -> Net-(F7-Pad2)
- J10 pad 5: Net-(F4-Pad2) -> GND
Routing:
- net /Low Power and Drivers/FRONT_LED_P: track 0.00 -> 50.9 mm
- net /FRONT_LED_P: track 50.9 -> 0.00 mm
- net +19V5: track 4.89 -> 0.22 mm
- net Net-(F7-Pad2): track 0.00 -> 2.08 mm
- net Net-(F6-Pad2): track 0.00 -> 2.05 mm
- net Net-(F5-Pad2): track 0.00 -> 2.05 mm
- net Net-(F4-Pad2): track 0.00 -> 2.05 mm
- net /CELL_4S: track 0.00 -> 1.90 mm, vias 0 -> 2
- net /CELL_3S: track 0.00 -> 1.78 mm, vias 0 -> 2
- net /CELL_2S: track 0.00 -> 1.78 mm, vias 0 -> 2
- net /CELL_1S: track 0.00 -> 1.75 mm, vias 0 -> 2
Other:
- copper layers 2 -> 4
- board text added: "LiPo 4S"
- board text removed: "BATT 4S"
